File: Hardware/ScienceMotorController_Hardware/ScienceMotorController_Hardware.sch (KiCad schematic (older format))
At the start: 64 parts, among them U1 TM4C129E_Launchpad, U2 3.3V OKI, U3 5V OKI, U4 VNH5019A_E, U5 VNH5019A_E, U6 VNH5019A_E, U7 VNH5019A_E

Commit message: Added Indicators and Pins
Parts:
- removed Conn? (x4): Molex_SL_02, symbol MRDT_Connectors:Molex_SL_02
- added D? (x4): LED_Small, symbol Device:LED_Small
- added D? (x3): M4_OUT_A_LED, symbol Device:LED_Small
- added D?: 3.3V_LED, symbol Device:LED_Small
- added D?: 5VL_LED, symbol Device:LED_Small
- added D?: 12VA_LED, symbol Device:LED_Small
- added D? (x3): M4_OUT_B_LED, symbol Device:LED_Small
- added D?: M3_OUT_A_LED, symbol Device:LED_Small
- added D?: M3_OUT_B_LED, symbol Device:LED_Small
- added D? (x2): LS_3_LED, symbol Device:LED_Small
- added D? (x2): LS_4_LED, symbol Device:LED_Small
- added D? (x2): LS_2_LED, symbol Device:LED_Small
- added D? (x2): LS_1_LED, symbol Device:LED_Small
- added R? (x4): 1K, symbol Device:R_Small
- added R? (x10): 500, symbol Device:R_Small
- added R? (x9): 1.5K, symbol Device:R_Small
Connections:
- net labels removed: LS_5, LS_6, LS_7, LS_8, M1_A, M1_B, M2_A, M2_B, M3_A, M3_B, M4_A, M4_B
- wire segments 305 -> 411
Other:
- note added: "Green"
- note added: "H-Bridges"
- note added: "Indicators"
- note added: "Limit Switches"
- note added: "Motor Outputs"
- note added: "Orange"
- note added: "Power Conversion"
- note added: "Power Inputs"
- note added: "TIVA Headers"
- note added: "Yellow"

Commit message: Controls Added and Schematic Organized
Parts:
- removed Conn? (x4): Molex_SL_02, symbol MRDT_Connectors:Molex_SL_02
- added Conn? (x4): Molex_SL_02, symbol MRDT_Connectors:Molex_SL_02
- added R? (x4): 500, symbol Device:R_Small
- added SW? (x4): SW_Push, symbol Switch:SW_Push
Connections:
- net labels added: MSW_1, MSW_2, MSW_3, MSW_4
- wire segments 411 -> 431
Other:
- note added: "Manual Controls"

Commit message: Updated Schematic Labels and Organization
Parts:
- C1, C2, C3, C4: renamed from C?; value C -> 10uF
- C5, C6, C7, C8: renamed from C?; value 33 nF -> 33nF
- D?: value LED_Small -> M1_PWM_LED
- D?: value LED_Small -> M2_PWM_LED
- D?: value LED_Small -> M3_PWM_LED
- D?: value LED_Small -> M4_PWM_LED
- D?: value LS_3_LED -> SW_IND_3_LED
- D?: value LS_4_LED -> SW_IND_4_LED
- D?: value LS_2_LED -> SW_IND_2_LED
- D?: value LS_1_LED -> SW_IND_1_LED
- gave numbers to parts that had none: 67
Connections:
- net labels added: SW_IND_1, SW_IND_2, SW_IND_3, SW_IND_4
- wire segments 431 -> 458
Other:
- note added: "Red"

Commit message: (Most) Footprints Assigned
Parts:
- C1, C2, C3, C4, C5, C6, C7, C8: footprint (none) -> Capacitor_SMD:C_0603_1608Metric_Pad1.05x0.95mm_HandSolder
- Conn2, Conn3, Conn4, Conn5: footprint (none) -> MRDT_Connectors:Anderson_2_Horizontal_Side_by_Side
- Conn6, Conn7, Conn8, Conn9: footprint (none) -> MRDT_Connectors:MOLEX_SL_02_Horizontal
- D1, D10, D11, D12, D13, D14, D15, D16, D17, D18, D19, D2, D20, D21, D22, D23, D3, D4, D5, D6, D7, D8, D9: renamed from D?; footprint (none) -> LED_SMD:LED_0603_1608Metric_Pad1.05x0.95mm_HandSolder
- R1, R10, R11, R12, R13, R14, R15, R16, R17, R18, R19, R2, R20, R21, R22, R23, R24, R25, R26, R27, R28, R29, R3, R30, R31, R32, R33, R34, R35, R36, R37, R38, R39, R4, R40, R41, R42, R43, R44, R45, R46, R47, R48, R49, R5, R50, R51, R52, R53, R54, R55, R6, R7, R8, R9: footprint (none) -> Resistor_SMD:R_0603_1608Metric_Pad1.05x0.95mm_HandSolder
- U2, U3: footprint (none) -> MRDT_Devices:OKI_Horizontal

Commit message: Footprints and Pins Finished Schematic
Parts:
- removed JP1, JP2, JP3, JP4: Jumper_NC_Small, symbol Device:Jumper_NC_Small
- SW1, SW2, SW3, SW4: footprint (none) -> Button_Switch_SMD:SW_SPST_TL3305A
- U1: footprint (none) -> MRDT_Shields:TM4C129E_Launchpad_FULL_THT_BOTTOM
- U4, U5, U6, U7: footprint (none) -> MRDT_ICs:MultiPowerSO_30
Connections:
- wire segments 458 -> 467

Commit message: Basic board organization
Parts:
- D16: value M4_OUT_A_LED -> M1_OUT_A_LED
- D17: value M4_OUT_B_LED -> M1_OUT_B_LED
- D18: value M4_OUT_A_LED -> M2_OUT_A_LED
- D19: value M4_OUT_B_LED -> M2_OUT_B_LED
Changed lines of the file:
@@
 P 12950 6675
 F 0 "D16" H 12950 6800 50  0000 C CNN
-F 1 "M4_OUT_A_LED" H 12950 6600 50  0000 C CNN
+F 1 "M1_OUT_A_LED" H 12950 6600 50  0000 C CNN
 F 2 "LED_SMD:LED_0603_1608Metric_Pad1.05x0.95mm_HandSolder" V 12950 6675 50  0001 C CNN
 F 3 "~" V 12950 6675 50  0001 C CNN
@@
 P 12950 7375
 F 0 "D18" H 12950 7500 50  0000 C CNN
-F 1 "M4_OUT_A_LED" H 12950 7300 50  0000 C CNN
+F 1 "M2_OUT_A_LED" H 12950 7300 50  0000 C CNN
 F 2 "LED_SMD:LED_0603_1608Metric_Pad1.05x0.95mm_HandSolder" V 12950 7375 50  0001 C CNN
 F 3 "~" V 12950 7375 50  0001 C CNN
@@
 P 12950 7725
 F 0 "D19" H 12950 7850 50  0000 C CNN
-F 1 "M4_OUT_B_LED" H 12950 7650 50  0000 C CNN
+F 1 "M2_OUT_B_LED" H 12950 7650 50  0000 C CNN
 F 2 "LED_SMD:LED_0603_1608Metric_Pad1.05x0.95mm_HandSolder" V 12950 7725 50  0001 C CNN
 F 3 "~" V 12950 7725 50  0001 C CNN
@@
 P 12950 7025
 F 0 "D17" H 12950 7150 50  0000 C CNN
-F 1 "M4_OUT_B_LED" H 12950 6950 50  0000 C CNN
+F 1 "M1_OUT_B_LED" H 12950 6950 50  0000 C CNN
 F 2 "LED_SMD:LED_0603_1608Metric_Pad1.05x0.95mm_HandSolder" V 12950 7025 50  0001 C CNN
 F 3 "~" V 12950 7025 50  0001 C CNN
@@
 	3525 8375 3625 8375
 $Comp
-L power:GND #PWR?
+L power:GND #PWR0118
 U 1 1 66986FAD
 P 4725 4475
-F 0 "#PWR?" H 4725 4225 50  0001 C CNN
+F 0 "#PWR0118" H 4725 4225 50  0001 C CNN
 F 1 "GND" H 4730 4302 50  0000 C CNN
 F 2 "" H 4725 4475 50  0001 C CNN
@@
 Connection ~ 8225 3000
 $Comp
-L power:GND #PWR?
+L power:GND #PWR0122
 U 1 1 66E72E79
 P 4725 2375
-F 0 "#PWR?" H 4725 2125 50  0001 C CNN
+F 0 "#PWR0122" H 4725 2125 50  0001 C CNN
 F 1 "GND" H 4730 2202 50  0000 C CNN
 F 2 "" H 4725 2375 50  0001 C CNN
@@
 	4725 2350 4850 2350
 $Comp
-L power:GND #PWR?
+L power:GND #PWR0126
 U 1 1 66EF83EB
 P 8275 2375
-F 0 "#PWR?" H 8275 2125 50  0001 C CNN
+F 0 "#PWR0126" H 8275 2125 50  0001 C CNN
 F 1 "GND" H 8280 2202 50  0000 C CNN
 F 2 "" H 8275 2375 50  0001 C CNN
@@
 	8275 2350 8400 2350
 $Comp
-L power:GND #PWR?
+L power:GND #PWR0130
 U 1 1 66F7DE40
 P 8275 4475
-F 0 "#PWR?" H 8275 4225 50  0001 C CNN
+F 0 "#PWR0130" H 8275 4225 50  0001 C CNN
 F 1 "GND" H 8280 4302 50  0000 C CNN
 F 2 "" H 8275 4475 50  0001 C CNN

Commit message: Went Overboard on Traces
Connections:
- no-connect marks 0 -> 74
Changed lines of the file:
@@
 Wire Notes Line
 	2000 9575 13500 9575
+NoConn ~ 4575 6900
+NoConn ~ 4575 7000
+NoConn ~ 4575 7100
+NoConn ~ 4575 7200
+NoConn ~ 4575 7300
+NoConn ~ 4575 7400
+NoConn ~ 4575 7500
+NoConn ~ 4575 7600
+NoConn ~ 4575 7700
+NoConn ~ 5475 7000
+NoConn ~ 5475 6800
+NoConn ~ 5475 7300
+NoConn ~ 5475 7400
+NoConn ~ 5475 7500
+NoConn ~ 5475 7600
+NoConn ~ 5475 7700
+NoConn ~ 5475 8125
+NoConn ~ 5475 8225
+NoConn ~ 5475 8325
+NoConn ~ 5475 8525
+NoConn ~ 5475 8425
+NoConn ~ 4575 8925
+NoConn ~ 4575 8825
+NoConn ~ 4575 8725
+NoConn ~ 4575 8625
+NoConn ~ 4575 8525
+NoConn ~ 4575 8425
+NoConn ~ 4575 8325
+NoConn ~ 4575 8225
+NoConn ~ 3500 8425
+NoConn ~ 3500 8825
+NoConn ~ 3500 8925
+NoConn ~ 2600 8525
+NoConn ~ 2600 8225
+NoConn ~ 2600 6900
+NoConn ~ 2600 7000
+NoConn ~ 2600 7100
+NoConn ~ 2600 7200
+NoConn ~ 2600 7300
+NoConn ~ 2600 7400
+NoConn ~ 2600 7500
+NoConn ~ 2600 7600
+NoConn ~ 2600 7700
+NoConn ~ 3500 7300
+NoConn ~ 3500 7200
+NoConn ~ 3500 6800
+NoConn ~ 5825 3750
+NoConn ~ 5825 3850
+NoConn ~ 5825 3950
+NoConn ~ 5825 4050
+NoConn ~ 5825 4150
+NoConn ~ 5825 4250
+NoConn ~ 5825 5100
+NoConn ~ 9375 5100
+NoConn ~ 9375 4250
+NoConn ~ 9375 4150
+NoConn ~ 9375 4050
+NoConn ~ 9375 3950
+NoConn ~ 9375 3850
+NoConn ~ 9375 3750
+NoConn ~ 9375 3000
+NoConn ~ 9375 2150
+NoConn ~ 9375 1650
+NoConn ~ 9375 1750
+NoConn ~ 9375 1850
+NoConn ~ 9375 1950
+NoConn ~ 9375 2050
+NoConn ~ 5825 3000
+NoConn ~ 5825 2150
+NoConn ~ 5825 2050
+NoConn ~ 5825 1950
+NoConn ~ 5825 1850
+NoConn ~ 5825 1750
+NoConn ~ 5825 1650
 $EndSCHEMATC
