File: Hardware/ScienceMotorController_Hardware/ScienceMotorController_Hardware.sch (KiCad schematic (older format))
At the start: 106 parts, among them SW1 SW_Push, SW2 SW_Push, SW3 SW_Push, SW4 SW_Push, U1 TM4C129E_Launchpad, U2 3.3V OKI, U3 5V OKI, U4 VNH5019A_E, U5 VNH5019A_E, U6 VNH5019A_E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

Commit message: Almost All Traces, Ground and 3V3 Polygons
Connections:
- wire segments 467 -> 475
Changed lines of the file:
@@
 NoConn ~ 5825 1750
 NoConn ~ 5825 1650
+Wire Wire Line
+	10975 4950 11075 4950
+Wire Wire Line
+	11075 4950 11075 4850
+Connection ~ 11075 4850
+Wire Wire Line
+	10975 2850 11075 2850
+Wire Wire Line
+	11075 2850 11075 2750
+Connection ~ 11075 2750
+Wire Wire Line
+	7425 2850 7525 2850
+Wire Wire Line
+	7525 2850 7525 2750
+Connection ~ 7525 2750
+Wire Wire Line
+	7425 4950 7525 4950
+Wire Wire Line
+	7525 4950 7525 4850
+Connection ~ 7525 4850
 $EndSCHEMATC

Commit message: PDR Advice
Removed 2 limit switches & relocated LS LEDs, added direction switch. Also relocated LS, Control, and Indicator blocks and revamped pin assignments to optimize traces.
Parts:
- removed Conn8, Conn9: Molex_SL_02, MRDT_Connectors:MOLEX_SL_02_Horizontal, symbol MRDT_Connectors:Molex_SL_02
- removed D10: LS_3_LED, LED_SMD:LED_0603_1608Metric_Pad1.05x0.95mm_HandSolder, symbol Device:LED_Small
- removed D11: LS_4_LED, LED_SMD:LED_0603_1608Metric_Pad1.05x0.95mm_HandSolder, symbol Device:LED_Small
- removed R42, R43: 500, Resistor_SMD:R_0603_1608Metric_Pad1.05x0.95mm_HandSolder, symbol Device:R_Small
- added R56: 500, Resistor_SMD:R_0603_1608Metric_Pad1.05x0.95mm_HandSolder, symbol Device:R_Small
- added SW5: SW_Push, Button_Switch_SMD:SW_SPST_TL3305A, symbol Switch:SW_Push
Connections:
- net labels added: MSW_5
- net labels removed: LS_3, LS_4
- wire segments 475 -> 469
- no-connect marks 74 -> 67

Commit message: Finished Traces
Connections:
- wire segments 469 -> 468
- no-connect marks 67 -> 75
Changed lines of the file:
@@
 Text GLabel 3600 8625 2    50   Input ~ 0
 M2_CS
+Text GLabel 3600 8925 2    50   Output ~ 0
+M2_IN_A
 Text GLabel 2500 8825 0    50   Output ~ 0
-M2_IN_A
-Text GLabel 3600 8925 2    50   Output ~ 0
 M2_PWM
 Text GLabel 2500 8925 0    50   Output ~ 0
@@
 	2600 8425 2500 8425
 Connection ~ 8500 8100
-Connection ~ 9575 8600
-Wire Wire Line
-	9575 8600 9575 8500
 Wire Wire Line
 	9575 8500 9575 9025
+NoConn ~ 3500 8325
+NoConn ~ 3500 8225
+NoConn ~ 3500 8125
+NoConn ~ 3500 8725
+NoConn ~ 3500 7100
+NoConn ~ 3500 7000
+NoConn ~ 3500 7600
+NoConn ~ 3500 7700
 $EndSCHEMATC

Commit message: Similar to PostPDR, but using 3V3 instead of 5V for VNH5019A-E
Parts:
- removed C3, C4: 10uF, Capacitor_SMD:C_0603_1608Metric_Pad1.05x0.95mm_HandSolder, symbol Device:C
- removed D2: 5VL_LED, LED_SMD:LED_0603_1608Metric_Pad1.05x0.95mm_HandSolder, symbol Device:LED_Small
- removed R34: 500, Resistor_SMD:R_0603_1608Metric_Pad1.05x0.95mm_HandSolder, symbol Device:R_Small
- removed U3: 5V OKI, MRDT_Devices:OKI_Horizontal, symbol MRDT_Devices:OKI
Connections:
- net labels removed: +5VL
- wire segments 468 -> 454
