File: ScienceMotorController/ScienceMotorController_Hardware/ScienceMotorController_Hardware/ScienceMotorController_Hardware.kicad_pcb (KiCad board)
At the start: 2 copper layers, 124.5 x 104.9 mm, 100 parts, among them SW1 SW_Push, SW2 SW_Push, SW3 SW_Push, SW4 SW_Push, SW5 SW_Push, U1 TM4C129E_Launchpad, U2 3.3V OKI, U4 VNH5019A_E, U5 VNH5019A_E, U6 VNH5019A_E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

Commit message: Moving to Rev1 PRR
Parts:
- added C10: 470 uF, Capacitor_THT:CP_Radial_D8.0mm_P3.50mm, F.Cu at (155.0, 68.6)
- added C3: 470 uF, Capacitor_THT:CP_Radial_D8.0mm_P3.50mm, F.Cu at (146.2, 60.0)
- added C4: 470 uF, Capacitor_THT:CP_Radial_D8.0mm_P3.50mm, F.Cu at (146.2, 68.6)
- added C9: 470 uF, Capacitor_THT:CP_Radial_D8.0mm_P3.50mm, F.Cu at (155.0, 60.0)
- added Conn8: Molex_SL_02, MRDT_Connectors:MOLEX_SL_02_Vertical, F.Cu at (81.4, 123.7)
- added Conn9: Molex_SL_02, MRDT_Connectors:MOLEX_SL_02_Vertical, F.Cu at (94.5, 123.7)
- added D10: LS_2_LED, LED_SMD:LED_0603_1608Metric_Pad1.05x0.95mm_HandSolder, F.Cu at (92.3, 128.7)
- added D2: LS_1_LED, LED_SMD:LED_0603_1608Metric_Pad1.05x0.95mm_HandSolder, F.Cu at (79.3, 128.7)
- added D24: 3.3, Diode_SMD:D_0603_1608Metric_Pad1.05x0.95mm_HandSolder, F.Cu at (45.6, 100.6)
- added D25: 3.3, Diode_SMD:D_0603_1608Metric_Pad1.05x0.95mm_HandSolder, F.Cu at (72.6, 100.6)
- added D26: 3.3, Diode_SMD:D_0603_1608Metric_Pad1.05x0.95mm_HandSolder, F.Cu at (99.6, 100.6)
- added D27: 3.3, Diode_SMD:D_0603_1608Metric_Pad1.05x0.95mm_HandSolder, F.Cu at (126.2, 100.6)
- added R42: 330, Resistor_SMD:R_0603_1608Metric_Pad1.05x0.95mm_HandSolder, F.Cu at (83.4, 128.7)
- added R43: 330, Resistor_SMD:R_0603_1608Metric_Pad1.05x0.95mm_HandSolder, F.Cu at (96.5, 128.7)
- R16, R2, R20, R23, R27, R9: value 3.3K -> 1K
- R39, R40, R41: value 500 -> 330
- R44, R45, R46, R47: value 1K -> 330
- moved D15 95.9 mm to (121.9, 49.6), turned to 270 degrees
- moved D12 88.8 mm to (41.2, 49.6), turned to 270 degrees
- moved R47 87.2 mm to (121.9, 56.2), turned to 270 degrees
- moved R44 86.5 mm to (41.2, 56.2), turned to 270 degrees
- moved D14 85.4 mm to (95.2, 49.6), turned to 270 degrees
- moved D13 82.8 mm to (68.1, 49.6), turned to 270 degrees
- moved R46 78.2 mm to (95.2, 56.2), turned to 270 degrees
- moved R45 77.9 mm to (68.1, 56.2), turned to 270 degrees
- moved D9 39.1 mm to (92.3, 117.2)
- moved Conn6 39.1 mm to (81.4, 112.3)
- moved Conn7 39.1 mm to (94.5, 112.3)
- moved D8 39.1 mm to (79.3, 117.2)
- moved R41 39.1 mm to (96.5, 117.2)
- moved R40 39.1 mm to (83.4, 117.2)
- moved R36 38.8 mm to (114.0, 120.5)
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Connections:
- R39 pad 1: SW_IND_4 -> SW_ERR
- U1 pad PA4: Net-(U1-PadPA4) -> SW_IND_2
- U1 pad PA5: Net-(U1-PadPA5) -> SW_IND_1
- U1 pad PA6: LS_2 -> LS_1
- U1 pad PB2: SW_IND_3 -> Net-(U1-PadPB2)
- U1 pad PB3: SW_IND_4 -> Net-(U1-PadPB3)
- U1 pad PC7: SW_IND_2 -> Net-(U1-PadPC7)
- U1 pad PD3: SW_IND_1 -> MSW_5
- U1 pad PD7: LS_1 -> LS_3
- U1 pad PE0: Net-(U1-PadPE0) -> MSW_1
- U1 pad PE1: Net-(U1-PadPE1) -> MSW_2
- U1 pad PE2: Net-(U1-PadPE2) -> MSW_3
- U1 pad PE3: Net-(U1-PadPE3) -> MSW_4
- U1 pad PF1: MSW_3 -> Net-(U1-PadPF1)
- U1 pad PF2: MSW_4 -> Net-(U1-PadPF2)
- U1 pad PF3: MSW_1 -> M1_PWM
- U1 pad PG0: MSW_2 -> M2_PWM
- U1 pad PK2: Net-(U1-PadPK2) -> SW_ERR
- U1 pad PK3: Net-(U1-PadPK3) -> SW_IND_3
- U1 pad PL2: M2_PWM -> Net-(U1-PadPL2)
- U1 pad PL4: MSW_5 -> Net-(U1-PadPL4)
- U1 pad PL5: M1_PWM -> Net-(U1-PadPL5)
- U1 pad PM4: Net-(U1-PadPM4) -> LS_2
- U1 pad PM5: Net-(U1-PadPM5) -> LS_4
Routing:
- net +3V3: track 7.95 -> 473.8 mm, vias 2 -> 1
- net GND: track 182.7 -> 0.93 mm, vias 33 -> 26
- net MSW_5: track 76.9 -> 19.8 mm
- net LS_2: track 11.5 -> 59.0 mm, vias 0 -> 1
- net LS_4: track 0.00 -> 47.3 mm, vias 0 -> 1
- net LS_3: track 0.00 -> 43.2 mm, vias 0 -> 1
- net +12L: track 53.2 -> 10.1 mm
- net LS_1: track 14.4 -> 54.4 mm, vias 0 -> 1
- net MSW_4: track 60.7 -> 38.8 mm
- net SW_IND_4: track 19.4 -> 0.00 mm, vias 1 -> 0
- net MSW_3: track 41.8 -> 23.9 mm
- net M1_PWM: track 75.0 -> 58.2 mm, vias 4 -> 2
- net M4_PWM: track 83.1 -> 67.8 mm, vias 2 -> 4
- net +12VA: track 204.5 -> 189.6 mm, vias 202 -> 201
- net SW_IND_3: track 24.8 -> 12.5 mm
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- added copper zone on F.Cu, net GND
- removed copper zone on F.Cu, net +3V3
Other:
- board size 124.5 x 104.9 mm -> 124.5 x 120.6 mm
- board text added: "Software Error"
- board text added: "Switch 3"
- board text added: "Switch 4"
- board text removed: "5VL"
- board text removed: "Software 4"
