File: ScienceMotorController/ScienceMotorController_Hardware/ScienceMotorController_Hardware/ScienceMotorController_Hardware.sch (KiCad schematic (older format))
At the start: 102 parts, among them SW1 SW_Push, SW2 SW_Push, SW3 SW_Push, SW4 SW_Push, SW5 SW_Push, U1 TM4C129E_Launchpad, U2 3.3V OKI, U3 5V OKI, U4 VNH5019A_E, U5 VNH5019A_E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

Commit message: Moving to Rev1 PRR
Parts:
- removed C3, C4: 10uF, Capacitor_SMD:C_0603_1608Metric_Pad1.05x0.95mm_HandSolder, symbol Device:C
- removed R34: 500, Resistor_SMD:R_0603_1608Metric_Pad1.05x0.95mm_HandSolder, symbol Device:R_Small
- removed SW5: SW_Push, Button_Switch_SMD:SW_SPST_TL3305A, symbol Switch:SW_Push
- removed U3: 5V OKI, MRDT_Devices:OKI_Horizontal, symbol MRDT_Devices:OKI
- added C10, C3, C4, C9: 470 uF, Capacitor_THT:CP_Radial_D8.0mm_P3.50mm, symbol Device:CP1
- added Conn8, Conn9: Molex_SL_02, MRDT_Connectors:MOLEX_SL_02_Vertical, symbol MRDT_Connectors:Molex_SL_02
- added D10: LS_2_LED, LED_SMD:LED_0603_1608Metric_Pad1.05x0.95mm_HandSolder, symbol Device:LED_Small
- added D24, D25, D26, D27: 3.3, Diode_SMD:D_0603_1608Metric_Pad1.05x0.95mm_HandSolder, symbol Device:D_Zener_Small
- added R42, R43: 330, Resistor_SMD:R_0603_1608Metric_Pad1.05x0.95mm_HandSolder, symbol Device:R_Small
- added SW5: SW_SPDT, Button_Switch_THT:SW_CuK_OS102011MA1QN1_SPDT_Angled, symbol Switch:SW_SPDT
- Conn6, Conn7: footprint MRDT_Connectors:MOLEX_SL_02_Horizontal -> MRDT_Connectors:MOLEX_SL_02_Vertical
- D2: value 5VL_LED -> LS_1_LED
- R16, R2, R20, R23, R27, R9: value 3.3K -> 1K
- R39, R40, R41: value 500 -> 330
- R44, R45, R46, R47: value 1K -> 330
- U1: footprint MRDT_Shields:TM4C129E_Launchpad_FULL_THT_BOTTOM -> MRDT_Shields:TM4C129E_Launchpad_FULL_SMD_BOTTOM
Connections:
- net labels added: LS_3, LS_4, SW_ERR
- net labels removed: +5VL, SW_IND_4
- wire segments 468 -> 494
- no-connect marks 75 -> 69
Other:
- note added: "Blue"
- note added: "Capacitance"
- note added: "M0PWM3"
- note added: "M0PWM4"
- note added: "M0PWM5"
- note added: "M0PWM6"
