File: ScienceMotorController/ScienceMotorController_Hardware/_saved_ScienceMotorController_Hardware.sch (KiCad schematic (older format))
At the start: 111 parts, among them SW1 SW_Push, SW2 SW_Push, SW3 SW_Push, SW4 SW_Push, SW5 SW_SPDT, U1 TM4C129E_Launchpad, U2 3.3V OKI, U4 VNH5019A_E, U5 VNH5019A_E, U6 VNH5019A_E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

Commit message: BOM
Parts:
- D10: value LS_2_LED -> LS_4_LED
- D2: value LS_1_LED -> LS_3_LED
- D7: value SW_IND_4_LED -> SW_ERR_LED
Changed lines of the file:
@@
 P 12950 3550
 F 0 "D7" H 12950 3675 50  0000 C CNN
-F 1 "SW_IND_4_LED" H 12950 3475 50  0000 C CNN
+F 1 "SW_ERR_LED" H 12950 3475 50  0000 C CNN
 F 2 "LED_SMD:LED_0603_1608Metric_Pad1.05x0.95mm_HandSolder" V 12950 3550 50  0001 C CNN
 F 3 "~" V 12950 3550 50  0001 C CNN
@@
 Text GLabel 7825 7700 0    50   Output ~ 0
 LS_2
-Text GLabel 3950 7000 2    50   Input ~ 0
+Text GLabel 3950 7100 2    50   Input ~ 0
 MSW_1
-Text GLabel 3950 7100 2    50   Input ~ 0
+Text GLabel 3950 7300 2    50   Input ~ 0
 MSW_2
 Text GLabel 3950 7200 2    50   Input ~ 0
 MSW_3
-Text GLabel 3950 7300 2    50   Input ~ 0
+Text GLabel 2850 7400 0    50   Input ~ 0
 MSW_4
 Wire Notes Line
@@
 	3950 7200 3850 7200
 Wire Wire Line
-	3950 7300 3850 7300
+	2850 7400 2950 7400
 Text GLabel 6525 7700 2    50   Output ~ 0
 SW_IND_1
@@
 	3950 6675 3950 6900
 Wire Wire Line
-	3850 7000 3950 7000
-Wire Wire Line
 	3850 7100 3950 7100
+Wire Wire Line
+	3850 7300 3950 7300
 Text GLabel 12350 2500 0    50   Input ~ 0
 SW_IND_1
@@
 $EndComp
 Connection ~ 10175 9075
-Wire Wire Line
-	9100 8250 9100 8775
-Text GLabel 2850 7400 0    50   Input ~ 0
+Text GLabel 3950 7000 2    50   Input ~ 0
 MSW_5
 Wire Wire Line
-	2950 7400 2850 7400
+	3850 7000 3950 7000
 Wire Wire Line
 	10175 8550 10175 9075
@@
 P 12950 4925
 F 0 "D10" H 12950 5050 50  0000 C CNN
-F 1 "LS_2_LED" H 12950 4850 50  0000 C CNN
+F 1 "LS_4_LED" H 12950 4850 50  0000 C CNN
 F 2 "LED_SMD:LED_0603_1608Metric_Pad1.05x0.95mm_HandSolder" V 12950 4925 50  0001 C CNN
 F 3 "~" V 12950 4925 50  0001 C CNN
@@
 P 12950 4575
 F 0 "D2" H 12950 4700 50  0000 C CNN
-F 1 "LS_1_LED" H 12950 4500 50  0000 C CNN
+F 1 "LS_3_LED" H 12950 4500 50  0000 C CNN
 F 2 "LED_SMD:LED_0603_1608Metric_Pad1.05x0.95mm_HandSolder" V 12950 4575 50  0001 C CNN
 F 3 "~" V 12950 4575 50  0001 C CNN
@@
 $EndComp
 NoConn ~ 9600 8875
+Wire Wire Line
+	9100 8150 9100 8775
+Connection ~ 9100 8150
 $EndSCHEMATC
