File: Hardware/ScienceMotorController/ScienceMotorController02.sch (KiCad schematic (older format))
At the start: 0 parts

Commit message: Placed Tiva headers, took note of which pins were PWM
Parts:
- added U1: TM4C129E_Launchpad, symbol MRDT_Shields:TM4C129E_Launchpad
Other:
- note added: "PWM Pins are:\nPF_1, PF_2, PF_3, PF_0\nPG_1, PK_4, PK_5"
Changed lines of the file:
@@
 Comment4 ""
 $EndDescr
+$Comp
+L MRDT_Shields:TM4C129E_Launchpad U1
+U 1 1 5F715123
+P 4200 3200
+F 0 "U1" H 4300 4450 60  0000 L CNN
+F 1 "TM4C129E_Launchpad" H 3500 4350 60  0000 L CNN
+F 2 "" H 4200 3200 60  0001 C CNN
+F 3 "" H 4200 3200 60  0001 C CNN
+	1    4200 3200
+	1    0    0    -1
+$EndComp
+$Comp
+L MRDT_Shields:TM4C129E_Launchpad U1
+U 2 1 5F716DA0
+P 4800 3200
+F 0 "U1" H 5000 4450 60  0000 C CNN
+F 1 "TM4C129E_Launchpad" H 4600 4350 60  0000 C CNN
+F 2 "" H 4800 3200 60  0001 C CNN
+F 3 "" H 4800 3200 60  0001 C CNN
+	2    4800 3200
+	-1   0    0    -1
+$EndComp
+$Comp
+L MRDT_Shields:TM4C129E_Launchpad U1
+U 3 1 5F7264AA
+P 6350 3200
+F 0 "U1" H 6450 4450 60  0000 L CNN
+F 1 "TM4C129E_Launchpad" H 5700 4350 60  0000 L CNN
+F 2 "" H 6350 3200 60  0001 C CNN
+F 3 "" H 6350 3200 60  0001 C CNN
+	3    6350 3200
+	1    0    0    -1
+$EndComp
+$Comp
+L MRDT_Shields:TM4C129E_Launchpad U1
+U 4 1 5F72B226
+P 6950 3200
+F 0 "U1" H 7100 4450 60  0000 C CNN
+F 1 "TM4C129E_Launchpad" H 6700 4350 60  0000 C CNN
+F 2 "" H 6950 3200 60  0001 C CNN
+F 3 "" H 6950 3200 60  0001 C CNN
+	4    6950 3200
+	-1   0    0    -1
+$EndComp
+$Comp
+L MRDT_Shields:TM4C129E_Launchpad U1
+U 5 1 5F733DC7
+P 4200 4700
+F 0 "U1" H 4300 5950 60  0000 L CNN
+F 1 "TM4C129E_Launchpad" H 3500 5850 60  0000 L CNN
+F 2 "" H 4200 4700 60  0001 C CNN
+F 3 "" H 4200 4700 60  0001 C CNN
+	5    4200 4700
+	1    0    0    -1
+$EndComp
+$Comp
+L MRDT_Shields:TM4C129E_Launchpad U1
+U 6 1 5F73B2DD
+P 4800 4700
+F 0 "U1" H 5000 5950 60  0000 C CNN
+F 1 "TM4C129E_Launchpad" H 4600 5850 60  0000 C CNN
+F 2 "" H 4800 4700 60  0001 C CNN
+F 3 "" H 4800 4700 60  0001 C CNN
+	6    4800 4700
+	-1   0    0    -1
+$EndComp
+$Comp
+L MRDT_Shields:TM4C129E_Launchpad U1
+U 7 1 5F740CF4
+P 6350 4700
+F 0 "U1" H 6450 5950 60  0000 L CNN
+F 1 "TM4C129E_Launchpad" H 5650 5850 60  0000 L CNN
+F 2 "" H 6350 4700 60  0001 C CNN
+F 3 "" H 6350 4700 60  0001 C CNN
+	7    6350 4700
+	1    0    0    -1
+$EndComp
+$Comp
+L MRDT_Shields:TM4C129E_Launchpad U1
+U 8 1 5F7529E8
+P 6950 4700
+F 0 "U1" H 7100 5950 60  0000 C CNN
+F 1 "TM4C129E_Launchpad" H 6700 5850 60  0000 C CNN
+F 2 "" H 6950 4700 60  0001 C CNN
+F 3 "" H 6950 4700 60  0001 C CNN
+	8    6950 4700
+	-1   0    0    -1
+$EndComp
+Text Notes 8450 2450 0    79   ~ 0
+PWM Pins are:\nPF_1, PF_2, PF_3, PF_0\nPG_1, PK_4, PK_5
 $EndSCHEMATC
