File: Hardware/ScienceMotorController/ScienceMotorController02.sch (KiCad schematic (older format))
At the start: 5 parts, among them U1 TM4C129E_Launchpad

Commit message: cleaned up sheet names
Connections:
- net sheet5FA34ACC/Current_Sense_1 renamed Motor Driver 1/Current_Sense_1
- net sheet5FA34ACC/In_A_1 renamed Motor Driver 1/In_A_1
- net sheet5FA34ACC/In_B_1 renamed Motor Driver 1/In_B_1
- net sheet5FA34ACC/PWM_1 renamed Motor Driver 1/PWM_1
- net sheet5FA34ACD/Current_Sense_2 renamed Motor Driver 2/Current_Sense_2
- net sheet5FA34ACD/In_A_2 renamed Motor Driver 2/In_A_2
- net sheet5FA34ACD/In_B_2 renamed Motor Driver 2/In_B_2
- net sheet5FA34ACD/PWM_2 renamed Motor Driver 2/PWM_2
- net sheet5FA34ACE/Current_Sense_3 renamed Motor Driver 3/Current_Sense_3
- net sheet5FA34ACE/In_A_3 renamed Motor Driver 3/In_A_3
- net sheet5FA34ACE/In_B_3 renamed Motor Driver 3/In_B_3
- net sheet5FA34ACE/PWM_3 renamed Motor Driver 3/PWM_3
- net sheet5FA34ACF/Current_Sense_4 renamed Motor Driver 4/Current_Sense_4
- net sheet5FA34ACF/In_A_4 renamed Motor Driver 4/In_A_4
- net sheet5FA34ACF/In_B_4 renamed Motor Driver 4/In_B_4
- net sheet5FA34ACF/PWM_4 renamed Motor Driver 4/PWM_4
- net sheet5FA34AD0/Current_Sense_5 renamed Motor Driver 5/Current_Sense_5
- net sheet5FA34AD0/In_A_5 renamed Motor Driver 5/In_A_5
- net sheet5FA34AD0/In_B_5 renamed Motor Driver 5/In_B_5
- net sheet5FA34AD0/PWM_5 renamed Motor Driver 5/PWM_5
- net sheet5FA34AD1/Current_Sense_6 renamed Motor Driver 6/Current_Sense_6
- net sheet5FA34AD1/In_A_6 renamed Motor Driver 6/In_A_6
- net sheet5FA34AD1/In_B_6 renamed Motor Driver 6/In_B_6
- net sheet5FA34AD1/PWM_6 renamed Motor Driver 6/PWM_6
- net sheet5FC42AEB/Limit_Switch_1 renamed Limit Switches/Limit_Switch_1
- net sheet5FC42AEB/Limit_Switch_2 renamed Limit Switches/Limit_Switch_2
- net sheet5FC42AEB/Limit_Switch_3 renamed Limit Switches/Limit_Switch_3
- net sheet5FC42AEB/Limit_Switch_4 renamed Limit Switches/Limit_Switch_4
Other:
- moved on the sheet: U1D
Changed lines of the file:
@@
 $Descr A4 11693 8268
 encoding utf-8
-Sheet 3 11
+Sheet 3 10
 Title ""
 Date ""
@@
 L MRDT_Shields:TM4C129E_Launchpad U1
 U 4 1 5F72B226
-P 8350 3100
-F 0 "U1" H 8500 4500 60  0000 C CNN
-F 1 "TM4C129E_Launchpad" H 8100 4400 60  0000 C CNN
-F 2 "" H 8350 3100 60  0001 C CNN
-F 3 "" H 8350 3100 60  0001 C CNN
-	4    8350 3100
+P 8300 3050
+F 0 "U1" H 8450 4450 60  0000 C CNN
+F 1 "TM4C129E_Launchpad" H 8050 4350 60  0000 C CNN
+F 2 "" H 8300 3050 60  0001 C CNN
+F 3 "" H 8300 3050 60  0001 C CNN
+	4    8300 3050
 	-1   0    0    -1
 $EndComp
@@
 NoConn ~ 7500 2950
 NoConn ~ 7500 3050
-NoConn ~ 8550 3050
-NoConn ~ 8550 2950
-NoConn ~ 8550 2850
-NoConn ~ 8550 2750
-NoConn ~ 8550 2650
-NoConn ~ 8550 2550
-NoConn ~ 8550 2450
-NoConn ~ 8550 2350
-NoConn ~ 8550 2250
-Wire Wire Line
-	8550 2150 8800 2150
-Wire Wire Line
-	8800 2150 8800 2200
+NoConn ~ 8500 3000
+NoConn ~ 8500 2900
+NoConn ~ 8500 2800
+NoConn ~ 8500 2700
+NoConn ~ 8500 2600
+NoConn ~ 8500 2500
+NoConn ~ 8500 2400
+NoConn ~ 8500 2300
+NoConn ~ 8500 2200
+Wire Wire Line
+	8500 2100 8750 2100
+Wire Wire Line
+	8750 2100 8750 2150
 $Comp
 L power:GND #PWR?
 U 1 1 5F8D9D39
-P 8800 2200
-F 0 "#PWR?" H 8800 1950 50  0001 C CNN
-F 1 "GND" H 8900 2050 50  0000 R CNN
-F 2 "" H 8800 2200 50  0001 C CNN
-F 3 "" H 8800 2200 50  0001 C CNN
-	1    8800 2200
+P 8750 2150
+F 0 "#PWR?" H 8750 1900 50  0001 C CNN
+F 1 "GND" H 8850 2000 50  0000 R CNN
+F 2 "" H 8750 2150 50  0001 C CNN
+F 3 "" H 8750 2150 50  0001 C CNN
+	1    8750 2150
 	1    0    0    -1
 $EndComp
@@
 S 2800 2400 1350 650
 U 5FA34AD5
-F0 "sheet5FA34ACD" 39
+F0 "Motor Driver 2" 39
 F1 "ScienceMotorController03b.sch" 39
 F2 "In_A_2" I L 2800 2600 50
@@
 S 4550 2400 1450 650
 U 5FA34AD7
-F0 "sheet5FA34ACE" 39
+F0 "Motor Driver 3" 39
 F1 "ScienceMotorController03c.sch" 39
 F2 "In_A_3" I L 4550 2600 50
@@
 S 1100 4900 1400 450
 U 5FA34AD9
-F0 "sheet5FA34ACF" 39
+F0 "Motor Driver 4" 39
 F1 "ScienceMotorController03d.sch" 39
 F2 "In_A_4" I L 1100 5100 50
@@
 S 2800 4950 1450 400
 U 5FA34ADB
-F0 "sheet5FA34AD0" 39
+F0 "Motor Driver 5" 39
 F1 "ScienceMotorController03e.sch" 39
 F2 "In_B_5" I L 2800 5250 50
@@
 S 4900 4950 1400 400
 U 5FA34ADD
-F0 "sheet5FA34AD1" 39
+F0 "Motor Driver 6" 39
 F1 "ScienceMotorController03f.sch" 39
 F2 "In_B_6" I L 4900 5250 50
@@
 S 4700 850  800  900
 U 5FC42AEE
-F0 "sheet5FC42AEB" 50
+F0 "Limit Switches" 50
 F1 "ScienceMotorController04.sch" 50
 F2 "3.3VA" I L 4700 1050 50
@@
 S 1000 2400 1450 650
 U 5FA34AD3
-F0 "sheet5FA34ACC" 39
+F0 "Motor Driver 1" 39
 F1 "ScienceMotorController03a.sch" 39
 F2 "In_A_1" I L 1000 2600 50

Commit message: Fixed 3.3V, added encoders
Connections:
- net Absolute Encoders/Encoder_PWM_1: now reaches U1.PM1 (C2_5)
- net Absolute Encoders/Encoder_PWM_2: now reaches U1.PM2 (C2_6)
- no-connect marks 44 -> 42
Changed lines of the file:
@@
 $Descr A4 11693 8268
 encoding utf-8
-Sheet 3 10
+Sheet 3 11
 Title ""
 Date ""
@@
 NoConn ~ 7600 5300
 NoConn ~ 7600 5200
-NoConn ~ 7600 5100
-NoConn ~ 7600 5000
 NoConn ~ 7600 4900
 Wire Wire Line
@@
 F4 "PWM_2" I L 2800 2500 50
 F5 "Current_Sense_2" O R 4150 2950 50
+F6 "3.3VA" I L 2800 2900 50
 $EndSheet
 $Sheet
@@
 F4 "PWM_3" I L 4550 2500 50
 F5 "Current_Sense_3" O R 6000 2950 50
+F6 "3.3VA" I L 4550 2900 50
 $EndSheet
 $Sheet
@@
 F1 "ScienceMotorController03d.sch" 39
 F2 "In_A_4" I L 1100 5100 50
-F3 "In_B_4" I L 1100 5250 50
+F3 "In_B_4" I L 1100 5200 50
 F4 "PWM_4" I L 1100 5000 50
 F5 "Current_Sense_4" O R 2500 4950 50
+F6 "3.3VA" I L 1100 5300 50
 $EndSheet
 $Sheet
@@
 F0 "Motor Driver 5" 39
 F1 "ScienceMotorController03e.sch" 39
-F2 "In_B_5" I L 2800 5250 50
+F2 "In_B_5" I L 2800 5200 50
 F3 "In_A_5" I L 2800 5100 50
 F4 "PWM_5" I L 2800 5000 50
 F5 "Current_Sense_5" O R 4250 5000 50
+F6 "3.3VA" I L 2800 5300 50
 $EndSheet
 $Sheet
@@
 F0 "Motor Driver 6" 39
 F1 "ScienceMotorController03f.sch" 39
-F2 "In_B_6" I L 4900 5250 50
+F2 "In_B_6" I L 4900 5200 50
 F3 "In_A_6" I L 4900 5100 50
 F4 "PWM_6" I L 4900 5000 50
 F5 "Current_Sense_6" O R 6300 5000 50
+F6 "3.3VA" I L 4900 5300 50
 $EndSheet
 Wire Wire Line
@@
 	1000 3900 3000 3900
 Wire Wire Line
-	900  4000 900  5250
-Wire Wire Line
-	900  5250 1100 5250
+	900  4000 900  5200
 Wire Wire Line
 	900  4000 3000 4000
@@
 	4800 5100 4900 5100
 Wire Wire Line
-	4700 5250 4900 5250
-Wire Wire Line
 	900  2600 1000 2600
 Wire Wire Line
@@
 	1050 5000 1050 4600
 Wire Wire Line
-	2650 5250 2650 4200
-Wire Wire Line
-	2650 5250 2800 5250
-Wire Wire Line
 	2650 4200 3000 4200
 Wire Wire Line
@@
 	2950 4500 4700 4500
 Wire Wire Line
-	4700 4500 4700 5250
+	4700 4500 4700 5200
 Wire Wire Line
 	2900 4300 2900 4550
@@
 F4 "PWM_1" I L 1000 2500 50
 F5 "Current_Sense_1" O R 2450 2950 50
+F6 "3.3VA" I L 1000 2900 50
 $EndSheet
 Wire Wire Line
@@
 Wire Wire Line
 	3950 1550 4700 1550
+Text HLabel 900  2900 0    50   Input ~ 0
+3.3VA
+Wire Wire Line
+	900  2900 1000 2900
+Wire Wire Line
+	4900 5200 4700 5200
+Wire Wire Line
+	2800 5200 2650 5200
+Wire Wire Line
+	2650 5200 2650 4200
+Wire Wire Line
+	1100 5200 900  5200
+Text HLabel 2750 2900 0    50   Input ~ 0
+3.3VA
+Wire Wire Line
+	2750 2900 2800 2900
+Text HLabel 4500 2900 0    50   Input ~ 0
+3.3VA
+Wire Wire Line
+	4500 2900 4550 2900
+Text HLabel 950  5300 0    50   Input ~ 0
+3.3VA
+Wire Wire Line
+	950  5300 1100 5300
+Text HLabel 2750 5300 0    50   Input ~ 0
+3.3VA
+Wire Wire Line
+	2750 5300 2800 5300
+Text HLabel 4750 5300 0    50   Input ~ 0
+3.3VA
+Wire Wire Line
+	4750 5300 4900 5300
+$Sheet
+S 6600 4900 750  750
+U 5FA24F1F
+F0 "Absolute Encoders" 50
+F1 "ScienceMotorController05.sch" 50
+F2 "3.3VA" I L 6600 5550 50
+F3 "Encoder_PWM_1" O R 7350 5000 50
+F4 "Encoder_PWM_2" O R 7350 5100 50
+$EndSheet
+Text HLabel 6500 5550 0    50   Input ~ 0
+3.3VA
+Wire Wire Line
+	6600 5550 6500 5550
+Wire Wire Line
+	7350 5000 7600 5000
+Wire Wire Line
+	7350 5100 7600 5100
 $EndSCHEMATC

Commit message: added logic line
Connections:
- net 3.3VA renamed 3.3V
Changed lines of the file:
@@
 NoConn ~ 4000 3500
 Text HLabel 2700 650  0    50   Input ~ 0
-3.3VA
+3.3V
 Text HLabel 2750 3500 0    50   Input ~ 0
-3.3VA
+3.3V
 Wire Wire Line
 	2750 3500 3000 3500
@@
 F4 "PWM_2" I L 2800 2500 50
 F5 "Current_Sense_2" O R 4150 2950 50
-F6 "3.3VA" I L 2800 2900 50
+F6 "3.3V" I L 2800 2900 50
 $EndSheet
 $Sheet
@@
 F4 "PWM_3" I L 4550 2500 50
 F5 "Current_Sense_3" O R 6000 2950 50
-F6 "3.3VA" I L 4550 2900 50
+F6 "3.3V" I L 4550 2900 50
 $EndSheet
 $Sheet
@@
 F4 "PWM_4" I L 1100 5000 50
 F5 "Current_Sense_4" O R 2500 4950 50
-F6 "3.3VA" I L 1100 5300 50
+F6 "3.3V" I L 1100 5300 50
 $EndSheet
 $Sheet
@@
 F4 "PWM_5" I L 2800 5000 50
 F5 "Current_Sense_5" O R 4250 5000 50
-F6 "3.3VA" I L 2800 5300 50
+F6 "3.3V" I L 2800 5300 50
 $EndSheet
 $Sheet
@@
 F4 "PWM_6" I L 4900 5000 50
 F5 "Current_Sense_6" O R 6300 5000 50
-F6 "3.3VA" I L 4900 5300 50
+F6 "3.3V" I L 4900 5300 50
 $EndSheet
 Wire Wire Line
@@
 F0 "Limit Switches" 50
 F1 "ScienceMotorController04.sch" 50
-F2 "3.3VA" I L 4700 1050 50
+F2 "3.3V" I L 4700 1050 50
 F3 "Limit_Switch_1" O L 4700 1250 50
 F4 "Limit_Switch_2" O L 4700 1350 50
@@
 F4 "PWM_1" I L 1000 2500 50
 F5 "Current_Sense_1" O R 2450 2950 50
-F6 "3.3VA" I L 1000 2900 50
+F6 "3.3V" I L 1000 2900 50
 $EndSheet
 Wire Wire Line
@@
 	6050 2950 6050 3900
 Text HLabel 4550 1050 0    50   Input ~ 0
-3.3VA
+3.3V
 Wire Wire Line
 	4550 1050 4700 1050
@@
 	3950 1550 4700 1550
 Text HLabel 900  2900 0    50   Input ~ 0
-3.3VA
+3.3V
 Wire Wire Line
 	900  2900 1000 2900
@@
 	1100 5200 900  5200
 Text HLabel 2750 2900 0    50   Input ~ 0
-3.3VA
+3.3V
 Wire Wire Line
 	2750 2900 2800 2900
 Text HLabel 4500 2900 0    50   Input ~ 0
-3.3VA
+3.3V
 Wire Wire Line
 	4500 2900 4550 2900
 Text HLabel 950  5300 0    50   Input ~ 0
-3.3VA
+3.3V
 Wire Wire Line
 	950  5300 1100 5300
 Text HLabel 2750 5300 0    50   Input ~ 0
-3.3VA
+3.3V
 Wire Wire Line
 	2750 5300 2800 5300
 Text HLabel 4750 5300 0    50   Input ~ 0
-3.3VA
+3.3V
 Wire Wire Line
 	4750 5300 4900 5300
@@
 F0 "Absolute Encoders" 50
 F1 "ScienceMotorController05.sch" 50
-F2 "3.3VA" I L 6600 5550 50
+F2 "3.3V" I L 6600 5550 50
 F3 "Encoder_PWM_1" O R 7350 5000 50
 F4 "Encoder_PWM_2" O R 7350 5100 50
 $EndSheet
 Text HLabel 6500 5550 0    50   Input ~ 0
-3.3VA
+3.3V
 Wire Wire Line
 	6600 5550 6500 5550

Commit message: annotated
Parts:
- gave numbers to parts that had none: 4
- renumbered U1 to U2
Changed lines of the file:
@@
 $EndDescr
 $Comp
-L MRDT_Shields:TM4C129E_Launchpad U1
+L MRDT_Shields:TM4C129E_Launchpad U2
 U 1 1 5F715123
 P 3150 1600
-F 0 "U1" H 2150 2650 60  0000 L CNN
+F 0 "U2" H 2150 2650 60  0000 L CNN
 F 1 "TM4C129E_Launchpad" H 1350 2550 60  0000 L CNN
 F 2 "" H 3150 1600 60  0001 C CNN
@@
 $EndComp
 $Comp
-L MRDT_Shields:TM4C129E_Launchpad U1
+L MRDT_Shields:TM4C129E_Launchpad U2
 U 2 1 5F716DA0
 P 3750 1600
-F 0 "U1" H 3300 2700 60  0000 C CNN
+F 0 "U2" H 3300 2700 60  0000 C CNN
 F 1 "TM4C129E_Launchpad" H 2950 2600 60  0000 C CNN
 F 2 "" H 3750 1600 60  0001 C CNN
@@
 $EndComp
 $Comp
-L MRDT_Shields:TM4C129E_Launchpad U1
+L MRDT_Shields:TM4C129E_Launchpad U2
 U 3 1 5F7264AA
 P 7700 3050
-F 0 "U1" H 7800 4450 60  0000 L CNN
+F 0 "U2" H 7800 4450 60  0000 L CNN
 F 1 "TM4C129E_Launchpad" H 7050 4350 60  0000 L CNN
 F 2 "" H 7700 3050 60  0001 C CNN
@@
 $EndComp
 $Comp
-L MRDT_Shields:TM4C129E_Launchpad U1
+L MRDT_Shields:TM4C129E_Launchpad U2
 U 4 1 5F72B226
 P 8300 3050
-F 0 "U1" H 8450 4450 60  0000 C CNN
+F 0 "U2" H 8450 4450 60  0000 C CNN
 F 1 "TM4C129E_Launchpad" H 8050 4350 60  0000 C CNN
 F 2 "" H 8300 3050 60  0001 C CNN
@@
 $EndComp
 $Comp
-L MRDT_Shields:TM4C129E_Launchpad U1
+L MRDT_Shields:TM4C129E_Launchpad U2
 U 5 1 5F733DC7
 P 3200 4450
-F 0 "U1" H 2750 5250 60  0000 L CNN
+F 0 "U2" H 2750 5250 60  0000 L CNN
 F 1 "TM4C129E_Launchpad" H 1950 5150 60  0000 L CNN
 F 2 "" H 3200 4450 60  0001 C CNN
@@
 $EndComp
 $Comp
-L MRDT_Shields:TM4C129E_Launchpad U1
+L MRDT_Shields:TM4C129E_Launchpad U2
 U 6 1 5F73B2DD
 P 3800 4450
-F 0 "U1" H 3450 4600 60  0000 C CNN
+F 0 "U2" H 3450 4600 60  0000 C CNN
 F 1 "TM4C129E_Launchpad" H 3050 4500 60  0000 C CNN
 F 2 "" H 3800 4450 60  0001 C CNN
@@
 $EndComp
 $Comp
-L MRDT_Shields:TM4C129E_Launchpad U1
+L MRDT_Shields:TM4C129E_Launchpad U2
 U 7 1 5F740CF4
 P 7800 5550
-F 0 "U1" H 7900 6900 60  0000 L CNN
+F 0 "U2" H 7900 6900 60  0000 L CNN
 F 1 "TM4C129E_Launchpad" H 7100 6800 60  0000 L CNN
 F 2 "" H 7800 5550 60  0001 C CNN
@@
 $EndComp
 $Comp
-L MRDT_Shields:TM4C129E_Launchpad U1
+L MRDT_Shields:TM4C129E_Launchpad U2
 U 8 1 5F7529E8
 P 8400 5550
-F 0 "U1" H 8550 6900 60  0000 C CNN
+F 0 "U2" H 8550 6900 60  0000 C CNN
 F 1 "TM4C129E_Launchpad" H 8150 6800 60  0000 C CNN
 F 2 "" H 8400 5550 60  0001 C CNN
@@
 	8600 5500 8700 5500
 $Comp
-L Device:R R?
+L Device:R R5
 U 1 1 5F836CF2
 P 8850 5500
-F 0 "R?" V 8750 5500 50  0000 C CNN
+F 0 "R5" V 8750 5500 50  0000 C CNN
 F 1 "330" V 8850 5500 50  0000 C CNN
 F 2 "" V 8780 5500 50  0001 C CNN
@@
 $EndComp
 $Comp
-L Device:LED D?
+L Device:LED D6
 U 1 1 5F838880
 P 9250 5500
-F 0 "D?" H 9250 5600 50  0000 C CNN
+F 0 "D6" H 9250 5600 50  0000 C CNN
 F 1 "Yellow" H 9050 5550 50  0000 C CNN
 F 2 "" H 9250 5500 50  0001 C CNN
@@
 	9000 5500 9100 5500
 $Comp
-L power:GND #PWR?
+L power:GND #PWR015
 U 1 1 5F83BC3E
 P 9750 5550
-F 0 "#PWR?" H 9750 5300 50  0001 C CNN
+F 0 "#PWR015" H 9750 5300 50  0001 C CNN
 F 1 "GND" H 10000 5500 50  0000 R CNN
 F 2 "" H 9750 5550 50  0001 C CNN
@@
 $EndComp
 $Comp
-L Device:R R?
+L Device:R R4
 U 1 1 5F83D1F8
 P 8850 5300
-F 0 "R?" V 8750 5300 50  0000 C CNN
+F 0 "R4" V 8750 5300 50  0000 C CNN
 F 1 "330" V 8850 5300 50  0000 C CNN
 F 2 "" V 8780 5300 50  0001 C CNN
@@
 $EndComp
 $Comp
-L Device:LED D?
+L Device:LED D5
 U 1 1 5F83D4EA
 P 9250 5300
-F 0 "D?" H 9250 5400 50  0000 C CNN
+F 0 "D5" H 9250 5400 50  0000 C CNN
 F 1 "Red" H 9100 5350 50  0000 C CNN
 F 2 "" H 9250 5300 50  0001 C CNN
@@
 $EndComp
 $Comp
-L power:GND #PWR?
+L power:GND #PWR014
 U 1 1 5F83E3D5
 P 9750 5350
-F 0 "#PWR?" H 9750 5100 50  0001 C CNN
+F 0 "#PWR014" H 9750 5100 50  0001 C CNN
 F 1 "GND" H 10000 5300 50  0000 R CNN
 F 2 "" H 9750 5350 50  0001 C CNN
@@
 	8800 4600 8800 4650
 $Comp
-L power:GND #PWR?
+L power:GND #PWR013
 U 1 1 5F8BF81D
 P 8800 4650
-F 0 "#PWR?" H 8800 4400 50  0001 C CNN
+F 0 "#PWR013" H 8800 4400 50  0001 C CNN
 F 1 "GND" H 9050 4600 50  0000 R CNN
 F 2 "" H 8800 4650 50  0001 C CNN
@@
 NoConn ~ 2950 850
 NoConn ~ 2950 750
-NoConn ~ 7500 2450
-NoConn ~ 7500 2550
-NoConn ~ 7500 2650
-NoConn ~ 7500 2750
-NoConn ~ 7500 2850
-NoConn ~ 7500 2950
-NoConn ~ 7500 3050
+NoConn ~ 7500 2400
+NoConn ~ 7500 2500
+NoConn ~ 7500 2600
+NoConn ~ 7500 2700
+NoConn ~ 7500 2800
+NoConn ~ 7500 2900
+NoConn ~ 7500 3000
 NoConn ~ 8500 3000
 NoConn ~ 8500 2900
@@
 	8750 2100 8750 2150
 $Comp
-L power:GND #PWR?
+L power:GND #PWR012
 U 1 1 5F8D9D39
 P 8750 2150
-F 0 "#PWR?" H 8750 1900 50  0001 C CNN
+F 0 "#PWR012" H 8750 1900 50  0001 C CNN
 F 1 "GND" H 8850 2000 50  0000 R CNN
 F 2 "" H 8750 2150 50  0001 C CNN
@@
 	4200 750  4200 800
 $Comp
-L power:GND #PWR?
+L power:GND #PWR010
 U 1 1 5F8DBCE3
 P 4200 800
-F 0 "#PWR?" H 4200 550 50  0001 C CNN
+F 0 "#PWR010" H 4200 550 50  0001 C CNN
 F 1 "GND" H 4300 650 50  0000 R CNN
 F 2 "" H 4200 800 50  0001 C CNN
@@
 	4550 3600 4550 3650
 $Comp
-L power:GND #PWR?
+L power:GND #PWR011
 U 1 1 5FC2B1A7
 P 4550 3650
-F 0 "#PWR?" H 4550 3400 50  0001 C CNN
+F 0 "#PWR011" H 4550 3400 50  0001 C CNN
 F 1 "GND" H 4555 3477 50  0000 C CNN
 F 2 "" H 4550 3650 50  0001 C CNN

Commit message: assigned most of the footprints
Parts:
- D5: value Red -> LED; footprint (none) -> LED_SMD:LED_0603_1608Metric_Pad1.05x0.95mm_HandSolder
- D6: value Yellow -> LED; footprint (none) -> LED_SMD:LED_0603_1608Metric_Pad1.05x0.95mm_HandSolder
- R4, R5: footprint (none) -> Resistor_SMD:R_0603_1608Metric_Pad1.05x0.95mm_HandSolder
- U2: footprint (none) -> MRDT_Shields:TM4C129E_Launchpad_FULL_SMD_TOP
Changed lines of the file:
@@
 F 0 "U2" H 2150 2650 60  0000 L CNN
 F 1 "TM4C129E_Launchpad" H 1350 2550 60  0000 L CNN
-F 2 "" H 3150 1600 60  0001 C CNN
+F 2 "MRDT_Shields:TM4C129E_Launchpad_FULL_SMD_TOP" H 3150 1600 60  0001 C CNN
 F 3 "" H 3150 1600 60  0001 C CNN
 	1    3150 1600
@@
 F 0 "U2" H 3300 2700 60  0000 C CNN
 F 1 "TM4C129E_Launchpad" H 2950 2600 60  0000 C CNN
-F 2 "" H 3750 1600 60  0001 C CNN
+F 2 "MRDT_Shields:TM4C129E_Launchpad_FULL_SMD_TOP" H 3750 1600 60  0001 C CNN
 F 3 "" H 3750 1600 60  0001 C CNN
 	2    3750 1600
@@
 F 0 "U2" H 7800 4450 60  0000 L CNN
 F 1 "TM4C129E_Launchpad" H 7050 4350 60  0000 L CNN
-F 2 "" H 7700 3050 60  0001 C CNN
+F 2 "MRDT_Shields:TM4C129E_Launchpad_FULL_SMD_TOP" H 7700 3050 60  0001 C CNN
 F 3 "" H 7700 3050 60  0001 C CNN
 	3    7700 3050
@@
 F 0 "U2" H 8450 4450 60  0000 C CNN
 F 1 "TM4C129E_Launchpad" H 8050 4350 60  0000 C CNN
-F 2 "" H 8300 3050 60  0001 C CNN
+F 2 "MRDT_Shields:TM4C129E_Launchpad_FULL_SMD_TOP" H 8300 3050 60  0001 C CNN
 F 3 "" H 8300 3050 60  0001 C CNN
 	4    8300 3050
@@
 F 0 "U2" H 2750 5250 60  0000 L CNN
 F 1 "TM4C129E_Launchpad" H 1950 5150 60  0000 L CNN
-F 2 "" H 3200 4450 60  0001 C CNN
+F 2 "MRDT_Shields:TM4C129E_Launchpad_FULL_SMD_TOP" H 3200 4450 60  0001 C CNN
 F 3 "" H 3200 4450 60  0001 C CNN
 	5    3200 4450
@@
 F 0 "U2" H 3450 4600 60  0000 C CNN
 F 1 "TM4C129E_Launchpad" H 3050 4500 60  0000 C CNN
-F 2 "" H 3800 4450 60  0001 C CNN
+F 2 "MRDT_Shields:TM4C129E_Launchpad_FULL_SMD_TOP" H 3800 4450 60  0001 C CNN
 F 3 "" H 3800 4450 60  0001 C CNN
 	6    3800 4450
@@
 F 0 "U2" H 7900 6900 60  0000 L CNN
 F 1 "TM4C129E_Launchpad" H 7100 6800 60  0000 L CNN
-F 2 "" H 7800 5550 60  0001 C CNN
+F 2 "MRDT_Shields:TM4C129E_Launchpad_FULL_SMD_TOP" H 7800 5550 60  0001 C CNN
 F 3 "" H 7800 5550 60  0001 C CNN
 	7    7800 5550
@@
 F 0 "U2" H 8550 6900 60  0000 C CNN
 F 1 "TM4C129E_Launchpad" H 8150 6800 60  0000 C CNN
-F 2 "" H 8400 5550 60  0001 C CNN
+F 2 "MRDT_Shields:TM4C129E_Launchpad_FULL_SMD_TOP" H 8400 5550 60  0001 C CNN
 F 3 "" H 8400 5550 60  0001 C CNN
 	8    8400 5550
@@
 F 0 "R5" V 8750 5500 50  0000 C CNN
 F 1 "330" V 8850 5500 50  0000 C CNN
-F 2 "" V 8780 5500 50  0001 C CNN
+F 2 "Resistor_SMD:R_0603_1608Metric_Pad1.05x0.95mm_HandSolder" V 8780 5500 50  0001 C CNN
 F 3 "~" H 8850 5500 50  0001 C CNN
 	1    8850 5500
@@
 P 9250 5500
 F 0 "D6" H 9250 5600 50  0000 C CNN
-F 1 "Yellow" H 9050 5550 50  0000 C CNN
-F 2 "" H 9250 5500 50  0001 C CNN
+F 1 "LED" H 9050 5550 50  0000 C CNN
+F 2 "LED_SMD:LED_0603_1608Metric_Pad1.05x0.95mm_HandSolder" H 9250 5500 50  0001 C CNN
 F 3 "~" H 9250 5500 50  0001 C CNN
 	1    9250 5500
@@
 F 0 "R4" V 8750 5300 50  0000 C CNN
 F 1 "330" V 8850 5300 50  0000 C CNN
-F 2 "" V 8780 5300 50  0001 C CNN
+F 2 "Resistor_SMD:R_0603_1608Metric_Pad1.05x0.95mm_HandSolder" V 8780 5300 50  0001 C CNN
 F 3 "~" H 8850 5300 50  0001 C CNN
 	1    8850 5300
@@
 P 9250 5300
 F 0 "D5" H 9250 5400 50  0000 C CNN
-F 1 "Red" H 9100 5350 50  0000 C CNN
-F 2 "" H 9250 5300 50  0001 C CNN
+F 1 "LED" H 9100 5350 50  0000 C CNN
+F 2 "LED_SMD:LED_0603_1608Metric_Pad1.05x0.95mm_HandSolder" H 9250 5300 50  0001 C CNN
 F 3 "~" H 9250 5300 50  0001 C CNN
 	1    9250 5300

Commit message: began placing footprints on layout
Parts:
- U2: footprint MRDT_Shields:TM4C129E_Launchpad_FULL_SMD_TOP -> MRDT_Shields:TM4C129E_Launchpad_FULL_THT_TOP
Changed lines of the file:
@@
 F 0 "U2" H 2150 2650 60  0000 L CNN
 F 1 "TM4C129E_Launchpad" H 1350 2550 60  0000 L CNN
-F 2 "MRDT_Shields:TM4C129E_Launchpad_FULL_SMD_TOP" H 3150 1600 60  0001 C CNN
+F 2 "MRDT_Shields:TM4C129E_Launchpad_FULL_THT_TOP" H 3150 1600 60  0001 C CNN
 F 3 "" H 3150 1600 60  0001 C CNN
 	1    3150 1600
@@
 F 0 "U2" H 3300 2700 60  0000 C CNN
 F 1 "TM4C129E_Launchpad" H 2950 2600 60  0000 C CNN
-F 2 "MRDT_Shields:TM4C129E_Launchpad_FULL_SMD_TOP" H 3750 1600 60  0001 C CNN
+F 2 "MRDT_Shields:TM4C129E_Launchpad_FULL_THT_TOP" H 3750 1600 60  0001 C CNN
 F 3 "" H 3750 1600 60  0001 C CNN
 	2    3750 1600
@@
 F 0 "U2" H 7800 4450 60  0000 L CNN
 F 1 "TM4C129E_Launchpad" H 7050 4350 60  0000 L CNN
-F 2 "MRDT_Shields:TM4C129E_Launchpad_FULL_SMD_TOP" H 7700 3050 60  0001 C CNN
+F 2 "MRDT_Shields:TM4C129E_Launchpad_FULL_THT_TOP" H 7700 3050 60  0001 C CNN
 F 3 "" H 7700 3050 60  0001 C CNN
 	3    7700 3050
@@
 F 0 "U2" H 8450 4450 60  0000 C CNN
 F 1 "TM4C129E_Launchpad" H 8050 4350 60  0000 C CNN
-F 2 "MRDT_Shields:TM4C129E_Launchpad_FULL_SMD_TOP" H 8300 3050 60  0001 C CNN
+F 2 "MRDT_Shields:TM4C129E_Launchpad_FULL_THT_TOP" H 8300 3050 60  0001 C CNN
 F 3 "" H 8300 3050 60  0001 C CNN
 	4    8300 3050
@@
 F 0 "U2" H 2750 5250 60  0000 L CNN
 F 1 "TM4C129E_Launchpad" H 1950 5150 60  0000 L CNN
-F 2 "MRDT_Shields:TM4C129E_Launchpad_FULL_SMD_TOP" H 3200 4450 60  0001 C CNN
+F 2 "MRDT_Shields:TM4C129E_Launchpad_FULL_THT_TOP" H 3200 4450 60  0001 C CNN
 F 3 "" H 3200 4450 60  0001 C CNN
 	5    3200 4450
@@
 F 0 "U2" H 3450 4600 60  0000 C CNN
 F 1 "TM4C129E_Launchpad" H 3050 4500 60  0000 C CNN
-F 2 "MRDT_Shields:TM4C129E_Launchpad_FULL_SMD_TOP" H 3800 4450 60  0001 C CNN
+F 2 "MRDT_Shields:TM4C129E_Launchpad_FULL_THT_TOP" H 3800 4450 60  0001 C CNN
 F 3 "" H 3800 4450 60  0001 C CNN
 	6    3800 4450
@@
 F 0 "U2" H 7900 6900 60  0000 L CNN
 F 1 "TM4C129E_Launchpad" H 7100 6800 60  0000 L CNN
-F 2 "MRDT_Shields:TM4C129E_Launchpad_FULL_SMD_TOP" H 7800 5550 60  0001 C CNN
+F 2 "MRDT_Shields:TM4C129E_Launchpad_FULL_THT_TOP" H 7800 5550 60  0001 C CNN
 F 3 "" H 7800 5550 60  0001 C CNN
 	7    7800 5550
@@
 F 0 "U2" H 8550 6900 60  0000 C CNN
 F 1 "TM4C129E_Launchpad" H 8150 6800 60  0000 C CNN
-F 2 "MRDT_Shields:TM4C129E_Launchpad_FULL_SMD_TOP" H 8400 5550 60  0001 C CNN
+F 2 "MRDT_Shields:TM4C129E_Launchpad_FULL_THT_TOP" H 8400 5550 60  0001 C CNN
 F 3 "" H 8400 5550 60  0001 C CNN
 	8    8400 5550
