File: Hardware/ScienceMotorController/ScienceMotorController.sch (KiCad schematic (older format))
At the start: 5 parts

Commit message: assigned most of the footprints
Parts:
- Conn1: footprint (none) -> MRDT_Connectors:Anderson_3_Vertical_Side_by_Side
- D1, D2: footprint (none) -> LED_SMD:LED_0603_1608Metric_Pad1.05x0.95mm_HandSolder
- R1, R2: footprint (none) -> Resistor_SMD:R_0603_1608Metric_Pad1.05x0.95mm_HandSolder
Changed lines of the file:
@@
 F 0 "Conn1" H 2708 4187 60  0000 C CNN
 F 1 "AndersonPP" H 2708 4081 60  0000 C CNN
-F 2 "" H 2350 3250 60  0001 C CNN
+F 2 "MRDT_Connectors:Anderson_3_Vertical_Side_by_Side" H 2350 3250 60  0001 C CNN
 F 3 "" H 2350 3250 60  0001 C CNN
 	3    2500 3800
@@
 F 0 "D1" H 3550 3600 50  0000 C CNN
 F 1 "LED" H 3550 3700 50  0000 C CNN
-F 2 "" H 3550 3800 50  0001 C CNN
+F 2 "LED_SMD:LED_0603_1608Metric_Pad1.05x0.95mm_HandSolder" H 3550 3800 50  0001 C CNN
 F 3 "~" H 3550 3800 50  0001 C CNN
 	1    3550 3800
@@
 F 0 "R1" V 2954 3800 50  0000 C CNN
 F 1 "1.2k" V 3150 3800 39  0000 C CNN
-F 2 "" H 3150 3800 50  0001 C CNN
+F 2 "Resistor_SMD:R_0603_1608Metric_Pad1.05x0.95mm_HandSolder" H 3150 3800 50  0001 C CNN
 F 3 "~" H 3150 3800 50  0001 C CNN
 	1    3150 3800
@@
 F 0 "Conn1" H 2708 5337 60  0000 C CNN
 F 1 "AndersonPP" H 2708 5231 60  0000 C CNN
-F 2 "" H 2350 4400 60  0001 C CNN
+F 2 "MRDT_Connectors:Anderson_3_Vertical_Side_by_Side" H 2350 4400 60  0001 C CNN
 F 3 "" H 2350 4400 60  0001 C CNN
 	1    2500 4950
@@
 F 0 "Conn1" H 2708 4737 60  0000 C CNN
 F 1 "AndersonPP" H 2708 4631 60  0000 C CNN
-F 2 "" H 2350 3800 60  0001 C CNN
+F 2 "MRDT_Connectors:Anderson_3_Vertical_Side_by_Side" H 2350 3800 60  0001 C CNN
 F 3 "" H 2350 3800 60  0001 C CNN
 	2    2500 4350
@@
 F 0 "R2" V 3200 4450 50  0000 C CNN
 F 1 "1.2k" V 3300 4450 39  0000 C CNN
-F 2 "" H 3300 4450 50  0001 C CNN
+F 2 "Resistor_SMD:R_0603_1608Metric_Pad1.05x0.95mm_HandSolder" H 3300 4450 50  0001 C CNN
 F 3 "~" H 3300 4450 50  0001 C CNN
 	1    3300 4450
@@
 F 0 "D2" H 3700 4400 50  0000 C CNN
 F 1 "LED" H 3600 4350 50  0000 C CNN
-F 2 "" H 3600 4450 50  0001 C CNN
+F 2 "LED_SMD:LED_0603_1608Metric_Pad1.05x0.95mm_HandSolder" H 3600 4450 50  0001 C CNN
 F 3 "~" H 3600 4450 50  0001 C CNN
 	1    3600 4450
