File: Hardware/ScienceMotorController/ScienceMotorController.sch (KiCad schematic (older format))
At the start: 127 parts, among them U1 LT1910, U10 OKI, U11 OKI, U12 TB67H400AFNG,EL, U13 TB67H400AFNG,EL, U14 LT1910, U15 PMN280ENEAX, U16 PMN280ENEAX, U17 LTC6900, U2 OKI, U3 TB67H400AFNG,EL, U4 TB67H400AFNG,EL, U5 TB67H400AFNG,EL, U6 TB67H400AFNG,EL, U7 LT1910, U8 PMN280ENEAX, U9 TM4C129E_Launchpad

Commit message: Edge cuts, GND plane, a little more organized
Parts:
- U15, U16, U8: symbol SciMoCoLib:PMN280ENEAX -> ScienceMotorController-rescue:PMN280ENEAX-SciMoCoLib
- U17: symbol SciMoCoLib:LTC6900 -> ScienceMotorController-rescue:LTC6900-SciMoCoLib
Changed lines of the file:
@@
 EESchema Schematic File Version 4
-EELAYER 30 0
+LIBS:ScienceMotorController-cache
+EELAYER 26 0
 EELAYER END
 $Descr C 22000 17000
@@
 	3600 10450 3600 10550
 $Comp
-L SciMoCoLib:PMN280ENEAX U8
+L ScienceMotorController-rescue:PMN280ENEAX-SciMoCoLib U8
 U 1 1 64F13429
 P 5100 14050
@@
 	5350 14150 5450 14150
 $Comp
-L SciMoCoLib:PMN280ENEAX U15
+L ScienceMotorController-rescue:PMN280ENEAX-SciMoCoLib U15
 U 1 1 65651C73
 P 9250 14000
@@
 Connection ~ 8950 13800
 $Comp
-L SciMoCoLib:PMN280ENEAX U16
+L ScienceMotorController-rescue:PMN280ENEAX-SciMoCoLib U16
 U 1 1 656CCAC6
 P 13350 13950
@@
 $EndComp
 $Comp
-L SciMoCoLib:LTC6900 U17
+L ScienceMotorController-rescue:LTC6900-SciMoCoLib U17
 U 1 1 65A4B48D
 P 16800 12650

Commit message: Worked on patterns for SolValve, LimSwitch, OKIs, and Clock for PCB
Parts:
- renumbered Conn14 to AbsEncode1, Conn15 to AbsEncode2, Conn16 to AbsEncode3, Conn17 to AbsEncode4, Conn18 to AbsEncode5, Conn19 to LimSwitch1, Conn20 to LimSwitch2, Conn9 to Servo1, Conn10 to Servo2, Conn11 to SolValve1, Conn12 to SolValve2, Conn13 to SolValve3
Other:
- note added: "2 are spares"
- note added: "Pump 3"
- note added: "Z-AXIS"
- note removed: "Drill\n"
- note removed: "Spare"
Changed lines of the file:
@@
 EESchema Schematic File Version 4
-LIBS:ScienceMotorController-cache
-EELAYER 26 0
+EELAYER 30 0
 EELAYER END
 $Descr C 22000 17000
@@
 	11100 11900 11550 11900
 $Comp
-L MRDT_Connectors:Molex_SL_03 Conn14
+L MRDT_Connectors:Molex_SL_03 AbsEncode1
 U 1 1 64D7FBFC
 P 16900 10150
-F 0 "Conn14" H 17027 10358 60  0000 L CNN
+F 0 "AbsEncode1" H 17027 10358 60  0000 L CNN
 F 1 "Molex_SL_03" H 17027 10252 60  0000 L CNN
 F 2 "MRDT_Connectors:MOLEX_SL_03_Vertical" H 16900 10150 60  0001 C CNN
@@
 	9950 11900 10100 11900
 $Comp
-L MRDT_Connectors:Molex_SL_03 Conn15
+L MRDT_Connectors:Molex_SL_03 AbsEncode2
 U 1 1 655831B5
 P 16900 10800
-F 0 "Conn15" H 17027 11008 60  0000 L CNN
+F 0 "AbsEncode2" H 17027 11008 60  0000 L CNN
 F 1 "Molex_SL_03" H 17027 10902 60  0000 L CNN
 F 2 "MRDT_Connectors:MOLEX_SL_03_Vertical" H 16900 10800 60  0001 C CNN
@@
 $EndComp
 $Comp
-L MRDT_Connectors:Molex_SL_03 Conn16
+L MRDT_Connectors:Molex_SL_03 AbsEncode3
 U 1 1 655EA6BC
 P 16900 11450
-F 0 "Conn16" H 17027 11658 60  0000 L CNN
+F 0 "AbsEncode3" H 17027 11658 60  0000 L CNN
 F 1 "Molex_SL_03" H 17027 11552 60  0000 L CNN
 F 2 "MRDT_Connectors:MOLEX_SL_03_Vertical" H 16900 11450 60  0001 C CNN
@@
 	11100 12400 11300 12400
 $Comp
-L MRDT_Connectors:Molex_SL_02 Conn19
+L MRDT_Connectors:Molex_SL_02 LimSwitch1
 U 1 1 66E6B4BD
 P 14350 10000
-F 0 "Conn19" H 14477 10158 60  0000 L CNN
+F 0 "LimSwitch1" H 14477 10158 60  0000 L CNN
 F 1 "Molex_SL_02" H 14477 10052 60  0000 L CNN
 F 2 "MRDT_Connectors:MOLEX_SL_02_Vertical" H 14350 9900 60  0001 C CNN
@@
 Connection ~ 14100 9950
 $Comp
-L MRDT_Connectors:Molex_SL_02 Conn20
+L MRDT_Connectors:Molex_SL_02 LimSwitch2
 U 1 1 6717C8FC
 P 14350 10850
-F 0 "Conn20" H 14477 11008 60  0000 L CNN
+F 0 "LimSwitch2" H 14477 11008 60  0000 L CNN
 F 1 "Molex_SL_02" H 14477 10902 60  0000 L CNN
 F 2 "MRDT_Connectors:MOLEX_SL_02_Vertical" H 14350 10750 60  0001 C CNN
@@
 $EndComp
 $Comp
-L MRDT_Connectors:Molex_SL_03 Conn9
+L MRDT_Connectors:Molex_SL_03 Servo1
 U 1 1 63690AD9
 P 13950 12400
-F 0 "Conn9" H 14077 12608 60  0000 L CNN
+F 0 "Servo1" H 14077 12608 60  0000 L CNN
 F 1 "Molex_SL_03" H 14077 12502 60  0000 L CNN
 F 2 "MRDT_Connectors:MOLEX_SL_03_Vertical" H 13950 12400 60  0001 C CNN
@@
 $EndComp
 $Comp
-L MRDT_Connectors:Molex_SL_03 Conn10
+L MRDT_Connectors:Molex_SL_03 Servo2
 U 1 1 63690AE0
 P 13950 13050
-F 0 "Conn10" H 14077 13258 60  0000 L CNN
+F 0 "Servo2" H 14077 13258 60  0000 L CNN
 F 1 "Molex_SL_03" H 14077 13152 60  0000 L CNN
 F 2 "MRDT_Connectors:MOLEX_SL_03_Vertical" H 13950 13050 60  0001 C CNN
@@
 Blue\n
 $Comp
-L MRDT_Connectors:Molex_SL_03 Conn17
+L MRDT_Connectors:Molex_SL_03 AbsEncode4
 U 1 1 61DF14A8
 P 18650 10150
-F 0 "Conn17" H 18777 10358 60  0000 L CNN
+F 0 "AbsEncode4" H 18777 10358 60  0000 L CNN
 F 1 "Molex_SL_03" H 18777 10252 60  0000 L CNN
 F 2 "MRDT_Connectors:MOLEX_SL_03_Vertical" H 18650 10150 60  0001 C CNN
@@
 $EndComp
 $Comp
-L MRDT_Connectors:Molex_SL_03 Conn18
+L MRDT_Connectors:Molex_SL_03 AbsEncode5
 U 1 1 61DF14AF
 P 18700 10800
-F 0 "Conn18" H 18827 11008 60  0000 L CNN
+F 0 "AbsEncode5" H 18827 11008 60  0000 L CNN
 F 1 "Molex_SL_03" H 18827 10902 60  0000 L CNN
 F 2 "MRDT_Connectors:MOLEX_SL_03_Vertical" H 18700 10800 60  0001 C CNN
@@
 Wire Notes Line width 8 style solid
 	10300 2000 10300 2350
-Text Notes 16500 2300 0    197  ~ 0
-Drill\n
+Text Notes 16450 2300 0    197  ~ 0
+Z-AXIS
 Wire Notes Line width 8 style solid
 	16450 2350 17200 2350
 Wire Notes Line width 8 style solid
-	17200 2350 17200 2000
+	17600 2350 17600 2000
 Wire Notes Line width 8 style solid
 	17200 2000 16450 2000
@@
 Wire Notes Line width 8 style solid
 	10250 9050 10250 9400
-Text Notes 16500 9450 0    157  ~ 0
-Spare
+Text Notes 16450 9450 0    197  ~ 0
+Pump 3
 Wire Notes Line width 8 style solid
-	16450 9500 17200 9500
-Wire Notes Line width 8 style solid
-	17200 9500 17200 9200
-Wire Notes Line width 8 style solid
-	17200 9200 16450 9200
+	17700 9500 17700 9200
 Wire Notes Line width 8 style solid
 	16450 9200 16450 9500
@@
 Does this need analogWrite() or can\nit just be connected to a "green" pin?
 $Comp
-L MRDT_Connectors:Molex_SL_02 Conn11
+L MRDT_Connectors:Molex_SL_02 SolValve1
 U 1 1 69094A05
 P 5750 14300
-F 0 "Conn11" H 5877 14458 60  0000 L CNN
+F 0 "SolValve1" H 5877 14458 60  0000 L CNN
 F 1 "Molex_SL_02" H 5877 14352 60  0000 L CNN
 F 2 "MRDT_Connectors:MOLEX_SL_02_Vertical" H 5750 14200 60  0001 C CNN
@@
 	4600 14750 4600 14800
 $Comp
-L MRDT_Connectors:Molex_SL_02 Conn12
+L MRDT_Connectors:Molex_SL_02 SolValve2
 U 1 1 6975F8A5
 P 9900 14250
-F 0 "Conn12" H 10027 14408 60  0000 L CNN
+F 0 "SolValve2" H 10027 14408 60  0000 L CNN
 F 1 "Molex_SL_02" H 10027 14302 60  0000 L CNN
 F 2 "MRDT_Connectors:MOLEX_SL_02_Vertical" H 9900 14150 60  0001 C CNN
@@
 	8750 14700 8750 14750
 $Comp
-L MRDT_Connectors:Molex_SL_02 Conn13
+L MRDT_Connectors:Molex_SL_02 SolValve3
 U 1 1 697E6C27
 P 14000 14200
-F 0 "Conn13" H 14127 14358 60  0000 L CNN
+F 0 "SolValve3" H 14127 14358 60  0000 L CNN
 F 1 "Molex_SL_02" H 14127 14252 60  0000 L CNN
 F 2 "MRDT_Connectors:MOLEX_SL_02_Vertical" H 14000 14100 60  0001 C CNN
@@
 	1    0    0    -1
 $EndComp
+Text Notes 20050 10650 0    157  ~ 0
+2 are spares
+Wire Notes Line width 8 style solid
+	16450 9500 17700 9500
+Wire Notes Line width 8 style solid
+	16450 9200 17700 9200
+Wire Notes Line width 8 style solid
+	17200 2000 17600 2000
+Wire Notes Line width 8 style solid
+	17600 2350 17200 2350
 $EndSCHEMATC

Commit message: Added 4 More Limit Switches
Parts:
- added D? (x4): LED, LED_SMD:LED_0603_1608Metric_Pad1.05x0.95mm_HandSolder, symbol Device:LED_Small
- added LimSwitch3, LimSwitch4, LimSwitch5, LimSwitch6: Molex_SL_02, MRDT_Connectors:MOLEX_SL_02_Vertical, symbol MRDT_Connectors:Molex_SL_02
- added R? (x4): 43, Resistor_SMD:R_0603_1608Metric_Pad1.05x0.95mm_HandSolder, symbol Device:R
Connections:
- net +3V3: now also LimSwitch3.1, LimSwitch4.1, LimSwitch5.1, LimSwitch6.1
- net GND: now also D?.1 (K), D?.1 (K), D?.1 (K), D?.1 (K)
- net InA1_1: now also U9.PE2 (B1_5); no longer U9.PC4 (A1_3)
- net InA1_2: now also U9.PF1 (C1_1); no longer U9.PC6 (A1_5)
- net InA1_3: now also U9.PF3 (C1_3); no longer U9.PF1 (C1_1)
- net InA1_4: now also U9.PL0 (C1_7); no longer U9.PF3 (C1_3)
- net InA1_5: now also U9.PH0 (C2_7); no longer U9.PQ0 (A2_7)
- net InA1_6: now also U9.PK6 (C2_9); no longer U9.PN5 (A2_9)
- net InA2_1: now also U9.PE3 (B1_6); no longer U9.PC5 (A1_4)
- net InA2_2: now also U9.PF2 (C1_2); no longer U9.PE5 (A1_6)
- net InA2_3: now also U9.PG0 (C1_4); no longer U9.PF2 (C1_2)
- net InA2_4: now also U9.PL1 (C1_8); no longer U9.PG0 (C1_4)
- net InA2_5: now also U9.PH1 (C2_8); no longer U9.PP4 (A2_8)
- net InA2_6: now also U9.PK7 (C2_10); no longer U9.PN4 (A2_10)
- net Limit_Switch_1: now also U9.PE4 (A1_2); no longer U9.PL0 (C1_7)
- net Limit_Switch_2: now also U9.PC4 (A1_3); no longer U9.PL1 (C1_8)
- net PWMA_2: now also U9.PL4 (C1_5); no longer U9.PA6 (B1_8)
- net PWMA_3: now also U9.PL5 (C1_6); no longer U9.PM4 (B1_9)
- net PWMA_4: now also U9.PD1 (D1_6); no longer U9.PM5 (B1_10)
- net Solenoid_Valve_1: now also U9.PP4 (A2_8); no longer U9.PH1 (C2_8)
- net Solenoid_Valve_2: now also U9.PN5 (A2_9); no longer U9.PK6 (C2_9)
- net Solenoid_Valve_3: now also U9.PN4 (A2_10); no longer U9.PK7 (C2_10)
- net Limit_Switch_6: now reaches U9.PC7 (A1_8)
- net Limit_Switch_6: now also LimSwitch6.2, R?.2
- new net: D?.2 (A), R?.1 (x4)
- new net Limit_Switch_3: LimSwitch3.2, R?.2, U9.PC5 (A1_4)
- new net Limit_Switch_4: LimSwitch4.2, R?.2, U9.PC6 (A1_5)
- new net Limit_Switch_5: LimSwitch5.2, R?.2, U9.PE5 (A1_6)
- no-connect marks 85 -> 81

Commit message: Reassigned Encoder Pins
Parts:
- gave numbers to parts that had none: 8
Connections:
- net Encoder_PWM_1: now also U9.PD2 (A2_2); no longer U9.PG1 (C2_1)
- net Encoder_PWM_2: now also U9.PD4 (A2_5); no longer U9.PK4 (C2_2)
- net Encoder_PWM_3: now also U9.PD5 (A2_6); no longer U9.PK5 (C2_3)
- net Encoder_PWM_4: now also U9.PA4 (B2_9); no longer U9.PD2 (A2_2)
- net Encoder_PWM_5: now also U9.PA5 (B2_10); no longer U9.PP0 (A2_3)
Changed lines of the file:
@@
 NoConn ~ 7450 12200
 NoConn ~ 8450 11900
-NoConn ~ 8450 12700
-NoConn ~ 8450 12800
 Wire Wire Line
 	8450 12000 8700 12000
@@
 Text Notes 9200 10650 0    276  ~ 0
 TIVA
-Text GLabel 9950 11900 0    35   Input ~ 0
-Encoder_PWM_1
-Text GLabel 9950 12000 0    35   Input ~ 0
-Encoder_PWM_2
-Text GLabel 9950 12100 0    35   Input ~ 0
-Encoder_PWM_3
 Wire Wire Line
 	9950 12100 10100 12100
@@
 NoConn ~ 11950 10900
 NoConn ~ 11950 11000
-NoConn ~ 7450 12300
-NoConn ~ 7450 12400
 NoConn ~ 8450 12100
 NoConn ~ 8450 12200
@@
 Text Notes 6350 15800 0    394  ~ 0
 Solenoid Valves
-Text GLabel 7250 12000 0    35   Input ~ 0
+Text GLabel 8650 12700 2    35   Input ~ 0
 Encoder_PWM_4
-Text GLabel 7250 12100 0    35   Input ~ 0
+Text GLabel 8650 12800 2    35   Input ~ 0
 Encoder_PWM_5
 Wire Wire Line
 	7450 12000 7250 12000
 Wire Wire Line
-	7450 12100 7250 12100
+	7450 12300 7250 12300
 NoConn ~ 10100 12400
 NoConn ~ 7450 12500
@@
 $EndComp
 $Comp
-L power:+3.3V #PWR?
+L power:+3.3V #PWR0122
 U 1 1 632C14BD
 P 19600 12350
-F 0 "#PWR?" H 19600 12200 50  0001 C CNN
+F 0 "#PWR0122" H 19600 12200 50  0001 C CNN
 F 1 "+3.3V" V 19600 12450 35  0000 L CNN
 F 2 "" H 19600 12350 50  0001 C CNN
@@
 	19600 12350 19750 12350
 $Comp
-L Device:R R?
+L Device:R R16
 U 1 1 632C14C4
 P 19350 12750
-F 0 "R?" V 19250 12750 50  0000 C CNN
+F 0 "R16" V 19250 12750 50  0000 C CNN
 F 1 "43" V 19350 12750 39  0000 C CNN
 F 2 "Resistor_SMD:R_0603_1608Metric_Pad1.05x0.95mm_HandSolder" V 19280 12750 50  0001 C CNN
@@
 $EndComp
 $Comp
-L Device:LED_Small D?
+L Device:LED_Small D29
 U 1 1 632C14CA
 P 18900 12750
-F 0 "D?" H 18800 12700 39  0000 C CNN
+F 0 "D29" H 18800 12700 39  0000 C CNN
 F 1 "LED" H 19000 12700 35  0000 C CNN
 F 2 "LED_SMD:LED_0603_1608Metric_Pad1.05x0.95mm_HandSolder" V 18900 12750 50  0001 C CNN
@@
 	19000 12750 19200 12750
 $Comp
-L power:GND #PWR?
+L power:GND #PWR0123
 U 1 1 632C14D2
 P 18550 12750
-F 0 "#PWR?" H 18550 12500 50  0001 C CNN
+F 0 "#PWR0123" H 18550 12500 50  0001 C CNN
 F 1 "GND" H 18550 12600 39  0000 C CNN
 F 2 "" H 18550 12750 50  0001 C CNN
@@
 $EndComp
 $Comp
-L power:+3.3V #PWR?
+L power:+3.3V #PWR0124
 U 1 1 6334ADAE
 P 19600 13050
-F 0 "#PWR?" H 19600 12900 50  0001 C CNN
+F 0 "#PWR0124" H 19600 12900 50  0001 C CNN
 F 1 "+3.3V" V 19600 13150 35  0000 L CNN
 F 2 "" H 19600 13050 50  0001 C CNN
@@
 	19600 13050 19750 13050
 $Comp
-L Device:R R?
+L Device:R R17
 U 1 1 6334ADB5
 P 19350 13450
-F 0 "R?" V 19250 13450 50  0000 C CNN
+F 0 "R17" V 19250 13450 50  0000 C CNN
 F 1 "43" V 19350 13450 39  0000 C CNN
 F 2 "Resistor_SMD:R_0603_1608Metric_Pad1.05x0.95mm_HandSolder" V 19280 13450 50  0001 C CNN
@@
 $EndComp
 $Comp
-L Device:LED_Small D?
+L Device:LED_Small D30
 U 1 1 6334ADBB
 P 18900 13450
-F 0 "D?" H 18800 13400 39  0000 C CNN
+F 0 "D30" H 18800 13400 39  0000 C CNN
 F 1 "LED" H 19000 13400 35  0000 C CNN
 F 2 "LED_SMD:LED_0603_1608Metric_Pad1.05x0.95mm_HandSolder" V 18900 13450 50  0001 C CNN
@@
 	19000 13450 19200 13450
 $Comp
-L power:GND #PWR?
+L power:GND #PWR0125
 U 1 1 6334ADC3
 P 18550 13450
-F 0 "#PWR?" H 18550 13200 50  0001 C CNN
+F 0 "#PWR0125" H 18550 13200 50  0001 C CNN
 F 1 "GND" H 18550 13300 39  0000 C CNN
 F 2 "" H 18550 13450 50  0001 C CNN
@@
 $EndComp
 $Comp
-L power:+3.3V #PWR?
+L power:+3.3V #PWR0126
 U 1 1 633D7CD6
 P 19650 13700
-F 0 "#PWR?" H 19650 13550 50  0001 C CNN
+F 0 "#PWR0126" H 19650 13550 50  0001 C CNN
 F 1 "+3.3V" V 19650 13800 35  0000 L CNN
 F 2 "" H 19650 13700 50  0001 C CNN
@@
 	19650 13700 19800 13700
 $Comp
-L Device:R R?
+L Device:R R40
 U 1 1 633D7CDD
 P 19400 14100
-F 0 "R?" V 19300 14100 50  0000 C CNN
+F 0 "R40" V 19300 14100 50  0000 C CNN
 F 1 "43" V 19400 14100 39  0000 C CNN
 F 2 "Resistor_SMD:R_0603_1608Metric_Pad1.05x0.95mm_HandSolder" V 19330 14100 50  0001 C CNN
@@
 $EndComp
 $Comp
-L Device:LED_Small D?
+L Device:LED_Small D31
 U 1 1 633D7CE3
 P 18950 14100
-F 0 "D?" H 18850 14050 39  0000 C CNN
+F 0 "D31" H 18850 14050 39  0000 C CNN
 F 1 "LED" H 19050 14050 35  0000 C CNN
 F 2 "LED_SMD:LED_0603_1608Metric_Pad1.05x0.95mm_HandSolder" V 18950 14100 50  0001 C CNN
@@
 	19050 14100 19250 14100
 $Comp
-L power:GND #PWR?
+L power:GND #PWR0127
 U 1 1 633D7CEB
 P 18600 14100
-F 0 "#PWR?" H 18600 13850 50  0001 C CNN
+F 0 "#PWR0127" H 18600 13850 50  0001 C CNN
 F 1 "GND" H 18600 13950 39  0000 C CNN
 F 2 "" H 18600 14100 50  0001 C CNN
@@
 $EndComp
 $Comp
-L power:+3.3V #PWR?
+L power:+3.3V #PWR0128
 U 1 1 633D7CFE
 P 19650 14400
-F 0 "#PWR?" H 19650 14250 50  0001 C CNN
+F 0 "#PWR0128" H 19650 14250 50  0001 C CNN
 F 1 "+3.3V" V 19650 14500 35  0000 L CNN
 F 2 "" H 19650 14400 50  0001 C CNN
@@
 	19650 14400 19800 14400
 $Comp
-L Device:R R?
+L Device:R R49
 U 1 1 633D7D05
 P 19400 14800
-F 0 "R?" V 19300 14800 50  0000 C CNN
+F 0 "R49" V 19300 14800 50  0000 C CNN
 F 1 "43" V 19400 14800 39  0000 C CNN
 F 2 "Resistor_SMD:R_0603_1608Metric_Pad1.05x0.95mm_HandSolder" V 19330 14800 50  0001 C CNN
@@
 $EndComp
 $Comp
-L Device:LED_Small D?
+L Device:LED_Small D32
 U 1 1 633D7D0B
 P 18950 14800
-F 0 "D?" H 18850 14750 39  0000 C CNN
+F 0 "D32" H 18850 14750 39  0000 C CNN
 F 1 "LED" H 19050 14750 35  0000 C CNN
 F 2 "LED_SMD:LED_0603_1608Metric_Pad1.05x0.95mm_HandSolder" V 18950 14800 50  0001 C CNN
@@
 	19050 14800 19250 14800
 $Comp
-L power:GND #PWR?
+L power:GND #PWR0129
 U 1 1 633D7D13
 P 18600 14800
-F 0 "#PWR?" H 18600 14550 50  0001 C CNN
+F 0 "#PWR0129" H 18600 14550 50  0001 C CNN
 F 1 "GND" H 18600 14650 39  0000 C CNN
 F 2 "" H 18600 14800 50  0001 C CNN
@@
 Wire Wire Line
 	7450 10800 7300 10800
+Text GLabel 7250 12400 0    35   Input ~ 0
+Encoder_PWM_3
+Text GLabel 7250 12300 0    35   Input ~ 0
+Encoder_PWM_2
+Text GLabel 7250 12000 0    35   Input ~ 0
+Encoder_PWM_1
+Wire Wire Line
+	8650 12800 8450 12800
+Wire Wire Line
+	7450 12400 7250 12400
+Wire Wire Line
+	8650 12700 8450 12700
+NoConn ~ 7450 12100
+NoConn ~ 9950 11900
+NoConn ~ 9950 12000
+NoConn ~ 9950 12100
 $EndSCHEMATC

Commit message: Bunch more traces, slightly fixed some schematic issues
- LEDs on the solenoid valves were incorrectly labeled as "green".

- The front plane of the board is now +12VA instead of ground
Other:
- note added: "Blue"
- note removed: "Green\n"
- moved on the sheet: Conn6A, Conn6B, D19, D25, R39, R44, R45, R46, R48, U13

Commit message: Put components on the board and added some traces
Connections:
- net Encoder_PWM_1: now also U9.PA5 (B2_10); no longer U9.PD2 (A2_2)
- net Encoder_PWM_2: now also U9.PA4 (B2_9); no longer U9.PD4 (A2_5)
- net Encoder_PWM_4: now also U9.PD4 (A2_5); no longer U9.PA4 (B2_9)
- net Encoder_PWM_5: now also U9.PD2 (A2_2); no longer U9.PA5 (B2_10)
- net InA1_1: now also U9.PG1 (C2_1); no longer U9.PE2 (B1_5)
- net InA1_2: now also U9.PF2 (C1_2); no longer U9.PF1 (C1_1)
- net InA1_3: now also U9.PG0 (C1_4); no longer U9.PF3 (C1_3)
- net InA1_4: now also U9.PL1 (C1_8); no longer U9.PL0 (C1_7)
- net InA1_5: now also U9.PH1 (C2_8); no longer U9.PH0 (C2_7)
- net InA2_1: now also U9.PK4 (C2_2); no longer U9.PE3 (B1_6)
- net InA2_2: now also U9.PF1 (C1_1); no longer U9.PF2 (C1_2)
- net InA2_3: now also U9.PF3 (C1_3); no longer U9.PG0 (C1_4)
- net InA2_4: now also U9.PL0 (C1_7); no longer U9.PL1 (C1_8)
- net InA2_5: now also U9.PH0 (C2_7); no longer U9.PH1 (C2_8)
- net PWMA_1: now also U9.PM2 (C2_6); no longer U9.PD7 (B1_7)
Changed lines of the file:
@@
 $EndComp
 Wire Wire Line
-	8600 10700 8450 10700
+	9950 12400 10100 12400
 Wire Wire Line
 	10950 10500 10800 10500
@@
 $EndComp
 Wire Wire Line
-	8600 10500 8450 10500
-Wire Wire Line
-	8600 10600 8450 10600
+	9950 11900 10100 11900
 Wire Wire Line
-	10800 10100 10950 10100
+	9950 12000 10100 12000
 Wire Wire Line
 	10800 10200 10950 10200
 Wire Wire Line
-	9950 12500 10100 12500
+	10800 10100 10950 10100
 Wire Wire Line
 	9950 12600 10100 12600
 Wire Wire Line
+	9950 12500 10100 12500
+Wire Wire Line
 	9950 12700 10100 12700
 Wire Wire Line
@@
 Text Notes 9200 10650 0    276  ~ 0
 TIVA
-Wire Wire Line
-	9950 12100 10100 12100
-Wire Wire Line
-	9950 12000 10100 12000
-Wire Wire Line
-	9950 11900 10100 11900
 $Comp
 L MRDT_Connectors:Molex_SL_03 AbsEncode2
@@
 Wire Notes Line width 8 style solid
 	16200 9050 16200 9400
-Text GLabel 8600 10500 2    37   Input ~ 0
+Text GLabel 9950 11900 0    37   Input ~ 0
 InA1_1
-Text GLabel 8600 10600 2    37   Input ~ 0
+Text GLabel 9950 12000 0    37   Input ~ 0
 InA2_1
-Text GLabel 8600 10700 2    35   Input ~ 0
+Text GLabel 9950 12400 0    35   Input ~ 0
 PWMA_1
-Text GLabel 10800 10100 0    37   Input ~ 0
-InA1_2
 Text GLabel 10800 10200 0    37   Input ~ 0
+InA1_2
+Text GLabel 10800 10100 0    37   Input ~ 0
 InA2_2
 Text GLabel 10800 10500 0    35   Input ~ 0
@@
 Text Notes 6350 15800 0    394  ~ 0
 Solenoid Valves
-Text GLabel 8650 12700 2    35   Input ~ 0
+Text GLabel 7250 12300 0    35   Input ~ 0
 Encoder_PWM_4
-Text GLabel 8650 12800 2    35   Input ~ 0
+Text GLabel 7250 12000 0    35   Input ~ 0
 Encoder_PWM_5
 Wire Wire Line
@@
 Wire Wire Line
 	7450 12300 7250 12300
-NoConn ~ 10100 12400
+NoConn ~ 8450 10700
 NoConn ~ 7450 12500
 Text GLabel 7300 12600 0    35   Input ~ 0
@@
 NoConn ~ 8450 10400
 Wire Wire Line
-	10800 10800 10950 10800
-Wire Wire Line
 	10800 10700 10950 10700
 Wire Wire Line
-	10800 10400 10950 10400
+	10800 10800 10950 10800
 Wire Wire Line
 	10800 10300 10950 10300
-Text GLabel 10800 10800 0    37   Input ~ 0
-InA2_4
+Wire Wire Line
+	10800 10400 10950 10400
 Text GLabel 10800 10700 0    37   Input ~ 0
+InA2_4
+Text GLabel 10800 10800 0    37   Input ~ 0
 InA1_4
-Text GLabel 10800 10400 0    37   Input ~ 0
-InA2_3
 Text GLabel 10800 10300 0    37   Input ~ 0
+InA2_3
+Text GLabel 10800 10400 0    37   Input ~ 0
 InA1_3
-Text GLabel 9950 12500 0    37   Input ~ 0
-InA1_5
 Text GLabel 9950 12600 0    37   Input ~ 0
+InA1_5
+Text GLabel 9950 12500 0    37   Input ~ 0
 InA2_5
 Text GLabel 9950 12700 0    37   Input ~ 0
@@
 Text GLabel 7250 12400 0    35   Input ~ 0
 Encoder_PWM_3
-Text GLabel 7250 12300 0    35   Input ~ 0
+Text GLabel 8650 12700 2    35   Input ~ 0
 Encoder_PWM_2
-Text GLabel 7250 12000 0    35   Input ~ 0
+Text GLabel 8650 12800 2    35   Input ~ 0
 Encoder_PWM_1
 Wire Wire Line
@@
 	8650 12700 8450 12700
 NoConn ~ 7450 12100
-NoConn ~ 9950 11900
-NoConn ~ 9950 12000
-NoConn ~ 9950 12100
+NoConn ~ 8450 10500
+NoConn ~ 8450 10600
+NoConn ~ 10100 12100
 $EndSCHEMATC

Commit message: added daisy chain ports, updated andersons
Parts:
- removed unit 2 of Conn1
- removed unit 2 of Conn2
- removed unit 2 of Conn3
- removed unit 2 of Conn4
- removed unit 2 of Conn5
- removed unit 2 of Conn6
- added unit 3 of Conn1
- added unit 3 of Conn2
- added unit 3 of Conn3
- added unit 3 of Conn4
- added unit 3 of Conn5
- added unit 3 of Conn6
- added Conn8: Output, MRDT_Connectors:Anderson_2_Horizontal_Side_by_Side, symbol MRDT_Connectors:AndersonPP
- Conn1: value Motor_5 -> Motor1
- Conn2: value Motor_5 -> Motor2
- Conn3: value Motor_5 -> Motor3
- Conn4: value Motor_5 -> Motor4
- Conn5: value Motor_5 -> Motor5
- Conn6: value Motor_5 -> Motor6
- Conn7: value AndersonPP -> Input
- renumbered C5 to C1, C8 to C10, C9 to C11, C10 to C12, C6 to C2, C11 to C3, C3 to C4, C1 to C5, C12 to C6, C4 to C7, C2 to C8, C7 to C9, D9 to D1, D26 to D10, D6 to D13, D7 to D14, D13 to D15, D14 to D16, D20 to D17, D21 to D18, D15 to D19, D10 to D2, D16 to D20, D8 to D21, D17 to D22, D22 to D23, D18 to D25, D19 to D26, D23 to D27, D25 to D28, D27 to D3, D2 to D4, D1 to D5, D4 to D6, D5 to D7, D28 to D8, D3 to D9, R18 to R1, R23 to R10, R24 to R11, R25 to R12, R5 to R13, R6 to R14, R14 to R15, R3 to R16, R74 to R17, R26 to R18, R27 to R19, R19 to R2, R7 to R20, R28 to R21, R29 to R22, R8 to R23, R9 to R24, R30 to R25, R31 to R26, R32 to R27, R33 to R28, R34 to R29, R4 to R3, R35 to R30, R10 to R31, R68 to R32, R69 to R33, R36 to R34, R37 to R35, R11 to R36, R12 to R37, R70 to R38, R72 to R39, R13 to R4, R38 to R40, R39 to R41, R41 to R42, R42 to R43, R43 to R44, R44 to R45, R45 to R46, R46 to R47, R15 to R48, R47 to R49, R2 to R5, R48 to R50, R16 to R51, R17 to R52, R40 to R53, R49 to R54, R1 to R6, R20 to R7, R21 to R8, R22 to R9, U15 to U10, U5 to U11, U6 to U12, U14 to U13, U16 to U14, U17 to U15, U12 to U16, U13 to U17, U11 to U3, U10 to U4, U3 to U5, U4 to U6, U8 to U7, U7 to U8
Connections:
- net +12VA: now also Conn8.3 (V+Act)
- net GND: now also Conn8.1 (GND)
- net at D1.2 (A), U5.16 (OUTA+), U5.17 (OUTA+)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: now also Conn1.1 (GND)
- net at D11.2 (A), U5.26 (OUTB-), U5.27 (OUTB-)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: now also Conn1.3 (V+Act); no longer Conn1.1 (GND)
- net at D2.2 (A), U6.16 (OUTA+), U6.17 (OUTA+)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: now also Conn4.1 (GND)
- net at D12.2 (A), U6.26 (OUTB-), U6.27 (OUTB-)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: now also Conn4.3 (V+Act); no longer Conn4.1 (GND)
- net at D15.2 (A), U11.16 (OUTA+), U11.17 (OUTA+)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: now also Conn2.1 (GND)
- net at D19.2 (A), U11.26 (OUTB-), U11.27 (OUTB-)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: now also Conn2.3 (V+Act); no longer Conn2.1 (GND)
- net at D16.2 (A), U12.16 (OUTA+), U12.17 (OUTA+)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: now also Conn5.1 (GND)
- net at D20.2 (A), U12.26 (OUTB-), U12.27 (OUTB-)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: now also Conn5.3 (V+Act); no longer Conn5.1 (GND)
- net at D25.2 (A), U16.16 (OUTA+), U16.17 (OUTA+)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: now also Conn3.1 (GND)
- net at D27.2 (A), U16.26 (OUTB-), U16.27 (OUTB-)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: now also Conn3.3 (V+Act); no longer Conn3.1 (GND)
- net at D26.2 (A), U17.16 (OUTA+), U17.17 (OUTA+)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: now also Conn6.1 (GND)
- net at D28.2 (A), U17.26 (OUTB-), U17.27 (OUTB-)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: now also Conn6.3 (V+Act); no longer Conn6.1 (GND)
Other:
- note added: "Outputs to Daisy Chain"
- note removed: "Does this need analogWrite() or can\nit just be connected to a "green" pin?"
- moved on the sheet: C3, C4, C5, C6, C7, C8, Conn7A, Conn7B, Conn7C, D10, D3, D4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
