File: Hardware/ScienceMotorController/ScienceMotorController.sch (KiCad schematic (older format))
At the start: 140 parts, among them U1 LT1910, U10 PMN280ENEAX, U11 TB67H400AFNG,EL, U12 TB67H400AFNG,EL, U13 LT1910, U14 PMN280ENEAX, U15 LTC6900, U16 TB67H400AFNG,EL, U17 TB67H400AFNG,EL, U2 OKI, U3 OKI, U4 OKI, U5 TB67H400AFNG,EL, U6 TB67H400AFNG,EL, U7 PMN280ENEAX, U8 LT1910, U9 TM4C129E_Launchpad

Commit message: restarted layout
Parts:
- removed D11, D12, D19, D20, D27, D28: LED, LED_SMD:LED_0603_1608Metric_Pad1.05x0.95mm_HandSolder, symbol Device:LED_Small
- removed R18, R19, R34, R35, R49, R50: 1.5k, Resistor_SMD:R_0603_1608Metric_Pad1.05x0.95mm_HandSolder, symbol Device:R_Small
Connections:
- net +12VA: now also Conn8.2 (V+Log); no longer Conn8.3 (V+Act)
- net at D1.2 (A), U5.16 (OUTA+), U5.17 (OUTA+)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: now also Conn1.2 (V+Log); no longer Conn1.1 (GND)
- net at D15.2 (A), U11.16 (OUTA+), U11.17 (OUTA+)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: now also Conn2.2 (V+Log); no longer Conn2.1 (GND)
- net at D25.2 (A), U16.16 (OUTA+), U16.17 (OUTA+)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: now also Conn3.2 (V+Log); no longer Conn3.1 (GND)
- net at D2.2 (A), U6.16 (OUTA+), U6.17 (OUTA+)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: now also Conn4.2 (V+Log); no longer Conn4.1 (GND)
- net at D16.2 (A), U12.16 (OUTA+), U12.17 (OUTA+)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: now also Conn5.2 (V+Log); no longer Conn5.1 (GND)
- net at D26.2 (A), U17.16 (OUTA+), U17.17 (OUTA+)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: now also Conn6.2 (V+Log); no longer Conn6.1 (GND)
- net at U5.26 (OUTB-), U5.27 (OUTB-), U5.32 (OUTB+)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: now also Conn1.1 (GND); no longer Conn1.3 (V+Act)
- net at U12.26 (OUTB-), U12.27 (OUTB-), U12.32 (OUTB+)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: now also Conn5.1 (GND); no longer Conn5.3 (V+Act)
- net at U16.26 (OUTB-), U16.27 (OUTB-), U16.32 (OUTB+)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: now also Conn3.1 (GND); no longer Conn3.3 (V+Act)
- net at U6.26 (OUTB-), U6.27 (OUTB-), U6.32 (OUTB+)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: now also Conn4.1 (GND); no longer Conn4.3 (V+Act)
- net at U11.26 (OUTB-), U11.27 (OUTB-), U11.32 (OUTB+)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: now also Conn2.1 (GND); no longer Conn2.3 (V+Act)
- net at U17.26 (OUTB-), U17.27 (OUTB-), U17.32 (OUTB+)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: now also Conn6.1 (GND); no longer Conn6.3 (V+Act)
Other:
- moved on the sheet: Conn1A, Conn2A, Conn3A, Conn4A, Conn5A, Conn6A
