File: Hardware/ScienceMotorController/ScienceMotorController.sch (KiCad schematic (older format))
At the start: 120 parts, among them U1 LT1910, U10 PMN280ENEAX, U11 TB67H400AFNG,EL, U12 TB67H400AFNG,EL, U13 LT1910, U14 PMN280ENEAX, U15 LTC6900, U16 TB67H400AFNG,EL, U17 TB67H400AFNG,EL, U2 OKI, U3 OKI, U4 OKI, U5 TB67H400AFNG,EL, U6 TB67H400AFNG,EL, U7 PMN280ENEAX, U8 LT1910, U9 TM4C129E_Launchpad

Commit message: began reworking moco IC control traces. Will need to rearrange the netlist to reduce complexity of traces
Connections:
- net InA1_3: now also U9.PL0 (C1_7); no longer U9.PL1 (C1_8)
- net InA1_6: now also U9.PG0 (C1_4); no longer U9.PF3 (C1_3)
- net InA2_3: now also U9.PL1 (C1_8); no longer U9.PL0 (C1_7)
- net InA2_6: now also U9.PF3 (C1_3); no longer U9.PG0 (C1_4)
Changed lines of the file:
@@
 Text GLabel 9950 12600 0    37   Input ~ 0
 InA1_4
+Text GLabel 10800 10800 0    37   Input ~ 0
+InA2_3
 Text GLabel 10800 10700 0    37   Input ~ 0
-InA2_3
-Text GLabel 10800 10800 0    37   Input ~ 0
 InA1_3
 Text GLabel 9950 12800 0    37   Input ~ 0
@@
 Text GLabel 9950 12700 0    37   Input ~ 0
 InA2_5
+Text GLabel 10800 10400 0    37   Input ~ 0
+InA1_6
 Text GLabel 10800 10300 0    37   Input ~ 0
-InA1_6
-Text GLabel 10800 10400 0    37   Input ~ 0
 InA2_6
 Wire Notes Line width 8 style solid

Commit message: Completed Board and reviewed with Electrical Leadership
Connections:
- net InA1_1: now also U9.PL0 (C1_7); no longer U9.PF2 (C1_2)
- net InA1_2: now also U9.PK4 (C2_2); no longer U9.PG1 (C2_1)
- net InA1_3: now also U9.PF2 (C1_2); no longer U9.PL0 (C1_7)
- net InA1_4: now also U9.PH0 (C2_7); no longer U9.PH1 (C2_8)
- net InA2_1: now also U9.PL1 (C1_8); no longer U9.PF1 (C1_1)
- net InA2_2: now also U9.PG1 (C2_1); no longer U9.PK4 (C2_2)
- net InA2_3: now also U9.PF1 (C1_1); no longer U9.PL1 (C1_8)
- net InA2_4: now also U9.PH1 (C2_8); no longer U9.PH0 (C2_7)
- net PWMA_1: now also U9.PD1 (D1_6); no longer U9.PL4 (C1_5)
- net PWMA_2: now also U9.PM1 (C2_5); no longer U9.PM0 (C2_4)
- net PWMA_3: now also U9.PM0 (C2_4); no longer U9.PM1 (C2_5)
- net PWMA_4: now also U9.PL4 (C1_5); no longer U9.PD1 (D1_6)
- net at U9.PP4 (A2_8): now also R33.2
- net at U9.PQ0 (A2_7): now also R32.1
- net at U9.PP3 (D2_8): no longer R33.2
- net at U9.PQ2 (D2_6): no longer R32.2
- net at D17.2 (A): now also R32.2; no longer R32.1
Other:
- moved on the sheet: D17, D18, R32, R33
Changed lines of the file:
@@
 L Device:R R33
 U 1 1 6639E6F2
-P 11450 12600
-F 0 "R33" V 11350 12600 50  0000 C CNN
-F 1 "43" V 11450 12600 39  0000 C CNN
-F 2 "Resistor_SMD:R_0603_1608Metric_Pad1.05x0.95mm_HandSolder" V 11380 12600 50  0001 C CNN
-F 3 "~" H 11450 12600 50  0001 C CNN
-	1    11450 12600
-	0    1    1    0
+P 7300 12600
+F 0 "R33" V 7300 12800 50  0000 C CNN
+F 1 "43" V 7300 12600 39  0000 C CNN
+F 2 "Resistor_SMD:R_0603_1608Metric_Pad1.05x0.95mm_HandSolder" V 7230 12600 50  0001 C CNN
+F 3 "~" H 7300 12600 50  0001 C CNN
+	1    7300 12600
+	0    -1   -1   0
 $EndComp
 $Comp
 L Device:LED_Small D18
 U 1 1 6639E6F9
-P 11900 12600
-F 0 "D18" H 12000 12650 39  0000 C CNN
-F 1 "LED" H 11800 12650 35  0000 C CNN
-F 2 "LED_SMD:LED_0603_1608Metric_Pad1.05x0.95mm_HandSolder" V 11900 12600 50  0001 C CNN
-F 3 "~" V 11900 12600 50  0001 C CNN
-	1    11900 12600
-	-1   0    0    -1
-$EndComp
-Wire Wire Line
-	12000 12600 12250 12600
-Wire Wire Line
-	11800 12600 11600 12600
-$Comp
-L power:GND #PWR076
-U 1 1 6639E703
-P 12250 12600
-F 0 "#PWR076" H 12250 12350 50  0001 C CNN
-F 1 "GND" H 12250 12450 39  0000 C CNN
-F 2 "" H 12250 12600 50  0001 C CNN
-F 3 "" H 12250 12600 50  0001 C CNN
-	1    12250 12600
-	1    0    0    -1
+P 6850 12600
+F 0 "D18" H 6950 12650 39  0000 C CNN
+F 1 "LED" H 6750 12650 35  0000 C CNN
+F 2 "LED_SMD:LED_0603_1608Metric_Pad1.05x0.95mm_HandSolder" V 6850 12600 50  0001 C CNN
+F 3 "~" V 6850 12600 50  0001 C CNN
+	1    6850 12600
+	1    0    0    1
 $EndComp
-Wire Wire Line
-	11100 12600 11300 12600
 $Comp
 L Device:R R32
 U 1 1 6640B5FD
-P 11450 12400
-F 0 "R32" V 11350 12400 50  0000 C CNN
-F 1 "43" V 11450 12400 39  0000 C CNN
-F 2 "Resistor_SMD:R_0603_1608Metric_Pad1.05x0.95mm_HandSolder" V 11380 12400 50  0001 C CNN
-F 3 "~" H 11450 12400 50  0001 C CNN
-	1    11450 12400
-	0    1    1    0
+P 7300 12500
+F 0 "R32" V 7300 12300 50  0000 C CNN
+F 1 "43" V 7300 12500 39  0000 C CNN
+F 2 "Resistor_SMD:R_0603_1608Metric_Pad1.05x0.95mm_HandSolder" V 7230 12500 50  0001 C CNN
+F 3 "~" H 7300 12500 50  0001 C CNN
+	1    7300 12500
+	0    1    -1   0
 $EndComp
 $Comp
 L Device:LED_Small D17
 U 1 1 6640B604
-P 11900 12400
-F 0 "D17" H 12000 12450 39  0000 C CNN
-F 1 "LED" H 11800 12450 35  0000 C CNN
-F 2 "LED_SMD:LED_0603_1608Metric_Pad1.05x0.95mm_HandSolder" V 11900 12400 50  0001 C CNN
-F 3 "~" V 11900 12400 50  0001 C CNN
-	1    11900 12400
-	-1   0    0    -1
+P 6850 12500
+F 0 "D17" H 6750 12550 39  0000 C CNN
+F 1 "LED" H 6950 12550 35  0000 C CNN
+F 2 "LED_SMD:LED_0603_1608Metric_Pad1.05x0.95mm_HandSolder" V 6850 12500 50  0001 C CNN
+F 3 "~" V 6850 12500 50  0001 C CNN
+	1    6850 12500
+	1    0    0    -1
 $EndComp
-Wire Wire Line
-	12000 12400 12250 12400
-Wire Wire Line
-	11800 12400 11600 12400
 $Comp
 L power:GND #PWR075
 U 1 1 6640B60E
-P 12250 12400
-F 0 "#PWR075" H 12250 12150 50  0001 C CNN
-F 1 "GND" H 12250 12250 39  0000 C CNN
-F 2 "" H 12250 12400 50  0001 C CNN
-F 3 "" H 12250 12400 50  0001 C CNN
-	1    12250 12400
-	1    0    0    -1
+P 6700 12650
+F 0 "#PWR075" H 6700 12400 50  0001 C CNN
+F 1 "GND" H 6700 12500 39  0000 C CNN
+F 2 "" H 6700 12650 50  0001 C CNN
+F 3 "" H 6700 12650 50  0001 C CNN
+	1    6700 12650
+	-1   0    0    -1
 $EndComp
-Wire Wire Line
-	11100 12400 11300 12400
 $Comp
 L MRDT_Connectors:Molex_SL_02 LimSwitch1
@@
 Text Notes 13350 10150 0    28   ~ 0
 Blue\n
-Text Notes 11950 12650 0    28   ~ 0
-Blue\n
-Text Notes 11950 12450 0    28   ~ 0
+Text Notes 6900 12750 2    28   ~ 0
 Blue\n
 $Comp
@@
 Wire Notes Line width 8 style solid
 	16200 9050 16200 9400
-Text GLabel 10800 10200 0    37   Input ~ 0
-InA1_1
-Text GLabel 10800 10100 0    37   Input ~ 0
-InA2_1
-Text GLabel 10800 10500 0    35   Input ~ 0
+Text GLabel 12100 10600 2    35   Input ~ 0
 PWMA_1
-Text GLabel 9950 11900 0    37   Input ~ 0
-InA1_2
 Text GLabel 9950 12000 0    37   Input ~ 0
+InA1_2
+Text GLabel 9950 11900 0    37   Input ~ 0
 InA2_2
-Text GLabel 9950 12200 0    35   Input ~ 0
-PWMA_2
 Text GLabel 9950 12300 0    35   Input ~ 0
+PWMA_2
+Text GLabel 9950 12200 0    35   Input ~ 0
 PWMA_3
-Text GLabel 12100 10600 2    35   Input ~ 0
+Text GLabel 10800 10500 0    35   Input ~ 0
 PWMA_4
 $Comp
@@
 	7450 12300 7250 12300
 NoConn ~ 8450 10700
-NoConn ~ 7450 12500
 Wire Wire Line
 	8600 12100 8450 12100
@@
 Wire Wire Line
 	10800 10400 10950 10400
-Text GLabel 9950 12500 0    37   Input ~ 0
-InA2_4
 Text GLabel 9950 12600 0    37   Input ~ 0
+InA2_4
+Text GLabel 9950 12500 0    37   Input ~ 0
 InA1_4
-Text GLabel 10800 10800 0    37   Input ~ 0
+Text GLabel 10800 10100 0    37   Input ~ 0
 InA2_3
-Text GLabel 10800 10700 0    37   Input ~ 0
+Text GLabel 10800 10200 0    37   Input ~ 0
 InA1_3
 Text GLabel 9950 12800 0    37   Input ~ 0
@@
 	-1   0    0    -1
 $EndComp
-NoConn ~ 7450 12600
 NoConn ~ 7450 12700
 NoConn ~ 7450 12800
 Wire Wire Line
 	8450 12000 9200 12000
+Text GLabel 10800 10800 0    37   Input ~ 0
+InA2_1
+Text GLabel 10800 10700 0    37   Input ~ 0
+InA1_1
+Wire Wire Line
+	7150 12500 6950 12500
+Wire Wire Line
+	6750 12500 6700 12500
+Wire Wire Line
+	6700 12500 6700 12600
+NoConn ~ 11100 12400
+NoConn ~ 11100 12600
+Wire Wire Line
+	7150 12600 6950 12600
+Wire Wire Line
+	6750 12600 6700 12600
+Connection ~ 6700 12600
+Wire Wire Line
+	6700 12600 6700 12650
 $EndSCHEMATC

Commit message: began fixing rescue libraries
created ScienceMotorController.lib as the new project level library
Parts:
- U10, U14, U7: symbol ScienceMotorController-rescue:PMN280ENEAX-SciMoCoLib -> ScienceMotorController:PMN280ENEAX-SciMoCoLib
- U15: symbol ScienceMotorController-rescue:LTC6900-SciMoCoLib -> MRDT_Devices:LTC6900
Changed lines of the file:
@@
 	2600 10450 2600 10550
 $Comp
-L ScienceMotorController-rescue:PMN280ENEAX-SciMoCoLib U7
+L ScienceMotorController:PMN280ENEAX-SciMoCoLib U7
 U 1 1 64F13429
 P 5100 14050
@@
 Connection ~ 4800 13850
 $Comp
-L ScienceMotorController-rescue:PMN280ENEAX-SciMoCoLib U10
+L ScienceMotorController:PMN280ENEAX-SciMoCoLib U10
 U 1 1 65651C73
 P 9250 14000
@@
 Connection ~ 8950 13800
 $Comp
-L ScienceMotorController-rescue:PMN280ENEAX-SciMoCoLib U14
+L ScienceMotorController:PMN280ENEAX-SciMoCoLib U14
 U 1 1 656CCAC6
 P 13350 13950
@@
 	1    0    0    -1
 $EndComp
-$Comp
-L ScienceMotorController-rescue:LTC6900-SciMoCoLib U15
-U 1 1 65A4B48D
-P 16800 12650
-F 0 "U15" H 16800 13025 50  0000 C CNN
-F 1 "LTC6900" H 16800 12934 50  0000 C CNN
-F 2 "Package_TO_SOT_SMD:SOT-23-5_HandSoldering" H 16800 12500 50  0001 C CNN
-F 3 "" H 16800 12500 50  0001 C CNN
-	1    16800 12650
-	1    0    0    -1
-$EndComp
 Wire Wire Line
 	16350 12700 16450 12700
@@
 Wire Wire Line
 	16000 12700 16000 12200
-Wire Wire Line
-	16450 12500 16400 12500
 Wire Wire Line
 	16400 12500 16400 12200
@@
 Text GLabel 17250 12600 2    50   Input ~ 0
 Oscillator
-Wire Wire Line
-	17150 12600 17250 12600
 Text GLabel 3900 2700 0    50   Input ~ 0
 Oscillator
@@
 Wire Wire Line
 	6700 12600 6700 12650
+Wire Wire Line
+	16450 12500 16400 12500
+$Comp
+L MRDT_Devices:LTC6900 U15
+U 1 1 65A4B48D
+P 16700 12560
+F 0 "U15" H 16700 12935 50  0000 C CNN
+F 1 "LTC6900" H 16700 12844 50  0000 C CNN
+F 2 "Package_TO_SOT_SMD:SOT-23-5_HandSoldering" H 16700 12410 50  0001 C CNN
+F 3 "" H 16700 12410 50  0001 C CNN
+	1    16700 12560
+	1    0    0    -1
+$EndComp
+Wire Wire Line
+	17090 12600 17250 12600
 $EndSCHEMATC

Commit message: Updated Schematic, Started Layout
Parts:
- removed C13: 10uF, Capacitor_SMD:C_0603_1608Metric_Pad1.05x0.95mm_HandSolder, symbol Device:C
- removed Conn5: Motor5, MRDT_Connectors:Anderson_2_Horizontal_Side_by_Side, symbol MRDT_Connectors:AndersonPP
- removed Conn6: Motor6, MRDT_Connectors:Anderson_2_Horizontal_Side_by_Side, symbol MRDT_Connectors:AndersonPP
- removed D15, D16, D24, D26, D29, D30, D31, D32: LED, LED_SMD:LED_0603_1608Metric_Pad1.05x0.95mm_HandSolder, symbol Device:LED_Small
- removed R40, R41: 1.5k, Resistor_SMD:R_0603_1608Metric_Pad1.05x0.95mm_HandSolder, symbol Device:R_Small
- removed R42, R43, R44, R45, R46, R47: 1k, Resistor_SMD:R_0603_1608Metric_Pad1.05x0.95mm_HandSolder, symbol Device:R_Small
- removed R48: 20k, Resistor_SMD:R_0603_1608Metric_Pad1.05x0.95mm_HandSolder, symbol Device:R
- removed R53, R54: 43, Resistor_SMD:R_0603_1608Metric_Pad1.05x0.95mm_HandSolder, symbol Device:R
- removed R6: 330, Resistor_SMD:R_0603_1608Metric_Pad1.05x0.95mm_HandSolder, symbol Device:R
- removed U11, U12, U16, U17, U5, U6: TB67H400AFNG,EL, MRDT_ICs:TB67H400AFNG,EL, symbol MRDT_ICs:TB67H400AFNG,EL
- removed U15: LTC6900, Package_TO_SOT_SMD:SOT-23-5_HandSoldering, symbol MRDT_Devices:LTC6900
- added AbsEncode6: Molex_SL_03, MRDT_Connectors:MOLEX_SL_03_Vertical, symbol MRDT_Connectors:Molex_SL_03
- added C1, C2, C3, C4: 33nF, Capacitor_SMD:C_0603_1608Metric_Pad1.08x0.95mm_HandSolder, symbol Device:C_Small
- added C21, C22: 10uF, Capacitor_SMD:C_0603_1608Metric_Pad1.08x0.95mm_HandSolder, symbol Device:C
- added C5, C6, C7, C8: 10uF, Capacitor_SMD:C_0603_1608Metric_Pad1.08x0.95mm_HandSolder, symbol Device:C_Small
- added Conn7: Output2, MRDT_Connectors:Anderson_2_Horizontal_Side_by_Side, symbol MRDT_Connectors:AndersonPP
- added D11, D17, D18, D19, D20, D21, D3, D4, D6, D7, D8: LED, LED_SMD:LED_0603_1608Metric_Pad1.05x0.95mm_HandSolder, symbol Device:LED_Small
- added R13, R14, R15, R16: 3.3k, Resistor_SMD:R_0603_1608Metric_Pad0.98x0.95mm_HandSolder, symbol Device:R_Small
- added R18, R19, R20, R34, R35, R36: 1k, Resistor_SMD:R_0603_1608Metric_Pad0.98x0.95mm_HandSolder, symbol Device:R_Small
- added R23, R24: 10k, Resistor_SMD:R_0603_1608Metric_Pad0.98x0.95mm_HandSolder, symbol Device:R_Small
- added R3, R31, R32, R4, R5, R6, R7, R8: 1.5k, Resistor_SMD:R_0603_1608Metric_Pad0.98x0.95mm_HandSolder, symbol Device:R_Small
- added R45, R46, R47: 130, Resistor_SMD:R_0603_1608Metric_Pad0.98x0.95mm_HandSolder, symbol Device:R
- added R56: 300, Resistor_SMD:R_0603_1608Metric_Pad0.98x0.95mm_HandSolder, symbol Device:R
- added U1, U2, U3, U4: VNH5019A_E, MRDT_ICs:MultiPowerSO_30, symbol MRDT_ICs:VNH5019A_E
- added U15: 5VA OKI, MRDT_Devices:OKI_Horizontal, symbol MRDT_Devices:OKI
- C10: renamed from C6; footprint Capacitor_SMD:C_0603_1608Metric_Pad1.05x0.95mm_HandSolder -> Capacitor_SMD:C_0603_1608Metric_Pad1.08x0.95mm_HandSolder
- C11: renamed from C4; footprint Capacitor_SMD:C_0603_1608Metric_Pad1.05x0.95mm_HandSolder -> Capacitor_SMD:C_0603_1608Metric_Pad1.08x0.95mm_HandSolder
- C12: renamed from C7; footprint Capacitor_SMD:C_0603_1608Metric_Pad1.05x0.95mm_HandSolder -> Capacitor_SMD:C_0603_1608Metric_Pad1.08x0.95mm_HandSolder
- C13: renamed from C5; footprint Capacitor_SMD:C_0603_1608Metric_Pad1.05x0.95mm_HandSolder -> Capacitor_SMD:C_0603_1608Metric_Pad1.08x0.95mm_HandSolder
- C14: renamed from C8; footprint Capacitor_SMD:C_0603_1608Metric_Pad1.05x0.95mm_HandSolder -> Capacitor_SMD:C_0603_1608Metric_Pad1.08x0.95mm_HandSolder
- C15: renamed from C11; footprint Capacitor_SMD:C_0603_1608Metric_Pad1.05x0.95mm_HandSolder -> Capacitor_SMD:C_0603_1608Metric_Pad1.08x0.95mm_HandSolder
- C17: renamed from C9; footprint Capacitor_SMD:C_0603_1608Metric_Pad1.05x0.95mm_HandSolder -> Capacitor_SMD:C_0603_1608Metric_Pad1.08x0.95mm_HandSolder
- C19: renamed from C1; footprint Capacitor_SMD:C_0603_1608Metric_Pad1.05x0.95mm_HandSolder -> Capacitor_SMD:C_0603_1608Metric_Pad1.08x0.95mm_HandSolder
- C9: renamed from C3; footprint Capacitor_SMD:C_0603_1608Metric_Pad1.05x0.95mm_HandSolder -> Capacitor_SMD:C_0603_1608Metric_Pad1.08x0.95mm_HandSolder
- Conn6: renamed from Conn8; value Output -> Output1
- R1, R10, R11, R12, R2: footprint Resistor_SMD:R_0603_1608Metric_Pad1.05x0.95mm_HandSolder -> Resistor_SMD:R_0603_1608Metric_Pad0.98x0.95mm_HandSolder
- R17: renamed from R9; footprint Resistor_SMD:R_0603_1608Metric_Pad1.05x0.95mm_HandSolder -> Resistor_SMD:R_0603_1608Metric_Pad0.98x0.95mm_HandSolder
- R21, R22: value 1.5k -> 10k; footprint Resistor_SMD:R_0603_1608Metric_Pad1.05x0.95mm_HandSolder -> Resistor_SMD:R_0603_1608Metric_Pad0.98x0.95mm_HandSolder
- R25, R26, R27, R28: value 1k -> 3.3k; footprint Resistor_SMD:R_0603_1608Metric_Pad1.05x0.95mm_HandSolder -> Resistor_SMD:R_0603_1608Metric_Pad0.98x0.95mm_HandSolder
- R29, R30: value 1k -> 1.5k; footprint Resistor_SMD:R_0603_1608Metric_Pad1.05x0.95mm_HandSolder -> Resistor_SMD:R_0603_1608Metric_Pad0.98x0.95mm_HandSolder
- R33: renamed from R8; footprint Resistor_SMD:R_0603_1608Metric_Pad1.05x0.95mm_HandSolder -> Resistor_SMD:R_0603_1608Metric_Pad0.98x0.95mm_HandSolder
- R37: renamed from R15; value 43 -> 300; footprint Resistor_SMD:R_0603_1608Metric_Pad1.05x0.95mm_HandSolder -> Resistor_SMD:R_0603_1608Metric_Pad0.98x0.95mm_HandSolder
- R38: renamed from R5; value 330 -> 1k; footprint Resistor_SMD:R_0603_1608Metric_Pad1.05x0.95mm_HandSolder -> Resistor_SMD:R_0603_1608Metric_Pad0.98x0.95mm_HandSolder
- R39: value 43 -> 1k; footprint Resistor_SMD:R_0603_1608Metric_Pad1.05x0.95mm_HandSolder -> Resistor_SMD:R_0603_1608Metric_Pad0.98x0.95mm_HandSolder
- R40: renamed from R16; value 43 -> 130; footprint Resistor_SMD:R_0603_1608Metric_Pad1.05x0.95mm_HandSolder -> Resistor_SMD:R_0603_1608Metric_Pad0.98x0.95mm_HandSolder
- R41: renamed from R17; value 43 -> 300; footprint Resistor_SMD:R_0603_1608Metric_Pad1.05x0.95mm_HandSolder -> Resistor_SMD:R_0603_1608Metric_Pad0.98x0.95mm_HandSolder
- R42: renamed from R32; value 43 -> 130; footprint Resistor_SMD:R_0603_1608Metric_Pad1.05x0.95mm_HandSolder -> Resistor_SMD:R_0603_1608Metric_Pad0.98x0.95mm_HandSolder
- R43: renamed from R33; value 43 -> 130; footprint Resistor_SMD:R_0603_1608Metric_Pad1.05x0.95mm_HandSolder -> Resistor_SMD:R_0603_1608Metric_Pad0.98x0.95mm_HandSolder
- R44: renamed from R38; value 43 -> 130; footprint Resistor_SMD:R_0603_1608Metric_Pad1.05x0.95mm_HandSolder -> Resistor_SMD:R_0603_1608Metric_Pad0.98x0.95mm_HandSolder
- R48: renamed from R31; footprint Resistor_SMD:R_0603_1608Metric_Pad1.05x0.95mm_HandSolder -> Resistor_SMD:R_0603_1608Metric_Pad0.98x0.95mm_HandSolder
- R49: renamed from R20; footprint Resistor_SMD:R_0603_1608Metric_Pad1.05x0.95mm_HandSolder -> Resistor_SMD:R_0603_1608Metric_Pad0.98x0.95mm_HandSolder
- R50: renamed from R3; footprint Resistor_SMD:R_0603_1608Metric_Pad1.05x0.95mm_HandSolder -> Resistor_SMD:R_0603_1608Metric_Pad0.98x0.95mm_HandSolder
- R51, R52: value 43 -> 130; footprint Resistor_SMD:R_0603_1608Metric_Pad1.05x0.95mm_HandSolder -> Resistor_SMD:R_0603_1608Metric_Pad0.98x0.95mm_HandSolder
- R53: renamed from R37; value 43 -> 130; footprint Resistor_SMD:R_0603_1608Metric_Pad1.05x0.95mm_HandSolder -> Resistor_SMD:R_0603_1608Metric_Pad0.98x0.95mm_HandSolder
- R54: renamed from R24; value 43 -> 130; footprint Resistor_SMD:R_0603_1608Metric_Pad1.05x0.95mm_HandSolder -> Resistor_SMD:R_0603_1608Metric_Pad0.98x0.95mm_HandSolder
- R55: renamed from R14; value 43 -> 130; footprint Resistor_SMD:R_0603_1608Metric_Pad1.05x0.95mm_HandSolder -> Resistor_SMD:R_0603_1608Metric_Pad0.98x0.95mm_HandSolder
- R9: renamed from R7; footprint Resistor_SMD:R_0603_1608Metric_Pad1.05x0.95mm_HandSolder -> Resistor_SMD:R_0603_1608Metric_Pad0.98x0.95mm_HandSolder
- U5: renamed from U2; value OKI -> 5V OKI
- U7: renamed from U3; value OKI -> 3V3 OKI
- U8: renamed from U4; value OKI -> 5VA OKI
- renumbered C12 to C16, C10 to C18, C2 to C20, Conn7 to Conn5, D4 to D10, D9 to D12, D10 to D13, D17 to D14, D18 to D15, D23 to D16, D14 to D23, D7 to D24, D8 to D9, SolValve3 to SolValve1, SolValve1 to SolValve3, U7 to U11, U13 to U12, U8 to U13, U1 to U14, U9 to U6, U14 to U9
Connections:
- net labels added: Current_Sense_1, Current_Sense_2, Current_Sense_3, Current_Sense_4, Encoder_PWM_6, INA_1, INA_2, INA_3, INA_4, INA_5, INA_6, INB_1, INB_2, INB_3, INB_4, INB_5, INB_6, PWM_1, PWM_2, PWM_3, PWM_4, PWM_5, PWM_6
- net labels removed: InA1_1, InA1_2, InA1_3, InA1_4, InA1_5, InA1_6, InA2_1, InA2_2, InA2_3, InA2_4, InA2_5, InA2_6, Oscillator, PWMA_1, PWMA_2, PWMA_3, PWMA_4, PWMA_5, PWMA_6
- wire segments 673 -> 625
- no-connect marks 81 -> 41
Other:
- note added: "Red\n"
- note added: "Spare"
- note removed: "2 are spares"
- note removed: "Clock Circuit"
- note removed: "Outputs to Daisy Chain"
- note removed: "Pump 1"
- note removed: "Pump 2"
- note removed: "Pump 3"
- moved on the sheet: AbsEncode1, C10, C11, C12, C13, C14, C15, C16, C17, C18, C19, C20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

Commit message: Layout Ready For Review
Parts:
- renumbered AbsEncode6 to AbsEncode1, AbsEncode4 to AbsEncode2, AbsEncode2 to AbsEncode3, AbsEncode5 to AbsEncode4, AbsEncode3 to AbsEncode5, AbsEncode1 to AbsEncode6, LimSwitch3 to LimSwitch2, LimSwitch5 to LimSwitch3, LimSwitch2 to LimSwitch4, LimSwitch4 to LimSwitch5, SolValve3 to SolValve1, SolValve1 to SolValve3
Connections:
- net Encoder_PWM_1: now also AbsEncode1.3, U6.PA6 (B1_8); no longer AbsEncode6.3, U6.PA5 (B2_10)
- net Encoder_PWM_2: now also AbsEncode2.3, U6.PD2 (A2_2); no longer AbsEncode5.3, U6.PA4 (B2_9)
- net Encoder_PWM_3: now also AbsEncode3.3, U6.PD0 (D1_7); no longer AbsEncode4.3, U6.PD3 (A1_7)
- net Encoder_PWM_4: now also AbsEncode4.3, U6.PD3 (A1_7); no longer AbsEncode3.3, U6.PD0 (D1_7)
- net Encoder_PWM_5: now also AbsEncode5.3, U6.PA4 (B2_9); no longer AbsEncode2.3, U6.PD2 (A2_2)
- net Encoder_PWM_6: now also AbsEncode6.3, U6.PA5 (B2_10); no longer AbsEncode1.3, U6.PA6 (B1_8)
- net INA_5: no longer names the net of U6.PK7 (C2_10)
- net INA_6: no longer names the net of U6.PG0 (C1_4)
- net INB_5: no longer names the net of U6.PK6 (C2_9)
- net INB_6: no longer names the net of U6.PF3 (C1_3)
- net PWM_5: no longer names the net of U6.PM2 (C2_6)
- net PWM_6: no longer names the net of U6.PL5 (C1_6)
- no-connect marks 41 -> 47
Other:
- moved on the sheet: AbsEncode1, AbsEncode2, AbsEncode3, AbsEncode4, AbsEncode5, AbsEncode6

Commit message: 9 Solenoids, Fixed PWM Overlap
Parts:
- removed C15, C17, C19: 0.1 uF, Capacitor_SMD:C_0603_1608Metric_Pad1.08x0.95mm_HandSolder, symbol Device:C
- removed C16, C18, C20: 10uF 50V, Capacitor_SMD:C_0603_1608Metric_Pad1.08x0.95mm_HandSolder, symbol Device:CP1
- removed R53, R54, R55: 130, Resistor_SMD:R_0603_1608Metric_Pad0.98x0.95mm_HandSolder, symbol Device:R
- removed SolValve1, SolValve2, SolValve3: Molex_SL_02, MRDT_Connectors:MOLEX_SL_02_Vertical, symbol MRDT_Connectors:Molex_SL_02
- removed U10, U11, U9: PMN280ENEAX, Mosfet:PMN280ENEAX, symbol ScienceMotorController:PMN280ENEAX-SciMoCoLib
- removed U12, U13, U14: LT1910, Package_SO:SOIC-8_3.9x4.9mm_P1.27mm, symbol MRDT_ICs:LT1910
- added D26, D27, D28, D29, D30, D31: LED, LED_SMD:LED_0603_1608Metric_Pad1.05x0.95mm_HandSolder, symbol Device:LED_Small
- added Q1, Q2, Q3, Q4, Q5, Q6, Q7, Q8, Q9: BSS138, Package_TO_SOT_SMD:SOT-23, symbol Transistor_FET:BSS138
- added R53, R54, R55, R57, R58, R59: 1k, Resistor_SMD:R_0603_1608Metric_Pad0.98x0.95mm_HandSolder, symbol Device:R_Small
- added SolVal1, SolVal2, SolVal3, SolVal4, SolVal5, SolVal6, SolVal7, SolVal8, SolVal9: Molex_SL_02, MRDT_Connectors:MOLEX_SL_02_Vertical, symbol MRDT_Connectors:Molex_SL_02
- R1, R2, R3, R4, R5, R6, R7, R8: value 1.5k -> 1k
- R48, R49, R50: value 5.1k -> 1k
Connections:
- net +12VA: now also D22.2 (A), D23.2 (A), D24.2 (A), D26.2 (A), D27.2 (A), D28.2 (A), D29.2 (A), D30.2 (A), D31.2 (A), SolVal1.1, SolVal2.1, SolVal3.1, SolVal4.1, SolVal5.1, SolVal6.1, SolVal7.1, SolVal8.1, SolVal9.1
- net +5V: no longer R48.2, R49.2, R50.2
- net Encoder_PWM_3: now also U6.PD5 (A2_6); no longer U6.PD0 (D1_7)
- net GND: now also Q1.2 (S), Q2.2 (S), Q3.2 (S), Q4.2 (S), Q5.2 (S), Q6.2 (S), Q7.2 (S), Q8.2 (S), Q9.2 (S); no longer D22.1 (K), D23.1 (K), D24.1 (K)
- net PWM_2: now also U6.PM4 (B1_9); no longer U6.PM1 (C2_5)
- net PWM_3: now also U6.PM5 (B1_10); no longer U6.PM0 (C2_4)
- net Solenoid_Valve_1: now also Q1.1 (G)
- net Solenoid_Valve_2: now also U6.PP0 (A2_3), Q2.1 (G); no longer U6.PB5 (B2_4)
- net Solenoid_Valve_3: now also U6.PB5 (B2_4), Q3.1 (G); no longer U6.PK0 (B2_5)
- net Solenoid_Valve_6: now reaches U6.PD4 (A2_5)
- net Solenoid_Valve_6: now also Q6.1 (G)
- net Solenoid_Valve_4: now reaches U6.PP1 (A2_4)
- net Solenoid_Valve_4: now also Q4.1 (G)
- net Solenoid_Valve_7: now reaches U6.PK1 (B2_6)
- net Solenoid_Valve_7: now also Q7.1 (G)
- net Solenoid_Valve_8: now reaches U6.PK2 (B2_7)
- net Solenoid_Valve_8: now also Q8.1 (G)
- net Solenoid_Valve_9: now reaches U6.PK3 (B2_8)
- net Solenoid_Valve_9: now also Q9.1 (G)
- net at R50.1: now also D24.1 (K)
- net at R49.1: now also D23.1 (K)
- net at R48.1: now also D22.1 (K)
- new net: Q1.3 (D), R48.2, SolVal1.2
- new net: Q2.3 (D), R49.2, SolVal2.2
- new net: Q3.3 (D), R50.2, SolVal3.2
- new net: Q4.3 (D), R53.2, SolVal4.2
- new net: D26.1 (K), R53.1
- new net: Q5.3 (D), R54.2, SolVal5.2
- new net: D27.1 (K), R54.1
- new net: Q6.3 (D), R55.2, SolVal6.2
- new net: D28.1 (K), R55.1
- new net: Q7.3 (D), R57.2, SolVal7.2
- new net: D29.1 (K), R57.1
- new net: Q8.3 (D), R58.2, SolVal8.2
- new net: D30.1 (K), R58.1
- new net: Q9.3 (D), R59.2, SolVal9.2
- new net: D31.1 (K), R59.1
- new net Solenoid_Valve_5: Q5.1 (G), U6.PK0 (B2_5)
- no-connect marks 47 -> 41
Other:
- note added: "Solenoid\nValves"
- note removed: "Solenoid Valves"
- moved on the sheet: D14

Commit message: Removed 5V Oki, Moved +12V Passthrough Trace, Added Zener Diodes for Current Sense
Parts:
- removed C10, C9: 10uF, Capacitor_SMD:C_0603_1608Metric_Pad1.08x0.95mm_HandSolder, symbol Device:C
- removed D9: LED, LED_SMD:LED_0603_1608Metric_Pad1.05x0.95mm_HandSolder, symbol Device:LED_Small
- removed R37: 300, Resistor_SMD:R_0603_1608Metric_Pad0.98x0.95mm_HandSolder, symbol Device:R
- removed U5: 5V OKI, MRDT_Devices:OKI_Horizontal, symbol MRDT_Devices:OKI
- added D10, D11, D12, D9: 3.3V, Diode_SMD:D_0603_1608Metric_Pad1.05x0.95mm_HandSolder, symbol Device:D_Zener_Small
- renumbered AbsEncode4 to AbsEncode2, AbsEncode2 to AbsEncode3, AbsEncode5 to AbsEncode4, AbsEncode3 to AbsEncode5, C12 to C10, C13 to C11, C14 to C12, C21 to C13, C22 to C14, C11 to C9, D12 to D13, D10 to D14, D11 to D15, D13 to D16, D25 to D17, D14 to D18, D15 to D19, D16 to D20, D17 to D21, D18 to D22, D19 to D23, D22 to D24, D23 to D25, D24 to D26, D26 to D27, D27 to D28, D28 to D29, D29 to D30, D30 to D31, D31 to D32, D20 to D33, D21 to D34, LimSwitch4 to LimSwitch2, LimSwitch2 to LimSwitch3, LimSwitch5 to LimSwitch4, LimSwitch3 to LimSwitch5, R40 to R37, R41 to R40, R56 to R41, R51 to R48, R52 to R49, R48 to R50, R49 to R51, R50 to R52, R57 to R56, R58 to R57, R59 to R58, U7 to U5, U8 to U7, U15 to U8
Connections:
- net +5V is gone; now on net +3V3: R13.2, R14.2, R15.2, R16.2, R25.2, R26.2, R27.2, R28.2
- net Current_Sense_1: now also D9.1 (K)
- net Current_Sense_2: now also D10.1 (K)
- net Current_Sense_3: now also D11.1 (K)
- net Current_Sense_4: now also D12.1 (K)
- net GND: now also D10.2 (A), D11.2 (A), D12.2 (A), D9.2 (A)
Other:
- moved on the sheet: C10, C11, C12, C13, C14, C4, C8, C9, Conn4A, Conn4B, D13, D16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
