File: Hardware/ScienceMotorController/ScienceMotorController03a.sch (KiCad schematic (older format))
At the start: 17 parts, among them U8 VNH5019A_E

Commit message: assigned most of the footprints
Parts:
- Conn11: footprint (none) -> MRDT_Connectors:Anderson_2_Vertical_Sidy_by_Side
- D26: footprint (none) -> Diode_SMD:D_0603_1608Metric_Pad1.05x0.95mm_HandSolder
- D27, D28: value Blue_LED -> LED; footprint (none) -> LED_SMD:LED_0603_1608Metric_Pad1.05x0.95mm_HandSolder
- R55, R56, R57, R58, R59, R60, R61, R62, R63: footprint (none) -> Resistor_SMD:R_0603_1608Metric_Pad1.05x0.95mm_HandSolder
Other:
- note added: "Blue"
Changed lines of the file:
@@
 F 0 "R59" V 4750 3550 50  0000 C CNN
 F 1 "1k" V 4800 3700 50  0000 C CNN
-F 2 "" H 4800 3700 50  0001 C CNN
+F 2 "Resistor_SMD:R_0603_1608Metric_Pad1.05x0.95mm_HandSolder" H 4800 3700 50  0001 C CNN
 F 3 "~" H 4800 3700 50  0001 C CNN
 	1    4800 3700
@@
 F 0 "R56" V 4000 3950 50  0000 C CNN
 F 1 "1k" V 4100 3950 50  0000 C CNN
-F 2 "" H 4100 3950 50  0001 C CNN
+F 2 "Resistor_SMD:R_0603_1608Metric_Pad1.05x0.95mm_HandSolder" H 4100 3950 50  0001 C CNN
 F 3 "~" H 4100 3950 50  0001 C CNN
 	1    4100 3950
@@
 F 0 "D26" V 3300 3800 50  0000 R CNN
 F 1 "D_Zener_Small" V 3200 3850 50  0000 R CNN
-F 2 "" V 3250 3950 50  0001 C CNN
+F 2 "Diode_SMD:D_0603_1608Metric_Pad1.05x0.95mm_HandSolder" V 3250 3950 50  0001 C CNN
 F 3 "~" V 3250 3950 50  0001 C CNN
 	1    3250 3950
@@
 F 0 "R55" V 3700 3800 50  0000 C CNN
 F 1 "10k" V 3800 3800 50  0000 C CNN
-F 2 "" H 3800 3800 50  0001 C CNN
+F 2 "Resistor_SMD:R_0603_1608Metric_Pad1.05x0.95mm_HandSolder" H 3800 3800 50  0001 C CNN
 F 3 "~" H 3800 3800 50  0001 C CNN
 	1    3800 3800
@@
 F 0 "R60" V 4750 3750 50  0000 C CNN
 F 1 "1k" V 4800 3900 50  0000 C CNN
-F 2 "" H 4800 3900 50  0001 C CNN
+F 2 "Resistor_SMD:R_0603_1608Metric_Pad1.05x0.95mm_HandSolder" H 4800 3900 50  0001 C CNN
 F 3 "~" H 4800 3900 50  0001 C CNN
 	1    4800 3900
@@
 F 0 "R58" V 4750 3350 50  0000 C CNN
 F 1 "1k" V 4800 3500 50  0000 C CNN
-F 2 "" H 4800 3500 50  0001 C CNN
+F 2 "Resistor_SMD:R_0603_1608Metric_Pad1.05x0.95mm_HandSolder" H 4800 3500 50  0001 C CNN
 F 3 "~" H 4800 3500 50  0001 C CNN
 	1    4800 3500
@@
 F 0 "R57" V 4750 3250 50  0000 C CNN
 F 1 "1k" V 4800 3400 50  0000 C CNN
-F 2 "" H 4800 3400 50  0001 C CNN
+F 2 "Resistor_SMD:R_0603_1608Metric_Pad1.05x0.95mm_HandSolder" H 4800 3400 50  0001 C CNN
 F 3 "~" H 4800 3400 50  0001 C CNN
 	1    4800 3400
@@
 F 0 "R61" V 4750 3850 50  0000 C CNN
 F 1 "1k" V 4800 4000 50  0000 C CNN
-F 2 "" H 4800 4000 50  0001 C CNN
+F 2 "Resistor_SMD:R_0603_1608Metric_Pad1.05x0.95mm_HandSolder" H 4800 4000 50  0001 C CNN
 F 3 "~" H 4800 4000 50  0001 C CNN
 	1    4800 4000
@@
 F 0 "Conn11" H 7772 3097 60  0000 R CNN
 F 1 "AndersonPP" H 7772 3203 60  0000 R CNN
-F 2 "" H 7650 2500 60  0001 C CNN
+F 2 "MRDT_Connectors:Anderson_2_Vertical_Sidy_by_Side" H 7650 2500 60  0001 C CNN
 F 3 "" H 7650 2500 60  0001 C CNN
 	1    7800 3050
@@
 F 0 "Conn11" H 7772 2697 60  0000 R CNN
 F 1 "AndersonPP" H 7772 2803 60  0000 R CNN
-F 2 "" H 7650 2100 60  0001 C CNN
+F 2 "MRDT_Connectors:Anderson_2_Vertical_Sidy_by_Side" H 7650 2100 60  0001 C CNN
 F 3 "" H 7650 2100 60  0001 C CNN
 	2    7800 2650
@@
 AR Path="/5F7148FA/5FA34AD3/5FA3492F" Ref="D27"  Part="1"
 F 0 "D27" H 7650 2900 50  0000 C CNN
-F 1 "Blue_LED" H 7700 3000 31  0000 C CNN
-F 2 "" V 7550 2950 50  0001 C CNN
+F 1 "LED" H 7700 3000 31  0000 C CNN
+F 2 "LED_SMD:LED_0603_1608Metric_Pad1.05x0.95mm_HandSolder" V 7550 2950 50  0001 C CNN
 F 3 "~" V 7550 2950 50  0001 C CNN
 	1    7550 2950
@@
 AR Path="/5F7148FA/5FA34AD3/5FA34935" Ref="D28"  Part="1"
 F 0 "D28" H 7650 3300 50  0000 C CNN
-F 1 "Blue_LED" H 7700 3400 31  0000 C CNN
-F 2 "" V 7550 3350 50  0001 C CNN
+F 1 "LED" H 7700 3400 31  0000 C CNN
+F 2 "LED_SMD:LED_0603_1608Metric_Pad1.05x0.95mm_HandSolder" V 7550 3350 50  0001 C CNN
 F 3 "~" V 7550 3350 50  0001 C CNN
 	1    7550 3350
@@
 F 0 "R63" V 7750 3250 50  0000 C CNN
 F 1 "1.5k" V 7800 3350 39  0000 C CNN
-F 2 "" H 7800 3350 50  0001 C CNN
+F 2 "Resistor_SMD:R_0603_1608Metric_Pad1.05x0.95mm_HandSolder" H 7800 3350 50  0001 C CNN
 F 3 "~" H 7800 3350 50  0001 C CNN
 	1    7800 3350
@@
 F 0 "R62" V 7750 2850 50  0000 C CNN
 F 1 "1.5k" V 7800 2950 39  0000 C CNN
-F 2 "" H 7800 2950 50  0001 C CNN
+F 2 "Resistor_SMD:R_0603_1608Metric_Pad1.05x0.95mm_HandSolder" H 7800 2950 50  0001 C CNN
 F 3 "~" H 7800 2950 50  0001 C CNN
 	1    7800 2950
@@
 Text HLabel 4550 3900 0    50   Output ~ 0
 3.3V
+Text Notes 7350 3050 0    20   ~ 0
+Blue
+Text Notes 7350 3450 0    20   ~ 0
+Blue
 $EndSCHEMATC
