File: Hardware/ScienceMotorController/ScienceMotorController03d.sch (KiCad schematic (older format))
At the start: 17 parts, among them U5 VNH5019A_E

Commit message: assigned most of the footprints
Parts:
- Conn4: footprint (none) -> MRDT_Connectors:Anderson_2_Vertical_Sidy_by_Side
- D13: footprint (none) -> Diode_SMD:D_0603_1608Metric_Pad1.05x0.95mm_HandSolder
- D14, D15: value Blue_LED -> LED; footprint (none) -> LED_SMD:LED_0603_1608Metric_Pad1.05x0.95mm_HandSolder
- R24, R25, R26, R27, R28, R29, R30, R31, R32: footprint (none) -> Resistor_SMD:R_0603_1608Metric_Pad1.05x0.95mm_HandSolder
Other:
- note added: "Blue"
Changed lines of the file:
@@
 F 0 "R28" V 4850 3900 50  0000 C CNN
 F 1 "1k" V 4900 4050 50  0000 C CNN
-F 2 "" H 4900 4050 50  0001 C CNN
+F 2 "Resistor_SMD:R_0603_1608Metric_Pad1.05x0.95mm_HandSolder" H 4900 4050 50  0001 C CNN
 F 3 "~" H 4900 4050 50  0001 C CNN
 	1    4900 4050
@@
 F 0 "R25" V 4100 4300 50  0000 C CNN
 F 1 "1k" V 4200 4300 50  0000 C CNN
-F 2 "" H 4200 4300 50  0001 C CNN
+F 2 "Resistor_SMD:R_0603_1608Metric_Pad1.05x0.95mm_HandSolder" H 4200 4300 50  0001 C CNN
 F 3 "~" H 4200 4300 50  0001 C CNN
 	1    4200 4300
@@
 F 0 "D13" V 3400 4150 50  0000 R CNN
 F 1 "D_Zener_Small" V 3300 4200 50  0000 R CNN
-F 2 "" V 3350 4300 50  0001 C CNN
+F 2 "Diode_SMD:D_0603_1608Metric_Pad1.05x0.95mm_HandSolder" V 3350 4300 50  0001 C CNN
 F 3 "~" V 3350 4300 50  0001 C CNN
 	1    3350 4300
@@
 F 0 "R24" V 3800 4150 50  0000 C CNN
 F 1 "10k" V 3900 4150 50  0000 C CNN
-F 2 "" H 3900 4150 50  0001 C CNN
+F 2 "Resistor_SMD:R_0603_1608Metric_Pad1.05x0.95mm_HandSolder" H 3900 4150 50  0001 C CNN
 F 3 "~" H 3900 4150 50  0001 C CNN
 	1    3900 4150
@@
 F 0 "R29" V 4850 4100 50  0000 C CNN
 F 1 "1k" V 4900 4250 50  0000 C CNN
-F 2 "" H 4900 4250 50  0001 C CNN
+F 2 "Resistor_SMD:R_0603_1608Metric_Pad1.05x0.95mm_HandSolder" H 4900 4250 50  0001 C CNN
 F 3 "~" H 4900 4250 50  0001 C CNN
 	1    4900 4250
@@
 F 0 "R27" V 4850 3700 50  0000 C CNN
 F 1 "1k" V 4900 3850 50  0000 C CNN
-F 2 "" H 4900 3850 50  0001 C CNN
+F 2 "Resistor_SMD:R_0603_1608Metric_Pad1.05x0.95mm_HandSolder" H 4900 3850 50  0001 C CNN
 F 3 "~" H 4900 3850 50  0001 C CNN
 	1    4900 3850
@@
 F 0 "R26" V 4850 3600 50  0000 C CNN
 F 1 "1k" V 4900 3750 50  0000 C CNN
-F 2 "" H 4900 3750 50  0001 C CNN
+F 2 "Resistor_SMD:R_0603_1608Metric_Pad1.05x0.95mm_HandSolder" H 4900 3750 50  0001 C CNN
 F 3 "~" H 4900 3750 50  0001 C CNN
 	1    4900 3750
@@
 F 0 "R30" V 4850 4200 50  0000 C CNN
 F 1 "1k" V 4900 4350 50  0000 C CNN
-F 2 "" H 4900 4350 50  0001 C CNN
+F 2 "Resistor_SMD:R_0603_1608Metric_Pad1.05x0.95mm_HandSolder" H 4900 4350 50  0001 C CNN
 F 3 "~" H 4900 4350 50  0001 C CNN
 	1    4900 4350
@@
 F 0 "Conn4" H 7922 3447 60  0000 R CNN
 F 1 "AndersonPP" H 7922 3553 60  0000 R CNN
-F 2 "" H 7800 2850 60  0001 C CNN
+F 2 "MRDT_Connectors:Anderson_2_Vertical_Sidy_by_Side" H 7800 2850 60  0001 C CNN
 F 3 "" H 7800 2850 60  0001 C CNN
 	1    7950 3400
@@
 F 0 "Conn4" H 7922 3047 60  0000 R CNN
 F 1 "AndersonPP" H 7922 3153 60  0000 R CNN
-F 2 "" H 7800 2450 60  0001 C CNN
+F 2 "MRDT_Connectors:Anderson_2_Vertical_Sidy_by_Side" H 7800 2450 60  0001 C CNN
 F 3 "" H 7800 2450 60  0001 C CNN
 	2    7950 3000
@@
 AR Path="/5F7148FA/5FA34AD9/5FA978D1" Ref="D14"  Part="1"
 F 0 "D14" H 7800 3250 50  0000 C CNN
-F 1 "Blue_LED" H 7850 3350 31  0000 C CNN
-F 2 "" V 7700 3300 50  0001 C CNN
+F 1 "LED" H 7850 3350 31  0000 C CNN
+F 2 "LED_SMD:LED_0603_1608Metric_Pad1.05x0.95mm_HandSolder" V 7700 3300 50  0001 C CNN
 F 3 "~" V 7700 3300 50  0001 C CNN
 	1    7700 3300
@@
 AR Path="/5F7148FA/5FA34AD9/5FA978D7" Ref="D15"  Part="1"
 F 0 "D15" H 7800 3650 50  0000 C CNN
-F 1 "Blue_LED" H 7850 3750 31  0000 C CNN
-F 2 "" V 7700 3700 50  0001 C CNN
+F 1 "LED" H 7850 3750 31  0000 C CNN
+F 2 "LED_SMD:LED_0603_1608Metric_Pad1.05x0.95mm_HandSolder" V 7700 3700 50  0001 C CNN
 F 3 "~" V 7700 3700 50  0001 C CNN
 	1    7700 3700
@@
 F 0 "R32" V 7900 3600 50  0000 C CNN
 F 1 "1.5k" V 7950 3700 39  0000 C CNN
-F 2 "" H 7950 3700 50  0001 C CNN
+F 2 "Resistor_SMD:R_0603_1608Metric_Pad1.05x0.95mm_HandSolder" H 7950 3700 50  0001 C CNN
 F 3 "~" H 7950 3700 50  0001 C CNN
 	1    7950 3700
@@
 F 0 "R31" V 7900 3200 50  0000 C CNN
 F 1 "1.5k" V 7950 3300 39  0000 C CNN
-F 2 "" H 7950 3300 50  0001 C CNN
+F 2 "Resistor_SMD:R_0603_1608Metric_Pad1.05x0.95mm_HandSolder" H 7950 3300 50  0001 C CNN
 F 3 "~" H 7950 3300 50  0001 C CNN
 	1    7950 3300
@@
 Text HLabel 4650 4250 0    50   Output ~ 0
 3.3V
+Text Notes 7500 3400 0    20   ~ 0
+Blue
+Text Notes 7500 3800 0    20   ~ 0
+Blue
 $EndSCHEMATC
