File: Hardware/ScienceMotorController/ScienceMotorController03e.sch (KiCad schematic (older format))
At the start: 17 parts, among them U6 VNH5019A_E

Commit message: assigned most of the footprints
Parts:
- Conn5: footprint (none) -> MRDT_Connectors:Anderson_2_Vertical_Sidy_by_Side
- D16: footprint (none) -> Diode_SMD:D_0603_1608Metric_Pad1.05x0.95mm_HandSolder
- D17, D18: value Blue_LED -> LED; footprint (none) -> LED_SMD:LED_0603_1608Metric_Pad1.05x0.95mm_HandSolder
- R33, R34, R35, R36, R37, R38, R39, R40, R41: footprint (none) -> Resistor_SMD:R_0603_1608Metric_Pad1.05x0.95mm_HandSolder
Other:
- note added: "Blue"
Changed lines of the file:
@@
 F 0 "R37" V 4400 3750 50  0000 C CNN
 F 1 "1k" V 4450 3900 50  0000 C CNN
-F 2 "" H 4450 3900 50  0001 C CNN
+F 2 "Resistor_SMD:R_0603_1608Metric_Pad1.05x0.95mm_HandSolder" H 4450 3900 50  0001 C CNN
 F 3 "~" H 4450 3900 50  0001 C CNN
 	1    4450 3900
@@
 F 0 "R34" V 3650 4150 50  0000 C CNN
 F 1 "1k" V 3750 4150 50  0000 C CNN
-F 2 "" H 3750 4150 50  0001 C CNN
+F 2 "Resistor_SMD:R_0603_1608Metric_Pad1.05x0.95mm_HandSolder" H 3750 4150 50  0001 C CNN
 F 3 "~" H 3750 4150 50  0001 C CNN
 	1    3750 4150
@@
 F 0 "D16" V 2950 4000 50  0000 R CNN
 F 1 "D_Zener_Small" V 2850 4050 50  0000 R CNN
-F 2 "" V 2900 4150 50  0001 C CNN
+F 2 "Diode_SMD:D_0603_1608Metric_Pad1.05x0.95mm_HandSolder" V 2900 4150 50  0001 C CNN
 F 3 "~" V 2900 4150 50  0001 C CNN
 	1    2900 4150
@@
 F 0 "R33" V 3350 4000 50  0000 C CNN
 F 1 "10k" V 3450 4000 50  0000 C CNN
-F 2 "" H 3450 4000 50  0001 C CNN
+F 2 "Resistor_SMD:R_0603_1608Metric_Pad1.05x0.95mm_HandSolder" H 3450 4000 50  0001 C CNN
 F 3 "~" H 3450 4000 50  0001 C CNN
 	1    3450 4000
@@
 F 0 "R38" V 4400 3950 50  0000 C CNN
 F 1 "1k" V 4450 4100 50  0000 C CNN
-F 2 "" H 4450 4100 50  0001 C CNN
+F 2 "Resistor_SMD:R_0603_1608Metric_Pad1.05x0.95mm_HandSolder" H 4450 4100 50  0001 C CNN
 F 3 "~" H 4450 4100 50  0001 C CNN
 	1    4450 4100
@@
 F 0 "R36" V 4400 3550 50  0000 C CNN
 F 1 "1k" V 4450 3700 50  0000 C CNN
-F 2 "" H 4450 3700 50  0001 C CNN
+F 2 "Resistor_SMD:R_0603_1608Metric_Pad1.05x0.95mm_HandSolder" H 4450 3700 50  0001 C CNN
 F 3 "~" H 4450 3700 50  0001 C CNN
 	1    4450 3700
@@
 F 0 "R35" V 4400 3450 50  0000 C CNN
 F 1 "1k" V 4450 3600 50  0000 C CNN
-F 2 "" H 4450 3600 50  0001 C CNN
+F 2 "Resistor_SMD:R_0603_1608Metric_Pad1.05x0.95mm_HandSolder" H 4450 3600 50  0001 C CNN
 F 3 "~" H 4450 3600 50  0001 C CNN
 	1    4450 3600
@@
 F 0 "R39" V 4400 4050 50  0000 C CNN
 F 1 "1k" V 4450 4200 50  0000 C CNN
-F 2 "" H 4450 4200 50  0001 C CNN
+F 2 "Resistor_SMD:R_0603_1608Metric_Pad1.05x0.95mm_HandSolder" H 4450 4200 50  0001 C CNN
 F 3 "~" H 4450 4200 50  0001 C CNN
 	1    4450 4200
@@
 F 0 "Conn5" H 7472 3297 60  0000 R CNN
 F 1 "AndersonPP" H 7472 3403 60  0000 R CNN
-F 2 "" H 7350 2700 60  0001 C CNN
+F 2 "MRDT_Connectors:Anderson_2_Vertical_Sidy_by_Side" H 7350 2700 60  0001 C CNN
 F 3 "" H 7350 2700 60  0001 C CNN
 	1    7500 3250
@@
 F 0 "Conn5" H 7472 2897 60  0000 R CNN
 F 1 "AndersonPP" H 7472 3003 60  0000 R CNN
-F 2 "" H 7350 2300 60  0001 C CNN
+F 2 "MRDT_Connectors:Anderson_2_Vertical_Sidy_by_Side" H 7350 2300 60  0001 C CNN
 F 3 "" H 7350 2300 60  0001 C CNN
 	2    7500 2850
@@
 AR Path="/5F7148FA/5FA34ADB/5FAB369A" Ref="D17"  Part="1"
 F 0 "D17" H 7350 3100 50  0000 C CNN
-F 1 "Blue_LED" H 7400 3200 31  0000 C CNN
-F 2 "" V 7250 3150 50  0001 C CNN
+F 1 "LED" H 7400 3200 31  0000 C CNN
+F 2 "LED_SMD:LED_0603_1608Metric_Pad1.05x0.95mm_HandSolder" V 7250 3150 50  0001 C CNN
 F 3 "~" V 7250 3150 50  0001 C CNN
 	1    7250 3150
@@
 AR Path="/5F7148FA/5FA34ADB/5FAB36A0" Ref="D18"  Part="1"
 F 0 "D18" H 7350 3500 50  0000 C CNN
-F 1 "Blue_LED" H 7400 3600 31  0000 C CNN
-F 2 "" V 7250 3550 50  0001 C CNN
+F 1 "LED" H 7400 3600 31  0000 C CNN
+F 2 "LED_SMD:LED_0603_1608Metric_Pad1.05x0.95mm_HandSolder" V 7250 3550 50  0001 C CNN
 F 3 "~" V 7250 3550 50  0001 C CNN
 	1    7250 3550
@@
 F 0 "R41" V 7450 3450 50  0000 C CNN
 F 1 "1.5k" V 7500 3550 39  0000 C CNN
-F 2 "" H 7500 3550 50  0001 C CNN
+F 2 "Resistor_SMD:R_0603_1608Metric_Pad1.05x0.95mm_HandSolder" H 7500 3550 50  0001 C CNN
 F 3 "~" H 7500 3550 50  0001 C CNN
 	1    7500 3550
@@
 F 0 "R40" V 7450 3050 50  0000 C CNN
 F 1 "1.5k" V 7500 3150 39  0000 C CNN
-F 2 "" H 7500 3150 50  0001 C CNN
+F 2 "Resistor_SMD:R_0603_1608Metric_Pad1.05x0.95mm_HandSolder" H 7500 3150 50  0001 C CNN
 F 3 "~" H 7500 3150 50  0001 C CNN
 	1    7500 3150
@@
 Text HLabel 4200 4100 0    50   Output ~ 0
 3.3V
+Text Notes 7050 3650 0    20   ~ 0
+Blue
+Text Notes 7050 3250 0    20   ~ 0
+Blue
 $EndSCHEMATC
