File: Hardware/ScienceMotorController/ScienceMotorController05.sch (KiCad schematic (older format))
At the start: 2 parts

Commit message: annotated
Parts:
- gave numbers to parts that had none: 2
Changed lines of the file:
@@
 $EndDescr
 $Comp
-L MRDT_Connectors:Molex_SL_03 Conn?
+L MRDT_Connectors:Molex_SL_03 Conn12
 U 1 1 5FA2AB8E
 P 6050 2850
-F 0 "Conn?" H 6178 3058 60  0000 L CNN
+F 0 "Conn12" H 6178 3058 60  0000 L CNN
 F 1 "Molex_SL_03" H 6178 2952 60  0000 L CNN
 F 2 "" H 6050 2850 60  0001 C CNN
@@
 $EndComp
 $Comp
-L MRDT_Connectors:Molex_SL_03 Conn?
+L MRDT_Connectors:Molex_SL_03 Conn13
 U 1 1 5FA2C457
 P 6050 3350
-F 0 "Conn?" H 6178 3558 60  0000 L CNN
+F 0 "Conn13" H 6178 3558 60  0000 L CNN
 F 1 "Molex_SL_03" H 6178 3452 60  0000 L CNN
 F 2 "" H 6050 3350 60  0001 C CNN
@@
 Connection ~ 5700 2600
 $Comp
-L power:GND #PWR?
+L power:GND #PWR050
 U 1 1 5FA2F0EE
 P 5650 3450
-F 0 "#PWR?" H 5650 3200 50  0001 C CNN
+F 0 "#PWR050" H 5650 3200 50  0001 C CNN
 F 1 "GND" H 5655 3277 50  0000 C CNN
 F 2 "" H 5650 3450 50  0001 C CNN

Commit message: assigned most of the footprints
Parts:
- Conn12, Conn13: footprint (none) -> MRDT_Connectors:MOLEX_SL_03_Vertical
Changed lines of the file:
@@
 F 0 "Conn12" H 6178 3058 60  0000 L CNN
 F 1 "Molex_SL_03" H 6178 2952 60  0000 L CNN
-F 2 "" H 6050 2850 60  0001 C CNN
+F 2 "MRDT_Connectors:MOLEX_SL_03_Vertical" H 6050 2850 60  0001 C CNN
 F 3 "" H 6050 2850 60  0001 C CNN
 	1    6050 2850
@@
 F 0 "Conn13" H 6178 3558 60  0000 L CNN
 F 1 "Molex_SL_03" H 6178 3452 60  0000 L CNN
-F 2 "" H 6050 3350 60  0001 C CNN
+F 2 "MRDT_Connectors:MOLEX_SL_03_Vertical" H 6050 3350 60  0001 C CNN
 F 3 "" H 6050 3350 60  0001 C CNN
 	1    6050 3350

Commit message: running traces
Parts:
- renumbered Conn12 to Conn13, Conn13 to Conn14
Changed lines of the file:
@@
 $EndDescr
 $Comp
-L MRDT_Connectors:Molex_SL_03 Conn12
+L MRDT_Connectors:Molex_SL_03 Conn13
 U 1 1 5FA2AB8E
 P 6050 2850
-F 0 "Conn12" H 6178 3058 60  0000 L CNN
+F 0 "Conn13" H 6178 3058 60  0000 L CNN
 F 1 "Molex_SL_03" H 6178 2952 60  0000 L CNN
 F 2 "MRDT_Connectors:MOLEX_SL_03_Vertical" H 6050 2850 60  0001 C CNN
@@
 $EndComp
 $Comp
-L MRDT_Connectors:Molex_SL_03 Conn13
+L MRDT_Connectors:Molex_SL_03 Conn14
 U 1 1 5FA2C457
 P 6050 3350
-F 0 "Conn13" H 6178 3558 60  0000 L CNN
+F 0 "Conn14" H 6178 3558 60  0000 L CNN
 F 1 "Molex_SL_03" H 6178 3452 60  0000 L CNN
 F 2 "MRDT_Connectors:MOLEX_SL_03_Vertical" H 6050 3350 60  0001 C CNN
