File: Hardware/ScienceMotorController/_autosave-ScienceMotorController.sch (KiCad schematic (older format))
At the start: 127 parts, among them U1 LT1910, U10 OKI, U11 OKI, U12 TB67H400AFNG,EL, U13 TB67H400AFNG,EL, U14 LT1910, U15 PMN280ENEAX, U16 PMN280ENEAX, U17 LTC6900, U2 OKI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

Commit message: Created PCB and Put Close Components Near Each other
Parts:
- Conn1: value Motor_5 -> Motor_X
- Conn2: value Motor_5 -> Motor_Y
- Conn3: value Motor_5 -> Motor_D
- Conn4: value Motor_5 -> Motor_1
- Conn5: value Motor_5 -> Motor_2
- Conn6: value Motor_5 -> Motor_S
Changed lines of the file:
@@
 P 6800 4600
 F 0 "Conn1" H 6772 4753 60  0000 R CNN
-F 1 "Motor_5" H 6772 4647 60  0000 R CNN
+F 1 "Motor_X" H 6772 4647 60  0000 R CNN
 F 2 "MRDT_Connectors:Anderson_2_Horizontal_Side_by_Side" H 6650 4050 60  0001 C CNN
 F 3 "" H 6650 4050 60  0001 C CNN
@@
 P 3100 4400
 F 0 "Conn1" H 3072 4447 60  0000 R CNN
-F 1 "Motor_5" H 3072 4553 60  0000 R CNN
+F 1 "Motor_X" H 3072 4553 60  0000 R CNN
 F 2 "MRDT_Connectors:Anderson_2_Horizontal_Side_by_Side" H 2950 3850 60  0001 C CNN
 F 3 "" H 2950 3850 60  0001 C CNN
@@
 P 6800 7950
 F 0 "Conn4" H 6772 8103 60  0000 R CNN
-F 1 "Motor_5" H 6772 7997 60  0000 R CNN
+F 1 "Motor_1" H 6772 7997 60  0000 R CNN
 F 2 "MRDT_Connectors:Anderson_2_Horizontal_Side_by_Side" H 6650 7400 60  0001 C CNN
 F 3 "" H 6650 7400 60  0001 C CNN
@@
 P 3100 7750
 F 0 "Conn4" H 3072 7797 60  0000 R CNN
-F 1 "Motor_5" H 3072 7903 60  0000 R CNN
+F 1 "Motor_1" H 3072 7903 60  0000 R CNN
 F 2 "MRDT_Connectors:Anderson_2_Horizontal_Side_by_Side" H 2950 7200 60  0001 C CNN
 F 3 "" H 2950 7200 60  0001 C CNN
@@
 P 12700 4600
 F 0 "Conn2" H 12672 4753 60  0000 R CNN
-F 1 "Motor_5" H 12672 4647 60  0000 R CNN
+F 1 "Motor_Y" H 12672 4647 60  0000 R CNN
 F 2 "MRDT_Connectors:Anderson_2_Horizontal_Side_by_Side" H 12550 4050 60  0001 C CNN
 F 3 "" H 12550 4050 60  0001 C CNN
@@
 P 9000 4400
 F 0 "Conn2" H 8972 4447 60  0000 R CNN
-F 1 "Motor_5" H 8972 4553 60  0000 R CNN
+F 1 "Motor_Y" H 8972 4553 60  0000 R CNN
 F 2 "MRDT_Connectors:Anderson_2_Horizontal_Side_by_Side" H 8850 3850 60  0001 C CNN
 F 3 "" H 8850 3850 60  0001 C CNN
@@
 P 12700 7950
 F 0 "Conn5" H 12672 8103 60  0000 R CNN
-F 1 "Motor_5" H 12672 7997 60  0000 R CNN
+F 1 "Motor_2" H 12672 7997 60  0000 R CNN
 F 2 "MRDT_Connectors:Anderson_2_Horizontal_Side_by_Side" H 12550 7400 60  0001 C CNN
 F 3 "" H 12550 7400 60  0001 C CNN
@@
 P 9000 7750
 F 0 "Conn5" H 8972 7797 60  0000 R CNN
-F 1 "Motor_5" H 8972 7903 60  0000 R CNN
+F 1 "Motor_2" H 8972 7903 60  0000 R CNN
 F 2 "MRDT_Connectors:Anderson_2_Horizontal_Side_by_Side" H 8850 7200 60  0001 C CNN
 F 3 "" H 8850 7200 60  0001 C CNN
@@
 P 18650 4600
 F 0 "Conn3" H 18622 4753 60  0000 R CNN
-F 1 "Motor_5" H 18622 4647 60  0000 R CNN
+F 1 "Motor_D" H 18622 4647 60  0000 R CNN
 F 2 "MRDT_Connectors:Anderson_2_Horizontal_Side_by_Side" H 18500 4050 60  0001 C CNN
 F 3 "" H 18500 4050 60  0001 C CNN
@@
 P 14950 4400
 F 0 "Conn3" H 14922 4447 60  0000 R CNN
-F 1 "Motor_5" H 14922 4553 60  0000 R CNN
+F 1 "Motor_D" H 14922 4553 60  0000 R CNN
 F 2 "MRDT_Connectors:Anderson_2_Horizontal_Side_by_Side" H 14800 3850 60  0001 C CNN
 F 3 "" H 14800 3850 60  0001 C CNN
@@
 P 18650 8100
 F 0 "Conn6" H 18622 8253 60  0000 R CNN
-F 1 "Motor_5" H 18622 8147 60  0000 R CNN
+F 1 "Motor_S" H 18622 8147 60  0000 R CNN
 F 2 "MRDT_Connectors:Anderson_2_Horizontal_Side_by_Side" H 18500 7550 60  0001 C CNN
 F 3 "" H 18500 7550 60  0001 C CNN
@@
 P 14950 7900
 F 0 "Conn6" H 14922 7947 60  0000 R CNN
-F 1 "Motor_5" H 14922 8053 60  0000 R CNN
+F 1 "Motor_S" H 14922 8053 60  0000 R CNN
 F 2 "MRDT_Connectors:Anderson_2_Horizontal_Side_by_Side" H 14800 7350 60  0001 C CNN
 F 3 "" H 14800 7350 60  0001 C CNN
