File: Hardware/ScienceMotorController/ScienceMotorController.kicad_sch (KiCad schematic)
At the start: 197 parts, among them J1 RJ45_LED_Shielded, Q1 SI4156DY, Q10 AO3401A, Q11 SI4156DY, Q12 SI4156DY, Q13 SI4156DY, Q14 SI4156DY, Q15 SI4156DY, Q16 SI4156DY, Q17 SI4156DY, Q18 SI4156DY, Q2 SI4156DY, Q3 SI4156DY, Q4 SI4156DY, Q5 SI4156DY, Q6 SI4156DY, Q7 SI4156DY, Q8 SI4156DY, Q9 BSS138, SW1 SW_Push, SW11 SW_DPDT_x2, SW2 SW_Push, SW3 SW_Push, SW4 SW_Push, SW5 SW_Push, SW6 SW_Push, SW7 SW_Push, SW8 SW_Push, SW9 SW_Push, U1 74LVC2G04, U10 IRS2005S, U11 IRS2005S, U12 Teensy4.1_DEV-16771, U13 IRS2005S, U14 IRS2005S, U2 74LVC2G04, U3 IRS2005S, U4 IRS2005S, U5 TSR_1-2450, U6 IRS2005S, U7 IRS2005S, U8 74LVC2G04, U9 74LVC2G04

Commit message: Board was Reviewed
Parts:
- SW1, SW2, SW3, SW4, SW5, SW6, SW7, SW8, SW9: footprint Button_Switch_SMD:SW_SPST_EVPBF -> Button_Switch_SMD:SW_SPST_TL3305A
Connections:
- net Limit_Switch_4: now also U12.37 (CS3); no longer U12.33 (MCLK2)
- net Limit_Switch_5: now also U12.36 (CS2); no longer U12.34 (RX8)
- net Limit_Switch_7: now also U12.34 (RX8); no longer U12.36 (CS2)
- net Limit_Switch_8: now also U12.33 (MCLK2); no longer U12.37 (CS3)
- net Manual_Control_Left: now also U12.17 (A3); no longer U12.21 (A7)
- net Manual_Control_Right: now also U12.16 (A2); no longer U12.20 (A6)
