File: Hardware/ScienceMocoBoard_1.01/ScienceMocoBoard_1.01.kicad_sch (KiCad schematic)
At the start: 157 parts, among them Q1 BSS138, Q10 SI4156DY, Q11 SI4156DY, Q12 SI4156DY, Q13 SI4156DY, Q14 BSS138, Q15 BSS138, Q16 BSS138, Q17 BSS138, Q18 SI4156DY, Q19 SI4156DY, Q2 BSS138, Q20 SI4156DY, Q21 SI4156DY, Q22 SI4156DY, Q23 SI4156DY, Q24 SI4156DY, Q25 SI4156DY, Q3 BSS138, Q4 SI4156DY, Q5 SI4156DY, Q6 SI4156DY, Q7 SI4156DY, Q8 BSS138, Q9 BSS138, U1 IRS2005S, U10 IRS2005S, U11 IRS2005S, U12 IRS2005S, U2 IRS2005S, U3 3V3 OKI, U4 5VA OKI, U5 5VA OKI, U6 IRS2005S, U7 IRS2005S, U8 TM4C129E_Launchpad, U9 IRS2005S

Commit message: Moved LED to motor outputs
Parts:
- removed D12, D13, D21, D23, D6, D7: BLUE, LED_SMD:LED_0603_1608Metric_Pad1.05x0.95mm_HandSolder, symbol Device:LED
- removed Q4, Q5, Q6, Q7: SI4156DY, Package_SO:SOIC-8_3.9x4.9mm_P1.27mm, symbol Transistor_FET:FDS2734
- added D12, D13, D35, D36, D37, D38, D6, D7: Pink, symbol Device:LED_Small
- added D21, D23, D39, D40: D_Small, symbol Device:D_Small
- added D31, D32, D33, D34, D41, D42: BLUE, LED_SMD:LED_0603_1608Metric_Pad1.05x0.95mm_HandSolder, symbol Device:LED
- added Q26, Q27, Q28, Q29, Q4, Q5, Q6, Q7: BSS138, Package_TO_SOT_SMD:SOT-23, symbol Transistor_FET:BSS138
- added Q30, Q31, Q32, Q33: SI4156DY, Package_SO:SOIC-8_3.9x4.9mm_P1.27mm, symbol Transistor_FET:FDS2734
- added R47, R48: 1k, Resistor_SMD:R_0603_1608Metric_Pad0.98x0.95mm_HandSolder, symbol Device:R
- added R49, R50, R53, R54: 100, Resistor_SMD:R_0603_1608Metric_Pad0.98x0.95mm_HandSolder, symbol Device:R
- added R51, R52: 1K, Resistor_SMD:R_0603_1608Metric_Pad0.98x0.95mm_HandSolder, symbol Device:R
- R14, R15, R16, R17, R33, R35: value 1K -> 100
- R19, R20, R21, R22: value 100 -> 1K
- R37, R38, R5, R6, R7, R8: value 100 -> 1k
Connections:
- net +12V: now also D12.2 (A), D13.2 (A), D21.2 (A), D23.2 (A), D35.2 (A), D36.2 (A), D37.2 (A), D38.2 (A), D39.2 (A), D40.2 (A), D6.2 (A), D7.2 (A), Q30.5 (D), Q30.6 (D), Q30.7 (D), Q30.8 (D), Q32.5 (D), Q32.6 (D), Q32.7 (D), Q32.8 (D); no longer C1.1, C11.1, C12.1, C2.1, U1.8 (VB), U10.8 (VB), U2.8 (VB), U9.8 (VB)
- net FWD_PWM_1: now also Q4.1 (G)
- net FWD_PWM_2: now also Q5.1 (G)
- net FWD_PWM_3: now also U9.2 (HIN), Q26.1 (G); no longer U10.2 (HIN)
- net FWD_PWM_4: now also U10.2 (HIN), Q27.1 (G); no longer U9.2 (HIN)
- net GND: now also R19.2, R20.2, R21.2, R22.2, Q26.2 (S), Q27.2 (S), Q28.2 (S), Q29.2 (S), Q31.1 (S), Q31.2 (S), Q31.3 (S), Q33.1 (S), Q33.2 (S), Q33.3 (S), Q4.2 (S), Q5.2 (S), Q6.2 (S), Q7.2 (S), R51.2, R52.2; no longer R14.2, R15.2, R16.2, R17.2, R33.2, R35.2
- net M+: now also Q10.1 (S), Q10.2 (S), Q10.3 (S), Q11.5 (D), Q11.6 (D), Q11.7 (D), Q11.8 (D), Q12.1 (S), Q12.2 (S), Q12.3 (S), Q13.5 (D), Q13.6 (D), Q13.7 (D), Q13.8 (D), D31.2 (A), D32.2 (A), D41.2 (A), Q30.1 (S), Q30.2 (S), Q30.3 (S), Q31.5 (D), Q31.6 (D), Q31.7 (D), Q31.8 (D); no longer Q18.1 (S), Q18.2 (S), Q18.3 (S), Q19.5 (D), Q19.6 (D), Q19.7 (D), Q19.8 (D)
- net M-: now also Q18.1 (S), Q18.2 (S), Q18.3 (S), Q19.5 (D), Q19.6 (D), Q19.7 (D), Q19.8 (D), D33.2 (A), D34.2 (A), D42.2 (A), Q32.1 (S), Q32.2 (S), Q32.3 (S), Q33.5 (D), Q33.6 (D), Q33.7 (D), Q33.8 (D); no longer Q10.1 (S), Q10.2 (S), Q10.3 (S), Q11.5 (D), Q11.6 (D), Q11.7 (D), Q11.8 (D), Q12.1 (S), Q12.2 (S), Q12.3 (S), Q13.5 (D), Q13.6 (D), Q13.7 (D), Q13.8 (D)
- net RVS_PWM_1: now also Q6.1 (G)
- net RVS_PWM_2: now also Q7.1 (G)
- net RVS_PWM_3: now also U9.3 (LIN), Q28.1 (G); no longer U10.3 (LIN)
- net RVS_PWM_4: now also U10.3 (LIN), Q29.1 (G); no longer U9.3 (LIN)
- net at R35.1: now also U7.5 (LO)
- net at R8.1: now also Q7.3 (D); no longer U2.5 (LO)
- net at R8.2: now also D13.1 (K)
- net at R32.1: now also U9.5 (LO); no longer U10.5 (LO)
- net at R16.1: now also U2.7 (HO)
- net at R29.1: now also U6.5 (LO); no longer U9.5 (LO)
- net at U9.7 (HO): now also R31.1; no longer R28.1
- net at Q10.4 (G): now also R14.2; no longer R19.2
- net at U10.7 (HO): now also R49.1; no longer R31.1
- net at R22.1: now also D32.1 (K); no longer U7.5 (LO)
- net at U7.7 (HO): now also R33.1; no longer R21.1
- net at Q23.4 (G): now also R35.2; no longer R38.2
- net at Q13.4 (G): now also R17.2; no longer R22.2
- net at R38.1: now also Q27.3 (D); no longer U11.5 (LO)
- net at R17.1: now also U2.5 (LO)
- net at Q22.4 (G): now also R33.2; no longer R37.2
- net at R7.2: now also D12.1 (K)
- net at U1.5 (LO): now also R15.1; no longer R6.1
- net at U1.7 (HO): now also R14.1; no longer R5.1
- net at Q12.4 (G): now also R16.2; no longer R21.2
- net at R20.1: now also D34.1 (K); no longer U6.5 (LO)
- net at Q11.4 (G): now also R15.2; no longer R20.2
- net at R5.2: now also D6.1 (K)
- net at R6.2: now also D7.1 (K)
- net at R7.1: now also Q6.3 (D); no longer U2.7 (HO)
- net at R19.1: now also D33.1 (K); no longer U6.7 (HO)
- net at R37.1: now also Q26.3 (D); no longer U11.7 (HO)
- new net: C1.1, D21.1 (K), U1.8 (VB)
- new net: D41.1 (K), R52.1
- new net: C12.1, D39.1 (K), U9.8 (VB)
- new net: C2.1, D23.1 (K), U2.8 (VB)
- new net: D42.1 (K), R51.1
- new net: D38.1 (K), R48.2
- new net: C11.1, D40.1 (K), U10.8 (VB)
- new net: R50.1, U10.5 (LO)
- new net: Q31.4 (G), R50.2
- new net: Q28.3 (D), R47.1
- new net: D37.1 (K), R47.2
- new net: Q33.4 (G), R54.2
- new net: Q29.3 (D), R48.1
- new net: R28.1, U6.7 (HO)
- new net: Q30.4 (G), R49.2
- new net: D31.1 (K), R21.1
- new net: Q32.4 (G), R53.2
- new net: Q4.3 (D), R5.1
- new net: Q5.3 (D), R6.1
- new net: D36.1 (K), R38.2
- new net: D35.1 (K), R37.2
- new net: R54.1, U11.5 (LO)
- new net: R53.1, U11.7 (HO)
Other:
- moved on the sheet: C12, C14, Conn7A, Conn7B, D22, D24, Q20, Q21, Q24, Q25, R31, R32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
