File: Hardware/ScienceMocoBoard_V1/ScienceMotorController_Hardware_2023.kicad_sch (KiCad schematic)
At the start: 166 parts, among them Q1 BSS138, Q10 SI4156DY, Q11 SI4156DY, Q12 SI4156DY, Q13 SI4156DY, Q14 SI4156DY, Q15 SI4156DY, Q16 SI4156DY, Q17 SI4156DY, Q18 SI4156DY, Q19 SI4156DY, Q2 BSS138, Q20 SI4156DY, Q21 SI4156DY, Q22 SI4156DY, Q23 SI4156DY, Q24 SI4156DY, Q25 SI4156DY, Q3 BSS138, Q4 BSS138, Q5 BSS138, Q6 BSS138, Q7 BSS138, Q8 BSS138, Q9 BSS138, U1 3V3 OKI, U10 IRS2005S, U11 IRS2005S, U2 TSR_1-2450, U3 TM4C129E_Launchpad, U4 IRS2005S, U5 IRS2005S, U6 IRS2005S, U7 IRS2005S, U8 IRS2005S, U9 IRS2005S

Commit message: Updated Motor Controllers
Now has 7 motor controllers. Relabeled flags on MOCOs. Deleted solenoids. Need to add flags to TIVAs.
Parts:
- removed D1, D11, D12, D13, D18, D2, D4, D5, D8: LED, LED_SMD:LED_0603_1608Metric_Pad1.05x0.95mm_HandSolder, symbol Device:LED_Small
- removed D22, D34: D_Small, symbol Device:D_Small
- removed D30: Pink, symbol Device:LED_Small
- removed Q1, Q2, Q3, Q4, Q5, Q6, Q7, Q8, Q9: BSS138, Package_TO_SOT_SMD:SOT-23, symbol Transistor_FET:BSS138
- removed R1, R11, R12, R13, R14, R3, R4, R7, R8: 1k, Resistor_SMD:R_0603_1608Metric_Pad0.98x0.95mm_HandSolder, symbol Device:R_Small
- removed SolVal1, SolVal2, SolVal3, SolVal4, SolVal5, SolVal6, SolVal7, SolVal8, SolVal9: Molex_SL_02, MRDT_Connectors:MOLEX_SL_02_Vertical, symbol MRDT_Connectors:Molex_SL_02
- added C15, C16, C17, C21, C22, C23: 0.1u, Capacitor_SMD:C_0603_1608Metric, symbol Device:C
- added C18, C19, C20: 10u, symbol Device:C_Small
- added Conn10, Conn8, Conn9: AndersonPP, MRDT_Connectors:Anderson_2_Horizontal_Side_by_Side, symbol MRDT_Connectors:AndersonPP
- added D1, D11, D12, D13, D2, D34, D4, D41, D42, D43, D44, D45, D5, D8: Pink, symbol Simulation_SPICE:DIODE
- added D18, D30, D46, D47, D48, D55, D56, D57: D_Small, symbol Device:D_Small
- added D22, D49, D50, D51, D52, D53, D54: Pink, symbol Device:LED_Small
- added Q1, Q2, Q26, Q27, Q28, Q3, Q4, Q5, Q6, Q7, Q8, Q9: SI4156DY, Package_SO:SOIC-8_3.9x4.9mm_P1.27mm, symbol Transistor_FET:FDS2734
- added R1, R11, R12, R13, R3, R4, R49, R50, R51, R52, R53, R7, R8: 120, symbol Device:R
- added R14, R54, R55, R56, R57, R58, R59, R66, R67, R68, R69, R70, R71: 100, Resistor_SMD:R_0603_1608Metric_Pad0.98x0.95mm_HandSolder, symbol Device:R
- added R60, R61, R62, R63, R64, R65: 500, Resistor_SMD:R_0603_1608Metric_Pad0.98x0.95mm_HandSolder, symbol Device:R
- added U12, U13, U14, U15, U16, U17: IRS2005S, Package_SO:SOIC-8_3.9x4.9mm_P1.27mm, symbol Driver_FET:IRS2005S
- R26: value 100 -> 500
- R34: value 500 -> 100
- R42: value 100 -> 120; footprint Resistor_SMD:R_0603_1608Metric_Pad0.98x0.95mm_HandSolder -> (none)
Connections:
- net +12V: now also Q11.5 (D), Q11.6 (D), Q11.7 (D), Q11.8 (D), Q13.5 (D), Q13.6 (D), Q13.7 (D), Q13.8 (D), Q17.5 (D), Q17.6 (D), Q17.7 (D), Q17.8 (D), Q19.5 (D), Q19.6 (D), Q19.7 (D), Q19.8 (D), Q21.5 (D), Q21.6 (D), Q21.7 (D), Q21.8 (D), Q25.5 (D), Q25.6 (D), Q25.7 (D), Q25.8 (D), D18.2 (A), D30.2 (A), D46.2 (A), D47.2 (A), D48.2 (A), D55.2 (A), D56.2 (A), D57.2 (A), Q1.5 (D), Q1.6 (D), Q1.7 (D), Q1.8 (D), Q27.5 (D), Q27.6 (D), Q27.7 (D), Q27.8 (D), Q3.5 (D), Q3.6 (D), Q3.7 (D), Q3.8 (D), Q5.5 (D), Q5.6 (D), Q5.7 (D), Q5.8 (D), Q7.5 (D), Q7.6 (D), Q7.7 (D), Q7.8 (D), Q9.5 (D), Q9.6 (D), Q9.7 (D), Q9.8 (D), U12.1 (VCC), U13.1 (VCC), U14.1 (VCC), U15.1 (VCC), U16.1 (VCC), U17.1 (VCC); no longer Q10.5 (D), Q10.6 (D), Q10.7 (D), Q10.8 (D), Q12.5 (D), Q12.6 (D), Q12.7 (D), Q12.8 (D), Q16.5 (D), Q16.6 (D), Q16.7 (D), Q16.8 (D), Q18.5 (D), Q18.6 (D), Q18.7 (D), Q18.8 (D), Q20.5 (D), Q20.6 (D), Q20.7 (D), Q20.8 (D), Q24.5 (D), Q24.6 (D), Q24.7 (D), Q24.8 (D)
- net FWD_PWM_1: now also D34.1 (A), U12.2 (HIN), U15.3 (LIN); no longer U11.3 (LIN), U7.2 (HIN)
- net FWD_PWM_2: now also D42.1 (A), U14.2 (HIN), U17.3 (LIN); no longer U5.2 (HIN), U9.3 (LIN)
- net FWD_PWM_3: now also D41.1 (A), U13.2 (HIN), U16.3 (LIN); no longer U4.2 (HIN), U8.3 (LIN)
- net FWD_PWM_4: now also U11.3 (LIN), U7.2 (HIN), D5.1 (A); no longer U10.3 (LIN), U6.2 (HIN)
- net GND: now also Q10.1 (S), Q10.2 (S), Q10.3 (S), Q12.1 (S), Q12.2 (S), Q12.3 (S), Q16.1 (S), Q16.2 (S), Q16.3 (S), Q18.1 (S), Q18.2 (S), Q18.3 (S), Q20.1 (S), Q20.2 (S), Q20.3 (S), Q24.1 (S), Q24.2 (S), Q24.3 (S), R26.2, R42.2, Q2.1 (S), Q2.2 (S), Q2.3 (S), Q26.1 (S), Q26.2 (S), Q26.3 (S), Q28.1 (S), Q28.2 (S), Q28.3 (S), Q4.1 (S), Q4.2 (S), Q4.3 (S), Q6.1 (S), Q6.2 (S), Q6.3 (S), Q8.1 (S), Q8.2 (S), Q8.3 (S), R1.2, R11.2, R12.2, R13.2, R3.2, R4.2, R49.2, R50.2, R51.2, R52.2, R53.2, R60.2, R61.2, R62.2, R63.2, R64.2, R65.2, R7.2, R8.2, U12.4 (COM), U13.4 (COM), U14.4 (COM), U15.4 (COM), U16.4 (COM), U17.4 (COM); no longer Q11.1 (S), Q11.2 (S), Q11.3 (S), Q13.1 (S), Q13.2 (S), Q13.3 (S), Q17.1 (S), Q17.2 (S), Q17.3 (S), Q19.1 (S), Q19.2 (S), Q19.3 (S), Q21.1 (S), Q21.2 (S), Q21.3 (S), Q25.1 (S), Q25.2 (S), Q25.3 (S), R34.2
- net M+: now also Q13.1 (S), Q13.2 (S), Q13.3 (S), Q16.5 (D), Q16.6 (D), Q16.7 (D), Q16.8 (D), Q17.1 (S), Q17.2 (S), Q17.3 (S), Q18.5 (D), Q18.6 (D), Q18.7 (D), Q18.8 (D), Q19.1 (S), Q19.2 (S), Q19.3 (S), Q20.5 (D), Q20.6 (D), Q20.7 (D), Q20.8 (D), C15.2, C16.2, C17.2, C18.1, C19.1, C20.1, Conn10.1 (GND), Conn8.1 (GND), Conn9.1 (GND), D22.2 (A), D49.2 (A), D50.2 (A), D51.2 (A), Q1.1 (S), Q1.2 (S), Q1.3 (S), Q2.5 (D), Q2.6 (D), Q2.7 (D), Q2.8 (D), Q3.1 (S), Q3.2 (S), Q3.3 (S), Q4.5 (D), Q4.6 (D), Q4.7 (D), Q4.8 (D), Q5.1 (S), Q5.2 (S), Q5.3 (S), Q6.5 (D), Q6.6 (D), Q6.7 (D), Q6.8 (D), U12.6 (VS), U13.6 (VS), U14.6 (VS); no longer D26.2 (A), Q10.1 (S), Q10.2 (S), Q10.3 (S), Q11.5 (D), Q11.6 (D), Q11.7 (D), Q11.8 (D), Q12.1 (S), Q12.2 (S), Q12.3 (S), Q13.5 (D), Q13.6 (D), Q13.7 (D), Q13.8 (D), Q16.1 (S), Q16.2 (S), Q16.3 (S), Q17.5 (D), Q17.6 (D), Q17.7 (D), Q17.8 (D)
- net M-: now also D26.2 (A), Q10.5 (D), Q10.6 (D), Q10.7 (D), Q10.8 (D), Q11.1 (S), Q11.2 (S), Q11.3 (S), Q12.5 (D), Q12.6 (D), Q12.7 (D), Q12.8 (D), Q21.1 (S), Q21.2 (S), Q21.3 (S), Q24.5 (D), Q24.6 (D), Q24.7 (D), Q24.8 (D), Q25.1 (S), Q25.2 (S), Q25.3 (S), C18.2, C19.2, C20.2, C21.2, C22.2, C23.2, Conn10.2 (V+Log), Conn8.2 (V+Log), Conn9.2 (V+Log), D52.2 (A), D53.2 (A), D54.2 (A), Q26.5 (D), Q26.6 (D), Q26.7 (D), Q26.8 (D), Q27.1 (S), Q27.2 (S), Q27.3 (S), Q28.5 (D), Q28.6 (D), Q28.7 (D), Q28.8 (D), Q7.1 (S), Q7.2 (S), Q7.3 (S), Q8.5 (D), Q8.6 (D), Q8.7 (D), Q8.8 (D), Q9.1 (S), Q9.2 (S), Q9.3 (S), U15.6 (VS), U16.6 (VS), U17.6 (VS); no longer Q18.1 (S), Q18.2 (S), Q18.3 (S), Q19.5 (D), Q19.6 (D), Q19.7 (D), Q19.8 (D), Q20.1 (S), Q20.2 (S), Q20.3 (S), Q21.5 (D), Q21.6 (D), Q21.7 (D), Q21.8 (D), Q24.1 (S), Q24.2 (S), Q24.3 (S), Q25.5 (D), Q25.6 (D), Q25.7 (D), Q25.8 (D)
- net RVS_PWM_1: now also D43.1 (A), U12.3 (LIN), U15.2 (HIN); no longer U11.2 (HIN), U7.3 (LIN)
- net RVS_PWM_2: now also D45.1 (A), U14.3 (LIN), U17.2 (HIN); no longer U5.3 (LIN), U9.2 (HIN)
- net RVS_PWM_3: now also D44.1 (A), U13.3 (LIN), U16.2 (HIN); no longer U4.3 (LIN), U8.2 (HIN)
- net RVS_PWM_4: now also U11.2 (HIN), U7.3 (LIN), D13.1 (A); no longer U10.2 (HIN), U6.3 (LIN)
- net at Q21.4 (G): now also R66.2; no longer R38.2
- net at R41.2: now also Q12.4 (G); no longer Q24.4 (G)
- net at Q25.4 (G): now also R68.2; no longer R42.2
- net at D23.1 (K): now also R29.1; no longer R28.1
- net at C4.1, U5.8 (VB): now also D19.1 (K); no longer D20.1 (K)
- net at R35.2: now also Q8.4 (G); no longer Q18.4 (G)
- net at C14.1, U11.8 (VB): now also D32.1 (K)
- net at Q17.4 (G): now also R56.2; no longer R26.2
- net at R25.1: now also U7.5 (LO); no longer U7.7 (HO)
- net at Q16.4 (G): now also R55.2; no longer R25.2
- net at R30.1: now also D28.1 (K); no longer D24.1 (K)
- net at R26.1: now also D26.1 (K); no longer U7.5 (LO)
- net at C6.1, U7.8 (VB): now also D20.1 (K)
- net at U9.5 (LO): now also R37.1; no longer R38.1
- net at C11.1, U8.8 (VB): now also D30.1 (K); no longer D31.1 (K)
- net at R27.1: now also D22.1 (K); no longer D27.1 (K)
- net at R22.1: now also U7.7 (HO); no longer U5.5 (LO)
- net at R22.2: now also Q5.4 (G); no longer Q13.4 (G)
- net at R41.1: now also U11.5 (LO); no longer U11.7 (HO)
- net at U8.5 (LO): now also R35.1; no longer R36.1
- net at U8.7 (HO): now also R34.1; no longer R35.1
- net at R42.1: now also D34.2 (K); no longer U11.5 (LO)
- net at Q11.4 (G): now also R38.2; no longer R20.2
- net at R36.2: now also Q9.4 (G); no longer Q19.4 (G)
- net at U9.7 (HO): now also R36.1; no longer R37.1
- net at C12.1, U9.8 (VB): now also D31.1 (K); no longer D32.1 (K)
- net at Q20.4 (G): now also R59.2; no longer R37.2
- net at R20.1: now also U5.7 (HO); no longer U4.5 (LO)
- net at R19.1: now also U4.5 (LO); no longer U4.7 (HO)
- net at C3.1, U4.8 (VB): now also D18.1 (K); no longer D19.1 (K)
- net at Q10.4 (G): now also R37.2; no longer R19.2
- net at R21.1: now also U5.5 (LO); no longer U5.7 (HO)
- net at R21.2: now also Q4.4 (G); no longer Q12.4 (G)
- net at R33.1: now also D24.1 (K)
- net Solenoid_Valve_1: no longer names the net of U3.PB4 (B2_3)
- net Solenoid_Valve_2: no longer names the net of U3.PP0 (A2_3)
- net Solenoid_Valve_3: no longer names the net of U3.PB5 (B2_4)
- net Solenoid_Valve_4: no longer names the net of U3.PP1 (A2_4)
- net Solenoid_Valve_5: no longer names the net of U3.PK0 (B2_5)
- net Solenoid_Valve_6: no longer names the net of U3.PD4 (A2_5)
- net Solenoid_Valve_7: no longer names the net of U3.PK1 (B2_6)
- net Solenoid_Valve_8: no longer names the net of U3.PK2 (B2_7)
- net Solenoid_Valve_9: no longer names the net of U3.PK3 (B2_8)
- new net: C16.1, D47.1 (K), U13.8 (VB)
- new net: D52.1 (K), R60.1
- new net: C21.1, D55.1 (K), U15.8 (VB)
- new net: D1.2 (K), R1.1
- new net: R59.1, U14.5 (LO)
- new net: R69.1, U16.5 (LO)
- new net: R68.1, U16.7 (HO)
- new net: C22.1, D56.1 (K), U16.8 (VB)
- new net: D5.2 (K), R7.1
- new net: D11.2 (K), R11.1
- new net: D12.2 (K), R12.1
- new net: C23.1, D57.1 (K), U17.8 (VB)
- new net: Q26.4 (G), R69.2
- new net: C17.1, D48.1 (K), U14.8 (VB)
- new net: R70.1, U17.7 (HO)
- new net: Q27.4 (G), R70.2
- new net: D51.1 (K), R65.1
- new net: R55.1, U12.5 (LO)
- new net: R38.1, U11.7 (HO)
- new net: Q3.4 (G), R20.2
- new net: D2.2 (K), R3.1
- new net: Q2.4 (G), R19.2
- new net: D41.2 (K), R49.1
- new net: D42.2 (K), R50.1
- new net: C15.1, D46.1 (K), U12.8 (VB)
- new net: R67.1, U15.5 (LO)
- new net: Q24.4 (G), R67.2
- new net: Q19.4 (G), R58.2
- new net: D50.1 (K), R63.1
- new net: R14.1, U4.7 (HO)
- new net: Q1.4 (G), R14.2
- new net: D13.2 (K), R13.1
- new net: D54.1 (K), R64.1
- new net: R58.1, U14.7 (HO)
- new net: D27.1 (K), R28.1
- new net: D43.2 (K), R51.1
- new net: Q28.4 (G), R71.2
- new net: D45.2 (K), R53.1
- new net: R66.1, U15.7 (HO)
- new net: D49.1 (K), R61.1
- new net: Q7.4 (G), R34.2
- new net: D8.2 (K), R8.1
- new net: D44.2 (K), R52.1
- new net: R54.1, U12.7 (HO)
- new net: R56.1, U13.7 (HO)
- new net: R57.1, U13.5 (LO)
- new net: Q18.4 (G), R57.2
- new net: Q6.4 (G), R25.2
- new net: D53.1 (K), R62.1
- new net: Q13.4 (G), R54.2
- new net: D4.2 (K), R4.1
- new net: R71.1, U17.5 (LO)
- new net FWD_PWM_5: D2.1 (A), U4.2 (HIN), U8.3 (LIN)
- new net FWD_PWM_6: D4.1 (A), U5.2 (HIN), U9.3 (LIN)
- new net FWD_PWM_7: D1.1 (A), U10.3 (LIN), U6.2 (HIN)
- new net RVS_PWM_5: D11.1 (A), U4.3 (LIN), U8.2 (HIN)
- new net RVS_PWM_6: D12.1 (A), U5.3 (LIN), U9.2 (HIN)
- new net RVS_PWM_7: D8.1 (A), U10.2 (HIN), U6.3 (LIN)
- no-connect marks 43 -> 52
Other:
- note added: "Pump-1"
- note added: "Pump-2"
- note added: "Pump-3"
- note added: "Science-Z"
- note added: "Scoop-Z"
- note added: "X-Axis"
- note removed: "Solenoid Valves"
- note removed: "X-AXIS"
- note removed: "Y-AXIS"
- note removed: "Z-AXIS"
- moved on the sheet: AbsEncode1, AbsEncode2, AbsEncode3, AbsEncode4, C1, C13, C2, C5, C9, Conn1A, Conn1B, Conn2A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

Commit message: Added Servos
Parts:
- removed C10, C7, C8: 10u, symbol Device:C_Small
- removed C11, C12, C14, C3, C4, C6: 0.1u, Capacitor_SMD:C_0603_1608Metric, symbol Device:C
- removed Conn4, Conn5, Conn7: AndersonPP, MRDT_Connectors:Anderson_2_Horizontal_Side_by_Side, symbol MRDT_Connectors:AndersonPP
- removed D11, D12, D13, D2, D4, D5: Pink, symbol Simulation_SPICE:DIODE
- removed D18, D19, D20, D30, D31, D32: D_Small, symbol Device:D_Small
- removed D22, D23, D24, D26, D27, D28: Pink, symbol Device:LED_Small
- removed Q1, Q10, Q11, Q12, Q2, Q3, Q4, Q5, Q6, Q7, Q8, Q9: SI4156DY, Package_SO:SOIC-8_3.9x4.9mm_P1.27mm, symbol Transistor_FET:FDS2734
- removed R11, R12, R13, R3, R4, R7: 120, symbol Device:R
- removed R14, R19, R20, R21, R22, R25, R34, R35, R36, R37, R38, R41: 100, Resistor_SMD:R_0603_1608Metric_Pad0.98x0.95mm_HandSolder, symbol Device:R
- removed R26, R27, R28, R29, R30, R33: 500, Resistor_SMD:R_0603_1608Metric_Pad0.98x0.95mm_HandSolder, symbol Device:R
- removed U11, U4, U5, U7, U8, U9: IRS2005S, Package_SO:SOIC-8_3.9x4.9mm_P1.27mm, symbol Driver_FET:IRS2005S
- added Servo? (x4): Molex_SL_03, MRDT_Connectors:MOLEX_SL_03_Vertical, symbol MRDT_Connectors:Molex_SL_03
Connections:
- net FWD_PWM_7 is gone; now on net FWD_PWM_4: D1.1 (A), U10.3 (LIN), U6.2 (HIN)
- net RVS_PWM_7 is gone; now on net RVS_PWM_4: D8.1 (A), U10.2 (HIN), U6.3 (LIN)
- net +5V: now also Servo?.1, Servo?.1, Servo?.1, Servo?.1
- net GND: now also Servo?.2, Servo?.2, Servo?.2, Servo?.2
- net Servo_3: now reaches U3.PD7 (B1_7)
- net Servo_3: now also Servo?.3
- net Servo_4: now reaches U3.PD4 (A2_5)
- net Servo_4: now also Servo?.3
- net Servo_5: now reaches U3.PA4 (B2_9)
- net Servo_5: now also Servo?.3
- net Servo_6: now reaches U3.PA5 (B2_10)
- net Servo_6: now also Servo?.3
- no-connect marks 52 -> 48
Other:
- note removed: "Pump-1"
- note removed: "Pump-2"
- note removed: "Pump-3"
- moved on the sheet: C13, C15, C16, C17, C18, C19, C20, C21, C22, C23, C5, C9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

Commit message: Added Annotations
Parts:
- gave numbers to parts that had none: 4
Changed lines of the file:
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@@
   (symbol (lib_id "power:+5V") (at 269.875 371.475 0) (unit 1)
     (in_bom yes) (on_board yes) (fields_autoplaced)
-    (property "Reference" "#PWR?" (id 0) (at 269.875 375.285 0)
+    (property "Reference" "#PWR024" (id 0) (at 269.875 375.285 0)
       (effects (font (size 1.27 1.27)) hide)
     )
@@
   (symbol (lib_id "power:GND") (at 254.635 353.695 0) (unit 1)
     (in_bom yes) (on_board yes)
-    (property "Reference" "#PWR?" (id 0) (at 254.635 360.045 0)
+    (property "Reference" "#PWR09" (id 0) (at 254.635 360.045 0)
       (effects (font (size 1.27 1.27)) hide)
     )
@@
   (symbol (lib_id "MRDT_Connectors:Molex_SL_03") (at 278.765 340.36 0) (unit 1)
     (in_bom yes) (on_board yes)
-    (property "Reference" "Servo?" (id 0) (at 281.9908 335.0768 0)
+    (property "Reference" "Servo4" (id 0) (at 281.9908 335.0768 0)
       (effects (font (size 1.524 1.524)) (justify left))
     )
@@
   (symbol (lib_id "power:GND") (at 254.635 316.23 0) (unit 1)
     (in_bom yes) (on_board yes)
-    (property "Reference" "#PWR?" (id 0) (at 254.635 322.58 0)
+    (property "Reference" "#PWR02" (id 0) (at 254.635 322.58 0)
       (effects (font (size 1.27 1.27)) hide)
     )
@@
   (symbol (lib_id "MRDT_Connectors:Molex_SL_03") (at 278.765 356.235 0) (unit 1)
     (in_bom yes) (on_board yes)
-    (property "Reference" "Servo?" (id 0) (at 281.9908 350.9518 0)
+    (property "Reference" "Servo5" (id 0) (at 281.9908 350.9518 0)
       (effects (font (size 1.524 1.524)) (justify left))
     )
@@
   (symbol (lib_id "power:+5V") (at 269.875 349.885 0) (unit 1)
     (in_bom yes) (on_board yes) (fields_autoplaced)
-    (property "Reference" "#PWR?" (id 0) (at 269.875 353.695 0)
+    (property "Reference" "#PWR023" (id 0) (at 269.875 353.695 0)
       (effects (font (size 1.27 1.27)) hide)
     )
@@
   (symbol (lib_id "power:+5V") (at 269.875 312.42 0) (unit 1)
     (in_bom yes) (on_board yes) (fields_autoplaced)
-    (property "Reference" "#PWR?" (id 0) (at 269.875 316.23 0)
+    (property "Reference" "#PWR019" (id 0) (at 269.875 316.23 0)
       (effects (font (size 1.27 1.27)) hide)
     )
@@
   (symbol (lib_id "MRDT_Connectors:Molex_SL_03") (at 278.765 318.77 0) (unit 1)
     (in_bom yes) (on_board yes)
-    (property "Reference" "Servo?" (id 0) (at 281.9908 313.4868 0)
+    (property "Reference" "Servo3" (id 0) (at 281.9908 313.4868 0)
       (effects (font (size 1.524 1.524)) (justify left))
     )
@@
   (symbol (lib_id "power:GND") (at 254.635 375.285 0) (unit 1)
     (in_bom yes) (on_board yes)
-    (property "Reference" "#PWR?" (id 0) (at 254.635 381.635 0)
+    (property "Reference" "#PWR014" (id 0) (at 254.635 381.635 0)
       (effects (font (size 1.27 1.27)) hide)
     )
@@
   (symbol (lib_id "power:+5V") (at 269.875 334.01 0) (unit 1)
     (in_bom yes) (on_board yes) (fields_autoplaced)
-    (property "Reference" "#PWR?" (id 0) (at 269.875 337.82 0)
+    (property "Reference" "#PWR020" (id 0) (at 269.875 337.82 0)
       (effects (font (size 1.27 1.27)) hide)
     )
@@
   (symbol (lib_id "power:GND") (at 254.635 337.82 0) (unit 1)
     (in_bom yes) (on_board yes)
-    (property "Reference" "#PWR?" (id 0) (at 254.635 344.17 0)
+    (property "Reference" "#PWR08" (id 0) (at 254.635 344.17 0)
       (effects (font (size 1.27 1.27)) hide)
     )
@@
   (symbol (lib_id "MRDT_Connectors:Molex_SL_03") (at 278.765 377.825 0) (unit 1)
     (in_bom yes) (on_board yes)
-    (property "Reference" "Servo?" (id 0) (at 281.9908 372.5418 0)
+    (property "Reference" "Servo6" (id 0) (at 281.9908 372.5418 0)
       (effects (font (size 1.524 1.524)) (justify left))
     )
@@
       (reference "#PWR01") (unit 1) (value "GND") (footprint "")
     )
+    (path "/2d51c380-348c-4c63-8e62-b2af5ba21f51"
+      (reference "#PWR02") (unit 1) (value "GND") (footprint "")
+    )
     (path "/3f0a462a-81e7-4802-9dbf-6d5bc63fdcf3"
       (reference "#PWR03") (unit 1) (value "GND") (footprint "")
@@
       (reference "#PWR07") (unit 1) (value "+12V") (footprint "")
     )
+    (path "/b6b23341-9551-47d5-9cfa-c85720fd58f4"
+      (reference "#PWR08") (unit 1) (value "GND") (footprint "")
+    )
+    (path "/203b65ac-ec7b-4cc8-a067-b3f0a416bc12"
+      (reference "#PWR09") (unit 1) (value "GND") (footprint "")
+    )
     (path "/f1577403-f94a-48b0-9735-9a46103c51eb"
       (reference "#PWR010") (unit 1) (value "GND") (footprint "")
@@
       (reference "#PWR013") (unit 1) (value "GND") (footprint "")
     )
+    (path "/a36f070c-e23e-4f28-9a86-fd1a8a017a93"
+      (reference "#PWR014") (unit 1) (value "GND") (footprint "")
+    )
     (path "/c887bbda-f1ca-4331-8cbf-dbd74075eec1"
       (reference "#PWR015") (unit 1) (value "GND") (footprint "")
@@
       (reference "#PWR018") (unit 1) (value "+3.3V") (footprint "")
     )
+    (path "/88330626-8613-4a95-9740-b8f6c433ba3d"
+      (reference "#PWR019") (unit 1) (value "+5V") (footprint "")
+    )
+    (path "/aa255952-3c09-4b83-ac60-923368058e1c"
+      (reference "#PWR020") (unit 1) (value "+5V") (footprint "")
+    )
     (path "/f9a050fc-db46-453e-9027-4930061b75b1"
       (reference "#PWR021") (unit 1) (value "GND") (footprint "")
@@
       (reference "#PWR022") (unit 1) (value "GND") (footprint "")
     )
+    (path "/70ca0e5e-99fb-4005-9919-89eba0f5485e"
+      (reference "#PWR023") (unit 1) (value "+5V") (footprint "")
+    )
+    (path "/06155180-77d0-49fa-958b-ea10dda023a7"
+      (reference "#PWR024") (unit 1) (value "+5V") (footprint "")
+    )
     (path "/55c6c8f1-287d-41a0-b55b-2ca02ca9b666"
       (reference "#PWR025") (unit 1) (value "GND") (footprint "")
@@
       (reference "#PWR0133") (unit 1) (value "GND") (footprint "")
     )
-    (path "/06155180-77d0-49fa-958b-ea10dda023a7"
-      (reference "#PWR?") (unit 1) (value "+5V") (footprint "")
-    )
-    (path "/203b65ac-ec7b-4cc8-a067-b3f0a416bc12"
-      (reference "#PWR?") (unit 1) (value "GND") (footprint "")
-    )
-    (path "/2d51c380-348c-4c63-8e62-b2af5ba21f51"
-      (reference "#PWR?") (unit 1) (value "GND") (footprint "")
-    )
-    (path "/70ca0e5e-99fb-4005-9919-89eba0f5485e"
-      (reference "#PWR?") (unit 1) (value "+5V") (footprint "")
-    )
-    (path "/88330626-8613-4a95-9740-b8f6c433ba3d"
-      (reference "#PWR?") (unit 1) (value "+5V") (footprint "")
-    )
-    (path "/a36f070c-e23e-4f28-9a86-fd1a8a017a93"
-      (reference "#PWR?") (unit 1) (value "GND") (footprint "")
-    )
-    (path "/aa255952-3c09-4b83-ac60-923368058e1c"
-      (reference "#PWR?") (unit 1) (value "+5V") (footprint "")
-    )
-    (path "/b6b23341-9551-47d5-9cfa-c85720fd58f4"
-      (reference "#PWR?") (unit 1) (value "GND") (footprint "")
-    )
     (path "/c8a67f34-9386-4d80-a420-d82b9d44494d"
       (reference "AbsEncode1") (unit 1) (value "Molex_SL_03") (footprint "MRDT_Connectors:MOLEX_SL_03_Vertical")
@@
       (reference "Servo2") (unit 1) (value "Molex_SL_03") (footprint "MRDT_Connectors:MOLEX_SL_03_Vertical")
     )
+    (path "/89576370-52f6-4833-9152-f59684fecb1a"
+      (reference "Servo3") (unit 1) (value "Molex_SL_03") (footprint "MRDT_Connectors:MOLEX_SL_03_Vertical")
+    )
     (path "/2ce6e20c-5e5f-4b6e-aa53-b48d0af505ae"
-      (reference "Servo?") (unit 1) (value "Molex_SL_03") (footprint "MRDT_Connectors:MOLEX_SL_03_Vertical")
+      (reference "Servo4") (unit 1) (value "Molex_SL_03") (footprint "MRDT_Connectors:MOLEX_SL_03_Vertical")
     )
     (path "/44e44281-283f-4213-bd55-fa1314f3cf26"
-      (reference "Servo?") (unit 1) (value "Molex_SL_03") (footprint "MRDT_Connectors:MOLEX_SL_03_Vertical")
-    )
-    (path "/89576370-52f6-4833-9152-f59684fecb1a"
-      (reference "Servo?") (unit 1) (value "Molex_SL_03") (footprint "MRDT_Connectors:MOLEX_SL_03_Vertical")
+      (reference "Servo5") (unit 1) (value "Molex_SL_03") (footprint "MRDT_Connectors:MOLEX_SL_03_Vertical")
     )
     (path "/e6a715b5-9935-4849-a11e-00a375ab6a2a"
-      (reference "Servo?") (unit 1) (value "Molex_SL_03") (footprint "MRDT_Connectors:MOLEX_SL_03_Vertical")
+      (reference "Servo6") (unit 1) (value "Molex_SL_03") (footprint "MRDT_Connectors:MOLEX_SL_03_Vertical")
     )
     (path "/2ca3e144-c5aa-4c0e-a343-bd942d3a2b8d"

Commit message: Started Layout
Update H-Bridges. Added Footprints. Started Layout with edge cuts and coopers.
Parts:
- removed D25, D29, D49, D50, D51, D52, D53, D54: Pink, symbol Device:LED_Small
- removed R31, R32, R60, R61, R62, R63, R64, R65: 500, Resistor_SMD:R_0603_1608Metric_Pad0.98x0.95mm_HandSolder, symbol Device:R
- C10: renamed from C17; footprint Capacitor_SMD:C_0603_1608Metric -> Capacitor_SMD:C_0603_1608Metric_Pad1.08x0.95mm_HandSolder
- C11: renamed from C19; footprint (none) -> Capacitor_SMD:C_0603_1608Metric_Pad1.08x0.95mm_HandSolder
- C12: renamed from C20; footprint (none) -> Capacitor_SMD:C_0603_1608Metric_Pad1.08x0.95mm_HandSolder
- C13: renamed from C22; footprint Capacitor_SMD:C_0603_1608Metric -> Capacitor_SMD:C_0603_1608Metric_Pad1.08x0.95mm_HandSolder
- C14: renamed from C23; footprint Capacitor_SMD:C_0603_1608Metric -> Capacitor_SMD:C_0603_1608Metric_Pad1.08x0.95mm_HandSolder
- C2: renamed from C15; footprint Capacitor_SMD:C_0603_1608Metric -> Capacitor_SMD:C_0603_1608Metric_Pad1.08x0.95mm_HandSolder
- C3: renamed from C5; footprint Capacitor_SMD:C_0603_1608Metric -> Capacitor_SMD:C_0603_1608Metric_Pad1.08x0.95mm_HandSolder
- C5: renamed from C18; footprint (none) -> Capacitor_SMD:C_0603_1608Metric_Pad1.08x0.95mm_HandSolder
- C6: renamed from C9; footprint (none) -> Capacitor_SMD:C_0603_1608Metric_Pad1.08x0.95mm_HandSolder
- C7: renamed from C21; footprint Capacitor_SMD:C_0603_1608Metric -> Capacitor_SMD:C_0603_1608Metric_Pad1.08x0.95mm_HandSolder
- C8: renamed from C13; footprint Capacitor_SMD:C_0603_1608Metric -> Capacitor_SMD:C_0603_1608Metric_Pad1.08x0.95mm_HandSolder
- C9: renamed from C16; footprint Capacitor_SMD:C_0603_1608Metric -> Capacitor_SMD:C_0603_1608Metric_Pad1.08x0.95mm_HandSolder
- Conn1, Conn2: footprint MRDT_Connectors:Square_Anderson_3_H_Side_By_Side -> MRDT_Connectors:Square_Anderson_2_V_Side_By_Side
- Conn3: footprint MRDT_Connectors:Square_Anderson_2_H_Side_By_Side -> MRDT_Connectors:Square_Anderson_2_V_Side_By_Side
- Conn4: renamed from Conn8; footprint MRDT_Connectors:Anderson_2_Horizontal_Side_by_Side -> MRDT_Connectors:Square_Anderson_2_V_Side_By_Side
- Conn5: renamed from Conn10; footprint MRDT_Connectors:Anderson_2_Horizontal_Side_by_Side -> MRDT_Connectors:Square_Anderson_2_V_Side_By_Side
- Conn6: renamed from Conn9; footprint MRDT_Connectors:Anderson_2_Horizontal_Side_by_Side -> MRDT_Connectors:Square_Anderson_2_V_Side_By_Side
- Conn7: renamed from Conn6; footprint MRDT_Connectors:Anderson_2_Horizontal_Side_by_Side -> MRDT_Connectors:Square_Anderson_2_V_Side_By_Side
- D1: renamed from D34; footprint (none) -> LED_SMD:LED_0603_1608Metric_Pad1.05x0.95mm_HandSolder
- D14: renamed from D55; footprint (none) -> Diode_SMD:D_0603_1608Metric_Pad1.05x0.95mm_HandSolder
- D15: renamed from D33; footprint (none) -> Diode_SMD:D_0603_1608Metric_Pad1.05x0.95mm_HandSolder
- D16: renamed from D41; footprint (none) -> LED_SMD:LED_0603_1608Metric_Pad1.05x0.95mm_HandSolder
- D17: renamed from D42; footprint (none) -> LED_SMD:LED_0603_1608Metric_Pad1.05x0.95mm_HandSolder
- D18: renamed from D44; footprint (none) -> LED_SMD:LED_0603_1608Metric_Pad1.05x0.95mm_HandSolder
- D19: renamed from D45; footprint (none) -> LED_SMD:LED_0603_1608Metric_Pad1.05x0.95mm_HandSolder
- D2: renamed from D1; footprint (none) -> LED_SMD:LED_0603_1608Metric_Pad1.05x0.95mm_HandSolder
- D20: renamed from D47; footprint (none) -> Diode_SMD:D_0603_1608Metric_Pad1.05x0.95mm_HandSolder
- D21: renamed from D48; footprint (none) -> Diode_SMD:D_0603_1608Metric_Pad1.05x0.95mm_HandSolder
- D22: renamed from D56; footprint (none) -> Diode_SMD:D_0603_1608Metric_Pad1.05x0.95mm_HandSolder
- D23: renamed from D57; footprint (none) -> Diode_SMD:D_0603_1608Metric_Pad1.05x0.95mm_HandSolder
- D4: renamed from D43; footprint (none) -> LED_SMD:LED_0603_1608Metric_Pad1.05x0.95mm_HandSolder
- D5: renamed from D8; footprint (none) -> LED_SMD:LED_0603_1608Metric_Pad1.05x0.95mm_HandSolder
- D6: renamed from D46; footprint (none) -> Diode_SMD:D_0603_1608Metric_Pad1.05x0.95mm_HandSolder
- D7: renamed from D21; footprint (none) -> Diode_SMD:D_0603_1608Metric_Pad1.05x0.95mm_HandSolder
- R1: renamed from R42; footprint (none) -> Resistor_SMD:R_0603_1608Metric_Pad0.98x0.95mm_HandSolder
- R2: renamed from R1; footprint (none) -> Resistor_SMD:R_0603_1608Metric_Pad0.98x0.95mm_HandSolder
- R20: renamed from R49; footprint (none) -> Resistor_SMD:R_0603_1608Metric_Pad0.98x0.95mm_HandSolder
- R21: renamed from R50; footprint (none) -> Resistor_SMD:R_0603_1608Metric_Pad0.98x0.95mm_HandSolder
- R22: renamed from R52; footprint (none) -> Resistor_SMD:R_0603_1608Metric_Pad0.98x0.95mm_HandSolder
- R23: renamed from R53; footprint (none) -> Resistor_SMD:R_0603_1608Metric_Pad0.98x0.95mm_HandSolder
- R4: renamed from R51; footprint (none) -> Resistor_SMD:R_0603_1608Metric_Pad0.98x0.95mm_HandSolder
- R5: renamed from R8; footprint (none) -> Resistor_SMD:R_0603_1608Metric_Pad0.98x0.95mm_HandSolder
- renumbered AbsEncode4 to AbsEncode2, AbsEncode2 to AbsEncode3, AbsEncode3 to AbsEncode4, C2 to C4, D14 to D10, D15 to D11, D17 to D12, D16 to D13, D9 to D24, D10 to D25, D36 to D26, D35 to D27, D40 to D28, D39 to D29, D37 to D30, D38 to D31, D6 to D8, D7 to D9, LimSwitch2 to LimSwitch1, LimSwitch1 to LimSwitch2, LimSwitch6 to LimSwitch3, LimSwitch5 to LimSwitch4, LimSwitch3 to LimSwitch5, LimSwitch4 to LimSwitch6, Q13 to Q1, Q18 to Q10, Q19 to Q11, Q20 to Q12, Q25 to Q13, Q26 to Q14, Q27 to Q15, Q28 to Q16, Q16 to Q2, Q14 to Q3, Q15 to Q4, Q21 to Q5, Q24 to Q6, Q22 to Q7, Q23 to Q8, Q17 to Q9, R5 to R10, R6 to R11, R66 to R12, R67 to R13, R39 to R14, R40 to R15, R15 to R16, R16 to R17, R17 to R19, R56 to R24, R57 to R25, R58 to R26, R59 to R27, R68 to R28, R69 to R29, R2 to R3, R70 to R30, R71 to R31, R9 to R32, R10 to R33, R44 to R34, R43 to R35, R48 to R36, R47 to R37, R45 to R38, R46 to R39, R54 to R6, R55 to R7, R23 to R8, R24 to R9, U12 to U1, U17 to U10, U3 to U11, U6 to U2, U1 to U3, U2 to U4, U15 to U5, U10 to U6, U13 to U7, U14 to U8, U16 to U9

Commit message: Started Layout Design
Connections:
- net Limit_Switch_1: now also R36.2
Changed lines of the file:
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@@
+    (stroke (width 0) (type default) (color 0 0 0 0))
+  )
+  (wire (pts (xy 534.035 50.8) (xy 535.305 50.8))
     (stroke (width 0) (type default) (color 0 0 0 0))
   )
