File: Hardware/ScienceMocoBoard_V1/ScienceMotorController_Hardware_2023.kicad_sch (KiCad schematic)
At the start: 166 parts, among them J1 RJ45_LED_Shielded, J2 Conn_02x03_Counter_Clockwise, Q1 SI4156DY, Q10 SI4156DY, Q11 SI4156DY, Q12 SI4156DY, Q13 SI4156DY, Q14 SI4156DY, Q15 SI4156DY, Q16 SI4156DY, Q2 SI4156DY, Q3 SI4156DY, Q4 SI4156DY, Q5 SI4156DY, Q6 SI4156DY, Q7 SI4156DY, Q8 SI4156DY, Q9 SI4156DY, U1 IRS2005S, U10 IRS2005S, U11 Teensy4.1_DEV-16771, U2 IRS2005S, U3 3V3 OKI, U4 TSR_1-2450, U5 IRS2005S, U6 IRS2005S, U7 IRS2005S, U8 IRS2005S, U9 IRS2005S

Commit message: Updated Schematic and Sorted Footprints
Parts:
- removed C10, C13, C3, C7: 1uF, Capacitor_SMD:C_0603_1608Metric_Pad1.08x0.95mm_HandSolder, symbol Device:C
- removed C11, C12, C5, C6: 10uF, Capacitor_SMD:C_0603_1608Metric_Pad1.08x0.95mm_HandSolder, symbol Device:C_Small
- removed D1, D16, D17, D18, D19, D2, D4, D5: Pink, LED_SMD:LED_0603_1608Metric_Pad1.05x0.95mm_HandSolder, symbol Simulation_SPICE:DIODE
- removed D15, D21, D23, D7: D_Small, Diode_SMD:D_0603_1608Metric_Pad1.05x0.95mm_HandSolder, symbol Device:D_Small
- removed DY?: LED, LED_SMD:LED_0603_1608Metric_Pad1.05x0.95mm_HandSolder, symbol Device:LED
- removed R1, R22, R5: 120, Resistor_SMD:R_0603_1608Metric_Pad0.98x0.95mm_HandSolder, symbol Device:R
- removed R12, R13, R14, R15, R29, R30, R8, R9, R?: 100, Resistor_SMD:R_0603_1608Metric_Pad0.98x0.95mm_HandSolder, symbol Device:R
- removed SW?: SW_Push, Button_Switch_SMD:SW_SPST_EVPBF, symbol Switch:SW_Push
- removed U1, U5, U9: IRS2005S, Package_SO:SOIC-8_3.9x4.9mm_P1.27mm, symbol Driver_FET:IRS2005S
- added C10, C13, C3, C7: 10u, Capacitor_SMD:C_0603_1608Metric, symbol Device:C_Small
- added C11, C12, C5, C6: 1u, Capacitor_SMD:C_0603_1608Metric, symbol Device:C
- added D1, D15, D16, D18, D21, D23, D4, D7: Pink, LED_SMD:LED_0603_1608Metric_Pad1.05x0.95mm_HandSolder, symbol Device:LED_Small
- added D17, D19, D2, D5: D_Small, LED_SMD:LED_0603_1608Metric_Pad1.05x0.95mm_HandSolder, symbol Device:D_Small
- added D25, D32: YELLOW, LED_SMD:LED_0603_1608Metric_Pad1.05x0.95mm_HandSolder, symbol Device:LED_Small
- added DY10, DY7, DY8, DY9: LED, LED_SMD:LED_0603_1608Metric_Pad1.05x0.95mm_HandSolder, symbol Device:LED
- added LimSwitch8, LimSwitch9: Molex_SL_02, MRDT_Connectors:MOLEX_SL_02_Vertical, symbol MRDT_Connectors:Molex_SL_02
- added R1, R22, R29, R30, R40, R47, R5, R50: 120, Resistor_SMD:R_0603_1608Metric_Pad0.98x0.95mm_HandSolder, symbol Device:R_Small
- added R33, R43, R44, R45, R46, R48, R49: 100, Resistor_SMD:R_0603_1608Metric_Pad0.98x0.95mm_HandSolder, symbol Device:R
- added R51, R52: 120, Resistor_SMD:R_0603_1608Metric_Pad0.98x0.95mm_HandSolder, symbol Device:R
- added SW10, SW7, SW8, SW9: SW_Push, Button_Switch_SMD:SW_SPST_EVPBF, symbol Switch:SW_Push
- added U1, U12, U5, U9: 74LVC2G04, Package_TO_SOT_SMD:SOT-23-6_Handsoldering, symbol 74xGxx:74LVC2G04
- added U13, U14, U15: IRS2005S, Package_SO:SOIC-8_3.9x4.9mm_P1.27mm, symbol Driver_FET:IRS2005S
- C14, C2, C8, C9: value 1uF -> 1u; footprint Capacitor_SMD:C_0603_1608Metric_Pad1.08x0.95mm_HandSolder -> Capacitor_SMD:C_0603_1608Metric
- D14, D20, D22, D6: footprint Diode_SMD:D_0603_1608Metric_Pad1.05x0.95mm_HandSolder -> LED_SMD:LED_0603_1608Metric_Pad1.05x0.95mm_HandSolder
- R2, R20, R21, R23, R4: value 120 -> 100
- gave numbers to parts that had none: 23
Connections:
- net +12V: now also D17.2 (A), D19.2 (A), D2.2 (A), D5.2 (A), U13.1 (VCC), U14.1 (VCC), U15.1 (VCC)
- net +3.3V: now also SW10.1, SW7.2, SW8.1, SW9.1
- net +3V3: now also LimSwitch8.1, LimSwitch9.1, U1.5 (VCC), U1.5 (VCC), U12.5 (VCC), U12.5 (VCC), U5.5 (VCC), U5.5 (VCC), U9.5 (VCC), U9.5 (VCC)
- net FWD_PWM_1: now also U6.2 (HIN), D4.2 (A), U5.1
- net FWD_PWM_2: now also D18.2 (A), U12.1, U13.2 (HIN); no longer U10.3 (LIN), U8.2 (HIN)
- net FWD_PWM_3: now also U10.2 (HIN), D15.2 (A), U9.1; no longer U7.2 (HIN)
- net FWD_PWM_4: now also D1.2 (A), U1.1; no longer U6.3 (LIN)
- net GND: now also D25.1 (K), D32.1 (K), DY10.1 (K), DY7.1 (K), DY8.1 (K), DY9.1 (K), R1.2, R22.1, R29.2, R30.1, R40.2, R47.1, R5.2, R50.1, U1.2 (GND), U1.2 (GND), U12.2 (GND), U12.2 (GND), U13.4 (COM), U14.4 (COM), U15.4 (COM), U5.2 (GND), U5.2 (GND), U9.2 (GND), U9.2 (GND); no longer R2.2, R20.2, R21.2, R23.2, R4.2
- net RVS_PWM_1: now also U8.2 (HIN), D16.2 (A), U5.3
- net RVS_PWM_2: now also D23.2 (A), U12.3, U15.2 (HIN); no longer U10.2 (HIN), U8.3 (LIN)
- net RVS_PWM_3: now also D21.2 (A), U14.2 (HIN), U9.3; no longer U7.3 (LIN)
- net RVS_PWM_4: now also U7.2 (HIN), D7.2 (A), U1.3; no longer U2.3 (LIN), U6.2 (HIN)
- net at D14.1 (K): now also C8.1, U8.8 (VB)
- net at R2.1: now also U2.7 (HO)
- net at U8.5 (LO): now also R24.1; no longer R27.1
- net at Q12.4 (G): now also R44.2; no longer R27.2
- net at R28.1: now also DY10.2 (A)
- net at D22.1 (K): now also C14.1, U15.8 (VB)
- net at U2.8 (VB): now also C2.1, D2.1 (K)
- net at U10.8 (VB): now also C9.1, D17.1 (K); no longer C14.1
- net at Q14.4 (G): now also R46.2
- net at Q5.4 (G): now also R20.2
- net at U10.7 (HO): now also R31.1
- net at Q15.4 (G): now also R48.2
- net at R7.1: now also U6.5 (LO)
- net at Q2.4 (G): now also R4.2; no longer R7.2
- net at R20.1: now also U7.7 (HO)
- net at R21.1: now also U7.5 (LO)
- net at D6.1 (K): now also U7.8 (VB), C6.1; no longer C2.1
- net at Q6.4 (G): now also R21.2
- net at Q3.4 (G): now also R6.2
- net at Q11.4 (G): now also R43.2; no longer R26.2
- net at Q8.4 (G): now also R24.2
- net at R26.1: now also DY8.2 (A); no longer U8.7 (HO)
- net at R4.1: now also U2.5 (LO)
- net at R31.2: now also Q9.4 (G); no longer Q16.4 (G)
- net at R23.1: now also U8.7 (HO)
- net at Q7.4 (G): now also R23.2
- net at U6.8 (VB): now also C5.1, D5.1 (K); no longer C8.1
- net at Q4.4 (G): now also R7.2
- net at Q13.4 (G): now also R45.2; no longer R28.2
- net at R6.1: now also U6.7 (HO)
- net at R25.1: now also DY7.2 (A); no longer U7.5 (LO)
- net at Q10.4 (G): now also R33.2; no longer R25.2
- net at Q1.4 (G): now also R2.2; no longer R6.2
- net at U10.5 (LO): now also R33.1; no longer R31.1
- net M+ renamed 1M+
- net 1M+: now also U10.6 (VS), U6.6 (VS), C10.1, C11.2, C13.1, C3.1, C5.2, C7.1, U13.6 (VS); no longer U7.6 (VS), U8.6 (VS)
- net M- renamed 1M-
- net 1M-: now also U7.6 (VS), U8.6 (VS), C10.2, C12.2, C13.2, C3.2, C6.2, C7.2, U14.6 (VS), U15.6 (VS); no longer U10.6 (VS), U6.6 (VS)
- new net: D15.1 (K), R29.1
- new net: U10.3 (LIN), U9.6
- new net: U14.3 (LIN), U9.4
- new net: R46.1, U14.5 (LO)
- new net: R45.1, U14.7 (HO)
- new net: C12.1, D20.1 (K), U14.8 (VB)
- new net: U5.6, U6.3 (LIN)
- new net: U1.6, U2.3 (LIN)
- new net: U12.4, U15.3 (LIN)
- new net: R49.1, U15.5 (LO)
- new net: R48.1, U15.7 (HO)
- new net: D32.2 (A), R52.1
- new net: C11.1, D19.1 (K), U13.8 (VB)
- new net: U5.4, U8.3 (LIN)
- new net: D25.2 (A), R51.1
- new net: D23.1 (K), R50.2
- new net: D16.1 (K), R30.2
- new net: D18.1 (K), R40.1
- new net: U12.6, U13.3 (LIN)
- new net: U1.4, U7.3 (LIN)
- new net: D7.1 (K), R22.2
- new net: D21.1 (K), R47.2
- new net: D1.1 (K), R1.1
- new net: Q16.4 (G), R49.2
- new net: R44.1, U13.5 (LO)
- new net: R43.1, U13.7 (HO)
- new net: DY9.2 (A), R27.1
- new net: D4.1 (K), R5.1
- new net Limit_Switch_8: LimSwitch8.2, R51.2
- new net Limit_Switch_9: LimSwitch9.2, R52.2
- new net Motor_1_SW: R25.2, SW7.1
- new net Motor_2_SW: R26.2, SW8.2
- new net Motor_3_SW: R27.2, SW9.2
- new net Motor_4_SW: R28.2, SW10.2
Other:
- note added: "Manual Motor Switches"
- moved on the sheet: D24, D26, D27, D28, D29, D30, D31, DY1, DY11, DY12, DY2, DY3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
