File: Hardware/Science Actuation/Science_Actuation.kicad_pcb (KiCad board)
At the start: 2 copper layers, 110.2 x 97.3 mm, 108 parts, among them J4 RJ45_LED_Shielded, Q1 BSS138, Q2 BSS138, Q3 BSS138, Q4 AO3401A, Q5 AO3401A, SW1 SW_Push, SW10 SW_SPDT, SW2 SW_Push, SW3 SW_Push, SW4 SW_Push, SW5 SW_Push, SW6 SW_Push, SW7 SW_Push, SW8 SW_Push, U1 Teensy4.1_DEV-16771, U2 OKI

Commit message: Final update for Rev1
Fixed edgecuts, made silkscreen labels cleaner. Regenerated gerb
Parts:
- moved D3 4.34 mm to (44.2, 24.6)
- moved R3 4.34 mm to (48.0, 24.6)
- moved D4 4.33 mm to (53.0, 24.6)
- moved R4 4.33 mm to (57.0, 24.6)
- moved D2 4.32 mm to (34.7, 24.6)
- moved D5 4.32 mm to (56.6, 42.9)
- moved D6 4.32 mm to (47.8, 42.9)
- moved D7 4.32 mm to (38.8, 42.9)
- moved R5 4.32 mm to (53.0, 42.9)
- moved R6 4.32 mm to (43.7, 42.9)
- moved R7 4.32 mm to (34.8, 42.9)
- moved R2 4.32 mm to (38.9, 24.6)
- moved Conn3 4.32 mm to (35.6, 30.6)
- moved Conn4 4.32 mm to (44.9, 30.6)
- moved Conn5 4.32 mm to (53.8, 30.6)
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Routing:
- net +12V: track 170.0 -> 155.5 mm
- net LimitSwitch4: track 31.8 -> 26.7 mm
- net LimitSwitch3: track 58.6 -> 53.5 mm
- net LimitSwitch5: track 86.9 -> 82.1 mm
- net LimitSwitch6: track 108.7 -> 104.3 mm
- net +3V3: track 490.7 -> 486.3 mm
- net Encoder_3b: track 67.0 -> 62.6 mm
- net Encoder_2a: track 70.5 -> 66.5 mm
- net LimitSwitch2: track 77.3 -> 73.8 mm
- net +5V: track 278.3 -> 275.4 mm
- net LimitSwitch1: track 90.2 -> 87.3 mm
- net Encoder_2b: track 70.0 -> 67.5 mm
- net T+: track 50.1 -> 52.4 mm
- net T-: track 50.1 -> 52.3 mm
- net LAS: track 54.9 -> 53.3 mm
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Other:
- board size 110.2 x 97.3 mm -> 109.7 x 97.1 mm
- board text added: "123 456 78"
- board text added: "H4"
- board text added: "MOCO1"
- board text added: "MOCO2"
- board text added: "MOCO3"
- board text added: "MOCO4"
- board text added: "Servo1"
- board text added: "Servo2"
- board text removed: "Anderson"
- board text removed: "Heaters"
- board text removed: "LEDS"
- board text removed: "Limit Switch"
- board text removed: "MOCO Breakout"
- board text removed: "Oki"
- board text removed: "Pumps"
- board text removed: "Quadrature Encoder"
- board text removed: "S1"
- board text removed: "S2"
- board text removed: "Servos"
- board text removed: "Teensy"

Commit message: Deleted Things
Parts:
- removed C1: 220uF, Capacitor_THT:CP_Radial_D6.3mm_P2.50mm
- removed C2: 0.1uF, Capacitor_SMD:C_0603_1608Metric_Pad1.08x0.95mm_HandSolder
- removed C3, C4: 10uF, Capacitor_SMD:C_0603_1608Metric_Pad1.08x0.95mm_HandSolder
- removed Conn1: AndersonPP, MRDT_Connectors:Square_Anderson_2_H_Side_By_Side
- removed Conn10, Conn11, Conn14, Conn15, Conn16, Conn17, Conn18, Conn9, Servo1, Servo2: Molex_SL_03, MRDT_Connectors:MOLEX_SL_03_Vertical
- removed Conn12, Conn13, Conn2, Conn3, Conn4, Conn5, Conn6, Conn7, Conn8: Molex_SL_02, MRDT_Connectors:MOLEX_SL_02_Vertical
- removed D1, D10, D11: Orange, LED_SMD:LED_0603_1608Metric_Pad1.05x0.95mm_HandSolder
- removed D12, D8, D9: Green, LED_SMD:LED_0603_1608Metric_Pad1.05x0.95mm_HandSolder
- removed D13, D14, D15, D16, D17, D18, D19, D20, D21: Blue, LED_SMD:LED_0603_1608Metric_Pad1.05x0.95mm_HandSolder
- removed D2, D23, D24, D25, D26, D27, D28, D3, D4, D5, D6, D7: YELLOW, LED_SMD:LED_0603_1608Metric_Pad1.05x0.95mm_HandSolder
- removed H1, H2, H3, H4: MountingHole, MRDT_Drill_Holes:4_40_Hole_Corner
- removed J4: RJ45_LED_Shielded, MRDT_Connectors:RJ45_Teensy
- removed Q1, Q2, Q3: BSS138, Package_TO_SOT_SMD:SOT-23
- removed Q4, Q5: AO3401A, Package_TO_SOT_SMD:SOT-23
- removed QuadEncode1, QuadEncode2, QuadEncode3: Molex_SL_04, MRDT_Connectors:MOLEX_SL_04_Vertical
- removed R1, R10: 300, Resistor_SMD:R_0603_1608Metric_Pad0.98x0.95mm_HandSolder
- removed R11, R12, R13, R14: 10k, Resistor_SMD:R_0603_1608Metric_Pad0.98x0.95mm_HandSolder
- removed R15, R16, R17: 1k, Resistor_SMD:R_0603_1608Metric_Pad0.98x0.95mm_HandSolder
- removed R18, R19, R2, R20, R21, R22, R23, R24, R25, R26, R28, R29, R3, R30, R31, R32, R33, R34, R4, R5, R6, R7: 100, Resistor_SMD:R_0603_1608Metric_Pad0.98x0.95mm_HandSolder
- removed R8, R9: 4.7k, Resistor_SMD:R_0603_1608Metric_Pad0.98x0.95mm_HandSolder
- removed SW1, SW2, SW3, SW4, SW5, SW6, SW7, SW8: SW_Push, Button_Switch_SMD:SW_SPST_TL3305A
- removed SW10: SW_SPDT, Button_Switch_THT:SW_Slide_1P2T_CK_OS102011MS2Q
- removed U1: Teensy4.1_DEV-16771, MRDT_Shields:Teensy_4_1_Ethernet
- removed U2: OKI, MRDT_Devices:OKI_Horizontal
Routing:
- net +3V3: track 486.3 -> 0.00 mm, vias 2 -> 0
- net +5V: track 275.4 -> 0.00 mm
- net +12V: track 155.5 -> 0.00 mm, vias 2 -> 0
- net LimitSwitch6: track 104.3 -> 0.00 mm
- net Heater_Temp4: track 97.8 -> 0.00 mm
- net LimitSwitch1: track 87.3 -> 0.00 mm, vias 1 -> 0
- net DIR_SW: track 85.8 -> 0.00 mm
- net LimitSwitch5: track 82.1 -> 0.00 mm
- net Heater_Temp: track 78.4 -> 0.00 mm
- net Encoder_1b: track 77.4 -> 0.00 mm
- net Encoder_1a: track 76.6 -> 0.00 mm
- net LimitSwitch2: track 73.8 -> 0.00 mm, vias 1 -> 0
- net Heater_On: track 73.3 -> 0.00 mm
- net Encoder_3a: track 69.1 -> 0.00 mm
- net Encoder_2b: track 67.5 -> 0.00 mm
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- removed copper zone on B.Cu, net GND
- removed copper zone on F.Cu, net GND
Other:
- board outline removed
- board text removed: "123 456 78"
- board text removed: "12V"
- board text removed: "3V3"
- board text removed: "5V"
- board text removed: "Dir. Switch"
- board text removed: "Enc1"
- board text removed: "Enc2"
- board text removed: "Enc3"
- board text removed: "H1"
- board text removed: "H2"
- board text removed: "H3"
- board text removed: "H4"
- board text removed: "LS1"
- board text removed: "LS2"
- board text removed: "LS3"
- board text removed: "LS4"
- board text removed: "LS5"
- board text removed: "LS6"
- board text removed: "Laser"
- board text removed: "MOCO1"
- board text removed: "MOCO2"
- board text removed: "MOCO3"
- board text removed: "MOCO4"
- board text removed: "P1"
- board text removed: "P2"
- board text removed: "Science Actuation, Rev1 Mars Rover Design Team Missouri S&T, 2024 Noah Schaben, Landon Meyer"
- board text removed: "Servo1"
- board text removed: "Servo2"

Commit message: Updating PCB
Parts:
- added C1: 220uF, Capacitor_THT:CP_Radial_D6.3mm_P2.50mm, F.Cu at (117.6, 66.4)
- added C2: 0.1uF, Capacitor_SMD:C_0603_1608Metric_Pad1.08x0.95mm_HandSolder, F.Cu at (114.4, 91.4)
- added C3: 10uF, Capacitor_SMD:C_0603_1608Metric_Pad1.08x0.95mm_HandSolder, F.Cu at (136.9, 48.8)
- added C4: 10uF, Capacitor_SMD:C_0603_1608Metric_Pad1.08x0.95mm_HandSolder, F.Cu at (131.8, 48.8)
- added Conn1: AndersonPP, MRDT_Connectors:Square_Anderson_2_H_Side_By_Side, F.Cu at (126.4, 71.8)
- added Conn10: Molex_SL_03, MRDT_Connectors:MOLEX_SL_03_Vertical, F.Cu at (56.9, 68.3)
- added Conn11: Molex_SL_03, MRDT_Connectors:MOLEX_SL_03_Vertical, F.Cu at (51.8, 62.0)
- added Conn17: Molex_SL_03, MRDT_Connectors:MOLEX_SL_03_Vertical, F.Cu at (63.5, 62.0)
- added Conn2: Molex_SL_03, MRDT_Connectors:MOLEX_SL_03_Vertical, F.Cu at (75.2, 62.0)
- added Conn3: Molex_SL_02, MRDT_Connectors:MOLEX_SL_02_Vertical, F.Cu at (55.7, 38.9)
- added Conn4: Molex_SL_02, MRDT_Connectors:MOLEX_SL_02_Vertical, F.Cu at (64.6, 38.7)
- added Conn5: Molex_SL_02, MRDT_Connectors:MOLEX_SL_02_Vertical, F.Cu at (58.2, 45.2)
- added Conn6: Molex_SL_02, MRDT_Connectors:MOLEX_SL_02_Vertical, F.Cu at (67.1, 45.2)
- added Conn7: Molex_SL_02, MRDT_Connectors:MOLEX_SL_02_Vertical, F.Cu at (76.5, 45.2)
- added Conn9: Molex_SL_03, MRDT_Connectors:MOLEX_SL_03_Vertical, F.Cu at (68.6, 68.3)
- added D12: Green, LED_SMD:LED_0603_1608Metric_Pad1.05x0.95mm_HandSolder, F.Cu at (118.2, 50.5)
- added D13: Blue, LED_SMD:LED_0603_1608Metric_Pad1.05x0.95mm_HandSolder, F.Cu at (77.9, 105.0)
- added D14: Blue, LED_SMD:LED_0603_1608Metric_Pad1.05x0.95mm_HandSolder, F.Cu at (51.8, 84.7)
- added D15: Blue, LED_SMD:LED_0603_1608Metric_Pad1.05x0.95mm_HandSolder, F.Cu at (63.6, 84.7)
- added D16: Blue, LED_SMD:LED_0603_1608Metric_Pad1.05x0.95mm_HandSolder, F.Cu at (75.1, 84.7)
- added D17: Blue, LED_SMD:LED_0603_1608Metric_Pad1.05x0.95mm_HandSolder, F.Cu at (52.0, 96.9)
- added D18: Blue, LED_SMD:LED_0603_1608Metric_Pad1.05x0.95mm_HandSolder, F.Cu at (63.5, 97.0)
- added D19: Blue, LED_SMD:LED_0603_1608Metric_Pad1.05x0.95mm_HandSolder, F.Cu at (75.1, 96.9)
- added D2: YELLOW, LED_SMD:LED_0603_1608Metric_Pad1.05x0.95mm_HandSolder, F.Cu at (55.8, 32.2)
- added D20: Blue, LED_SMD:LED_0603_1608Metric_Pad1.05x0.95mm_HandSolder, F.Cu at (51.7, 108.6)
- added D23: YELLOW, LED_SMD:LED_0603_1608Metric_Pad1.05x0.95mm_HandSolder, F.Cu at (118.1, 42.7)
- added D24: YELLOW, LED_SMD:LED_0603_1608Metric_Pad1.05x0.95mm_HandSolder, F.Cu at (120.7, 42.7)
- added D25: YELLOW, LED_SMD:LED_0603_1608Metric_Pad1.05x0.95mm_HandSolder, F.Cu at (103.6, 42.4)
- added D26: YELLOW, LED_SMD:LED_0603_1608Metric_Pad1.05x0.95mm_HandSolder, F.Cu at (106.2, 42.4)
- added D27: YELLOW, LED_SMD:LED_0603_1608Metric_Pad1.05x0.95mm_HandSolder, F.Cu at (89.4, 42.2)
- added D28: YELLOW, LED_SMD:LED_0603_1608Metric_Pad1.05x0.95mm_HandSolder, F.Cu at (91.9, 42.2)
- added D3: YELLOW, LED_SMD:LED_0603_1608Metric_Pad1.05x0.95mm_HandSolder, F.Cu at (64.5, 32.2)
- added D4: YELLOW, LED_SMD:LED_0603_1608Metric_Pad1.05x0.95mm_HandSolder, F.Cu at (57.9, 51.6)
- added D5: YELLOW, LED_SMD:LED_0603_1608Metric_Pad1.05x0.95mm_HandSolder, F.Cu at (67.2, 51.4)
- added D6: YELLOW, LED_SMD:LED_0603_1608Metric_Pad1.05x0.95mm_HandSolder, F.Cu at (76.6, 51.7)
- added D8: Green, LED_SMD:LED_0603_1608Metric_Pad1.05x0.95mm_HandSolder, F.Cu at (118.2, 54.4)
- added D9: Green, LED_SMD:LED_0603_1608Metric_Pad1.05x0.95mm_HandSolder, F.Cu at (118.2, 58.2)
- added H1: MountingHole, MRDT_Drill_Holes:4_40_Hole_Corner, F.Cu at (146.6, 110.8)
- added H2: MountingHole, MRDT_Drill_Holes:4_40_Hole_Corner, F.Cu at (145.1, 31.9)
- added H3: MountingHole, MRDT_Drill_Holes:4_40_Hole_Corner, F.Cu at (48.5, 111.3)
- added H4: MountingHole, MRDT_Drill_Holes:4_40_Hole_Corner, F.Cu at (50.2, 35.5)
- added J4: RJ45_LED_Shielded, MRDT_Connectors:RJ45_Teensy, F.Cu at (147.2, 86.7)
- added QuadEncode1: Molex_SL_04, MRDT_Connectors:MOLEX_SL_04_Vertical, F.Cu at (115.6, 32.8)
- added QuadEncode2: Molex_SL_04, MRDT_Connectors:MOLEX_SL_04_Vertical, F.Cu at (101.1, 32.8)
- added QuadEncode3: Molex_SL_04, MRDT_Connectors:MOLEX_SL_04_Vertical, F.Cu at (86.9, 32.8)
- added R10: 300, Resistor_SMD:R_0603_1608Metric_Pad0.98x0.95mm_HandSolder, F.Cu at (120.8, 54.4)
- added R15: 1k, Resistor_SMD:R_0603_1608Metric_Pad0.98x0.95mm_HandSolder, F.Cu at (120.8, 58.2)
- added R18: 100, Resistor_SMD:R_0603_1608Metric_Pad0.98x0.95mm_HandSolder, F.Cu at (120.8, 50.5)
- added R19: 100, Resistor_SMD:R_0603_1608Metric_Pad0.98x0.95mm_HandSolder, F.Cu at (55.8, 84.7)
- added R2: 100, Resistor_SMD:R_0603_1608Metric_Pad0.98x0.95mm_HandSolder, F.Cu at (58.3, 32.2)
- added R20: 100, Resistor_SMD:R_0603_1608Metric_Pad0.98x0.95mm_HandSolder, F.Cu at (67.4, 84.7)
- added R21: 100, Resistor_SMD:R_0603_1608Metric_Pad0.98x0.95mm_HandSolder, F.Cu at (78.9, 84.7)
- added R22: 100, Resistor_SMD:R_0603_1608Metric_Pad0.98x0.95mm_HandSolder, F.Cu at (55.8, 96.9)
- added R23: 100, Resistor_SMD:R_0603_1608Metric_Pad0.98x0.95mm_HandSolder, F.Cu at (67.5, 97.0)
- added R24: 100, Resistor_SMD:R_0603_1608Metric_Pad0.98x0.95mm_HandSolder, F.Cu at (79.2, 96.9)
- added R25: 100, Resistor_SMD:R_0603_1608Metric_Pad0.98x0.95mm_HandSolder, F.Cu at (55.5, 108.6)
- added R28: 100, Resistor_SMD:R_0603_1608Metric_Pad0.98x0.95mm_HandSolder, F.Cu at (75.9, 105.0)
- added R29: 100, Resistor_SMD:R_0603_1608Metric_Pad0.98x0.95mm_HandSolder, F.Cu at (118.1, 38.4)
- added R3: 100, Resistor_SMD:R_0603_1608Metric_Pad0.98x0.95mm_HandSolder, F.Cu at (67.1, 32.2)
- added R30: 100, Resistor_SMD:R_0603_1608Metric_Pad0.98x0.95mm_HandSolder, F.Cu at (120.6, 38.4)
- added R31: 100, Resistor_SMD:R_0603_1608Metric_Pad0.98x0.95mm_HandSolder, F.Cu at (103.7, 38.1)
- added R32: 100, Resistor_SMD:R_0603_1608Metric_Pad0.98x0.95mm_HandSolder, F.Cu at (106.2, 38.1)
- added R33: 100, Resistor_SMD:R_0603_1608Metric_Pad0.98x0.95mm_HandSolder, F.Cu at (89.4, 38.1)
- added R34: 100, Resistor_SMD:R_0603_1608Metric_Pad0.98x0.95mm_HandSolder, F.Cu at (91.9, 38.1)
- added R4: 100, Resistor_SMD:R_0603_1608Metric_Pad0.98x0.95mm_HandSolder, F.Cu at (55.6, 51.6)
- added R5: 100, Resistor_SMD:R_0603_1608Metric_Pad0.98x0.95mm_HandSolder, F.Cu at (64.5, 51.4)
- added R6: 100, Resistor_SMD:R_0603_1608Metric_Pad0.98x0.95mm_HandSolder, F.Cu at (74.0, 51.7)
- added SW1: SW_Push, Button_Switch_SMD:SW_SPST_TL3305A, F.Cu at (54.1, 80.7)
- added SW10: SW_SPDT, Button_Switch_THT:SW_Slide_1P2T_CK_OS102011MS2Q, F.Cu at (69.0, 104.8)
- added SW2: SW_Push, Button_Switch_SMD:SW_SPST_TL3305A, F.Cu at (65.7, 80.7)
- added SW3: SW_Push, Button_Switch_SMD:SW_SPST_TL3305A, F.Cu at (77.2, 80.7)
- added SW4: SW_Push, Button_Switch_SMD:SW_SPST_TL3305A, F.Cu at (54.1, 93.2)
- added SW5: SW_Push, Button_Switch_SMD:SW_SPST_TL3305A, F.Cu at (65.7, 93.2)
- added SW6: SW_Push, Button_Switch_SMD:SW_SPST_TL3305A, F.Cu at (77.4, 93.2)
- added SW7: SW_Push, Button_Switch_SMD:SW_SPST_TL3305A, F.Cu at (53.8, 104.9)
- added Servo1: Molex_SL_03, MRDT_Connectors:MOLEX_SL_03_Vertical, F.Cu at (121.7, 104.1)
- added Servo2: Molex_SL_03, MRDT_Connectors:MOLEX_SL_03_Vertical, F.Cu at (133.3, 104.1)
- added U1: Teensy4.1_DEV-16771, MRDT_Shields:Teensy_4_1_Ethernet, F.Cu at (96.8, 81.6)
- added U2: OKI, MRDT_Devices:OKI_Horizontal, F.Cu at (136.9, 44.1)
Routing:
- net +5V: track 0.00 -> 45.1 mm
- net +12V: track 0.00 -> 44.6 mm
- net +3V3: track 0.00 -> 36.5 mm
- net DIR_SW: track 0.00 -> 13.0 mm
- net SW2: track 0.00 -> 10.6 mm
- net SW3: track 0.00 -> 10.5 mm
- net SW1: track 0.00 -> 10.4 mm
- net SW5: track 0.00 -> 10.1 mm
- net SW4: track 0.00 -> 10.1 mm
- net SW7: track 0.00 -> 10.0 mm
- net SW6: track 0.00 -> 9.96 mm
- net LimitSwitch1: track 0.00 -> 5.73 mm
- net LimitSwitch2: track 0.00 -> 5.60 mm
- net LimitSwitch5: track 0.00 -> 5.59 mm
- net LimitSwitch3: track 0.00 -> 5.44 mm
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