File: Hardware/Science Actuation/Science_Actuation.kicad_pcb (KiCad board)
At the start: 2 copper layers, 79 parts, among them J4 RJ45_LED_Shielded, SW1 SW_Push, SW10 SW_SPDT, SW2 SW_Push, SW3 SW_Push, SW4 SW_Push, SW5 SW_Push, SW6 SW_Push, SW7 SW_Push, U1 Teensy4.1_DEV-16771, U2 OKI

Commit message: Updated Science Actuation again (definitely not finished)
Parts:
- added D30: YELLOW, LED_SMD:LED_0603_1608Metric_Pad1.05x0.95mm_HandSolder, F.Cu at (75.3, 42.3)
- added D31: YELLOW, LED_SMD:LED_0603_1608Metric_Pad1.05x0.95mm_HandSolder, F.Cu at (77.8, 42.3)
- added QuadEncode4: Molex_SL_04, MRDT_Connectors:MOLEX_SL_04_Vertical, F.Cu at (72.7, 32.7)
- added R40: 100, Resistor_SMD:R_0603_1608Metric_Pad0.98x0.95mm_HandSolder, F.Cu at (75.2, 37.9)
- added R41: 100, Resistor_SMD:R_0603_1608Metric_Pad0.98x0.95mm_HandSolder, F.Cu at (77.9, 37.9)
- moved R24 5.20 mm to (74.7, 99.5), turned to 0 degrees
- moved R23 5.03 mm to (63.1, 99.6), turned to 0 degrees
- moved R25 5.01 mm to (51.2, 111.1), turned to 0 degrees
- moved D4 4.88 mm to (56.6, 56.3)
- moved D6 4.88 mm to (75.2, 56.4)
- moved R4 4.88 mm to (54.3, 56.3)
- moved D3 4.88 mm to (63.2, 36.9)
- moved R5 4.88 mm to (63.2, 56.1)
- moved Conn3 4.88 mm to (54.4, 43.6)
- moved Conn6 4.88 mm to (65.7, 49.9)
- moved D2 4.88 mm to (54.4, 36.9)
- moved D5 4.88 mm to (65.8, 56.1)
- moved R2 4.88 mm to (57.0, 36.9)
- moved R3 4.88 mm to (65.7, 36.9)
- moved R6 4.88 mm to (72.7, 56.4)
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Connections:
- U1 pad 10: unconnected-(U1-CS1-Pad10) -> MOCO1_RVS
- U1 pad 11: MOCO_SP_RVS -> MOCO2_FWD
- U1 pad 12: MOCO_SP_FWD -> MOCO2_RVS
- U1 pad 24: LimitSwitch5 -> SW3
- U1 pad 25: Servo_1 -> SW2
- U1 pad 26: unconnected-(U1-A12-Pad26) -> SW1
- U1 pad 27: unconnected-(U1-A13-Pad27) -> SW4
- U1 pad 28: unconnected-(U1-RX7-Pad28) -> SW5
- U1 pad 29: Servo_SP -> SW6
- U1 pad 30: unconnected-(U1-CRX3-Pad30) -> SW7
- U1 pad 31: unconnected-(U1-CTX3-Pad31) -> DIR_SW
- U1 pad 36: SW6 -> SW4
- U1 pad 38: SW4 -> a
- U1 pad 39: SW3 -> s
- U1 pad 40: SW2 -> a
- U1 pad 41: SW1 -> q
- U1 pad 5: MOCO1_FWD -> MOCO4_FWD
- U1 pad 6: MOCO1_RVS -> MOCO4_RVS
- U1 pad 7: MOCO4_FWD -> MOCO_SP_RVS
- U1 pad 8: MOCO4_RVS -> MOCO_SP_FWD
- U1 pad 9: unconnected-(U1-OUT1C-Pad9) -> MOCO1_FWD
Routing:
- net +3V3: track 36.5 -> 273.6 mm
- net +5V: track 45.1 -> 124.1 mm
- net MOCO2_RVS: track 0.00 -> 46.7 mm
- net MOCO2_FWD: track 0.00 -> 42.7 mm
- net SW7: track 10.0 -> 50.4 mm
- net MOCO3_FWD: track 0.00 -> 37.6 mm
- net SW4: track 10.1 -> 46.5 mm
- net MOCO3_RVS: track 0.00 -> 35.9 mm
- net MOCO1_RVS: track 0.00 -> 30.3 mm
- net MOCO4_FWD: track 0.00 -> 29.6 mm
- net DIR_SW: track 13.0 -> 40.7 mm
- net MOCO1_FWD: track 0.00 -> 27.7 mm
- net SW5: track 10.1 -> 36.5 mm
- net MOCO4_RVS: track 0.00 -> 26.3 mm
- net MOCO_SP_FWD: track 0.00 -> 16.1 mm
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
Commit message: Updated PCB Board
Parts:
- moved D14 4.08 mm to (55.6, 87.2), turned to 180 degrees
- moved R21 3.94 mm to (74.7, 87.2), turned to 0 degrees
- moved R19 3.84 mm to (51.7, 87.2), turned to 0 degrees
- moved D15 3.82 mm to (67.2, 87.2), turned to 180 degrees
- moved R20 3.82 mm to (63.4, 87.2), turned to 0 degrees
- moved D16 3.82 mm to (78.6, 87.2), turned to 180 degrees
Connections:
- U1 pad 0: LimitSwitch4 -> LimitSwitch5
- U1 pad 1: MOCO2_FWD -> LimitSwitch4
- U1 pad 13: Encoder_3a -> unconnected-(U1-SCK-Pad13)
- U1 pad 14: Encoder_3b -> Encoder_1b
- U1 pad 15: Encoder_2a -> h
- U1 pad 16: Encoder_2b -> a
- U1 pad 17: Encoder_1a -> a
- U1 pad 18: Encoder_1b -> a
- U1 pad 2: MOCO2_RVS -> LimitSwitch3
- U1 pad 22: LimitSwitch2 -> LimitSwitch1
- U1 pad 23: LimitSwitch3 -> LimitSwitch2
- U1 pad 24: SW3 -> SW1
- U1 pad 26: SW1 -> SW3
- U1 pad 33: unconnected-(U1-MCLK2-Pad33) -> Servo_SP
- U1 pad 34: unconnected-(U1-RX8-Pad34) -> Encoder_4a
- U1 pad 35: SW7 -> Encoder_4b
- U1 pad 36: SW4 -> Servo_1
- U1 pad 37: SW5 -> Encoder_3a
- U1 pad 38: a -> Encoder_3b
- U1 pad 39: s -> Encoder_2a
- U1 pad 40: a -> Encoder_2b
- U1 pad 41: q -> Encoder_1a
Routing:
- net Encoder_4a: track 4.31 -> 103.9 mm
- net Encoder_4b: track 4.31 -> 98.4 mm
- net +5V: track 124.1 -> 216.8 mm
- net Encoder_1a: track 4.68 -> 91.3 mm
- net Encoder_1b: track 4.69 -> 86.2 mm
- net Encoder_2b: track 4.42 -> 83.6 mm
- net Encoder_2a: track 4.43 -> 83.2 mm
- net Encoder_3a: track 4.43 -> 82.5 mm
- net Encoder_3b: track 4.42 -> 79.6 mm
- net LimitSwitch1: track 5.73 -> 71.3 mm, vias 0 -> 1
- net LED: track 0.00 -> 58.2 mm
- net LimitSwitch2: track 5.60 -> 60.1 mm, vias 0 -> 1
- net T-: track 0.00 -> 52.2 mm
- net T+: track 0.00 -> 52.2 mm
- net R+: track 0.00 -> 45.6 mm
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
Commit message: Updated PCB components
Parts:
- removed C1: 220uF, Capacitor_THT:CP_Radial_D6.3mm_P2.50mm
- removed Conn11, Conn17: Molex_SL_03, MRDT_Connectors:MOLEX_SL_03_Vertical
- removed D17, D18, D19, D20: Blue, LED_SMD:LED_0603_1608Metric_Pad1.05x0.95mm_HandSolder
- removed D23, D24, D25, D26, D27, D28, D3, D30, D31, D4, D5, D6: YELLOW, LED_SMD:LED_0603_1608Metric_Pad1.05x0.95mm_HandSolder
- removed R32, R33, R34, R40, R41: 100, Resistor_SMD:R_0603_1608Metric_Pad0.98x0.95mm_HandSolder
- removed SW7: SW_Push, Button_Switch_SMD:SW_SPST_TL3305A
- added C10: 1uF, Capacitor_SMD:C_0603_1608Metric_Pad1.08x0.95mm_HandSolder, F.Cu at (119.6, 91.4)
- added C11: 1uF, Capacitor_SMD:C_0603_1608Metric_Pad1.08x0.95mm_HandSolder, F.Cu at (119.6, 93.9)
- added C12: 10uF, Capacitor_SMD:C_0603_1608Metric_Pad1.08x0.95mm_HandSolder, F.Cu at (119.6, 96.4)
- added C13: 1uF, Capacitor_SMD:C_0603_1608Metric_Pad1.08x0.95mm_HandSolder, F.Cu at (119.6, 98.9)
- added C14: 1uF, Capacitor_SMD:C_0603_1608Metric_Pad1.08x0.95mm_HandSolder, F.Cu at (119.6, 101.4)
- added C15: 10uF, Capacitor_SMD:C_0603_1608Metric_Pad1.08x0.95mm_HandSolder, F.Cu at (119.6, 103.9)
- added C16: 1uF, Capacitor_SMD:C_0603_1608Metric_Pad1.08x0.95mm_HandSolder, F.Cu at (124.0, 81.4)
- added C17: 1uF, Capacitor_SMD:C_0603_1608Metric_Pad1.08x0.95mm_HandSolder, F.Cu at (124.0, 83.9)
- added C18: 10uF, Capacitor_SMD:C_0603_1608Metric_Pad1.08x0.95mm_HandSolder, F.Cu at (124.0, 86.4)
- added C19: 1uF, Capacitor_SMD:C_0603_1608Metric_Pad1.08x0.95mm_HandSolder, F.Cu at (124.0, 88.9)
- added C20: 10uF, Capacitor_SMD:C_0603_1608Metric_Pad1.08x0.95mm_HandSolder, F.Cu at (124.0, 91.4)
- added C21: 220uF, Capacitor_THT:CP_Radial_D6.3mm_P2.50mm, F.Cu at (112.1, 111.4)
- added C22: 330uF, Capacitor_THT:CP_Radial_D8.0mm_P5.00mm, F.Cu at (165.5, 69.4)
- added C23: 470uF, Capacitor_THT:CP_Radial_D10.0mm_P5.00mm, F.Cu at (154.8, 70.4)
- added C8: 1uF, Capacitor_SMD:C_0603_1608Metric_Pad1.08x0.95mm_HandSolder, F.Cu at (119.6, 88.9)
- added C9: 100uF, Capacitor_THT:CP_Radial_D6.3mm_P2.50mm, F.Cu at (112.1, 103.5)
- added Conn8: AndersonPP, MRDT_Connectors:Square_Anderson_2_H_Side_By_Side, F.Cu at (115.8, 52.9)
- added D1: SD0603S04, Diode_SMD:D_0603_1608Metric_Pad1.05x0.95mm_HandSolder, F.Cu at (119.6, 106.5)
- added D10: SD0603S04, Diode_SMD:D_0603_1608Metric_Pad1.05x0.95mm_HandSolder, F.Cu at (124.0, 109.1)
- added D11: SD0603S04, Diode_SMD:D_0603_1608Metric_Pad1.05x0.95mm_HandSolder, F.Cu at (124.0, 111.7)
- added D7: SD0603S04, Diode_SMD:D_0603_1608Metric_Pad1.05x0.95mm_HandSolder, F.Cu at (119.6, 111.7)
- added Q1: Si4156DY, Package_SO:SOIC-8_3.9x4.9mm_P1.27mm, F.Cu at (121.7, 38.2)
- added Q10: Si4156DY, Package_SO:SOIC-8_3.9x4.9mm_P1.27mm, F.Cu at (130.1, 51.1)
- added Q11: Si4156DY, Package_SO:SOIC-8_3.9x4.9mm_P1.27mm, F.Cu at (130.1, 57.5)
- added Q12: Si4156DY, Package_SO:SOIC-8_3.9x4.9mm_P1.27mm, F.Cu at (130.1, 64.0)
- added Q13: Si4156DY, Package_SO:SOIC-8_3.9x4.9mm_P1.27mm, F.Cu at (130.1, 70.4)
- added Q14: Si4156DY, Package_SO:SOIC-8_3.9x4.9mm_P1.27mm, F.Cu at (130.1, 76.9)
- added Q15: Si4156DY, Package_SO:SOIC-8_3.9x4.9mm_P1.27mm, F.Cu at (138.6, 38.2)
- added Q16: Si4156DY, Package_SO:SOIC-8_3.9x4.9mm_P1.27mm, F.Cu at (138.6, 44.6)
- added Q2: Si4156DY, Package_SO:SOIC-8_3.9x4.9mm_P1.27mm, F.Cu at (121.7, 44.6)
- added Q3: Si4156DY, Package_SO:SOIC-8_3.9x4.9mm_P1.27mm, F.Cu at (121.7, 51.1)
- added Q4: Si4156DY, Package_SO:SOIC-8_3.9x4.9mm_P1.27mm, F.Cu at (121.7, 57.5)
- added Q5: Si4156DY, Package_SO:SOIC-8_3.9x4.9mm_P1.27mm, F.Cu at (121.7, 64.0)
- added Q6: Si4156DY, Package_SO:SOIC-8_3.9x4.9mm_P1.27mm, F.Cu at (121.7, 70.4)
- added Q7: Si4156DY, Package_SO:SOIC-8_3.9x4.9mm_P1.27mm, F.Cu at (121.7, 76.9)
- added Q8: Si4156DY, Package_SO:SOIC-8_3.9x4.9mm_P1.27mm, F.Cu at (130.1, 38.2)
- added Q9: Si4156DY, Package_SO:SOIC-8_3.9x4.9mm_P1.27mm, F.Cu at (130.1, 44.6)
- added R1: 100, Resistor_SMD:R_0603_1608Metric_Pad0.98x0.95mm_HandSolder, F.Cu at (124.0, 93.9)
- added R11: 100, Resistor_SMD:R_0603_1608Metric_Pad0.98x0.95mm_HandSolder, F.Cu at (128.3, 93.9)
- added R12: 100, Resistor_SMD:R_0603_1608Metric_Pad0.98x0.95mm_HandSolder, F.Cu at (128.3, 96.4)
- added R13: 100, Resistor_SMD:R_0603_1608Metric_Pad0.98x0.95mm_HandSolder, F.Cu at (128.3, 98.9)
- added R14: 100, Resistor_SMD:R_0603_1608Metric_Pad0.98x0.95mm_HandSolder, F.Cu at (128.3, 101.4)
- added R16: 100, Resistor_SMD:R_0603_1608Metric_Pad0.98x0.95mm_HandSolder, F.Cu at (132.7, 81.4)
- added R17: 100, Resistor_SMD:R_0603_1608Metric_Pad0.98x0.95mm_HandSolder, F.Cu at (132.7, 83.9)
- added R26: 100, Resistor_SMD:R_0603_1608Metric_Pad0.98x0.95mm_HandSolder, F.Cu at (137.0, 81.4)
- added R27: 100, Resistor_SMD:R_0603_1608Metric_Pad0.98x0.95mm_HandSolder, F.Cu at (137.0, 83.9)
- added R7: 100, Resistor_SMD:R_0603_1608Metric_Pad0.98x0.95mm_HandSolder, F.Cu at (128.3, 83.9)
- added R8: 100, Resistor_SMD:R_0603_1608Metric_Pad0.98x0.95mm_HandSolder, F.Cu at (128.3, 86.4)
- added R9: 100, Resistor_SMD:R_0603_1608Metric_Pad0.98x0.95mm_HandSolder, F.Cu at (128.3, 88.9)
- added U10: IRS2308, Package_SO:SOIC-8_3.9x4.9mm_P1.27mm, F.Cu at (138.6, 76.9)
- added U11: IRS2308, Package_SO:SOIC-8_3.9x4.9mm_P1.27mm, F.Cu at (147.0, 38.2)
- added U12: 74LVC2G04, Package_TO_SOT_SMD:SOT-23-6_Handsoldering, F.Cu at (174.4, 51.2)
- added U13: IRS2308, Package_SO:SOIC-8_3.9x4.9mm_P1.27mm, F.Cu at (147.0, 44.6)
- added U14: IRS2308, Package_SO:SOIC-8_3.9x4.9mm_P1.27mm, F.Cu at (147.0, 51.1)
- added U3: 74LVC2G04, Package_TO_SOT_SMD:SOT-23-6_Handsoldering, F.Cu at (174.4, 37.3)
- added U4: IRS2308, Package_SO:SOIC-8_3.9x4.9mm_P1.27mm, F.Cu at (138.6, 51.1)
- added U5: IRS2308, Package_SO:SOIC-8_3.9x4.9mm_P1.27mm, F.Cu at (138.6, 57.5)
- added U6: 74LVC2G04, Package_TO_SOT_SMD:SOT-23-6_Handsoldering, F.Cu at (174.4, 41.9)
- added U7: IRS2308, Package_SO:SOIC-8_3.9x4.9mm_P1.27mm, F.Cu at (138.6, 64.0)
- added U8: IRS2308, Package_SO:SOIC-8_3.9x4.9mm_P1.27mm, F.Cu at (138.6, 70.4)
- added U9: 74LVC2G04, Package_TO_SOT_SMD:SOT-23-6_Handsoldering, F.Cu at (174.4, 46.6)
- Conn10, Conn2, Conn9: value Molex_SL_03 -> AndersonPP; footprint MRDT_Connectors:MOLEX_SL_03_Vertical -> MRDT_Connectors:Square_Anderson_2_H_Side_By_Side
- D13, D14, D15, D16: value Blue -> SD0603S04; footprint LED_SMD:LED_0603_1608Metric_Pad1.05x0.95mm_HandSolder -> Diode_SMD:D_0603_1608Metric_Pad1.05x0.95mm_HandSolder
- D2: value YELLOW -> Blue
- R10: value 300 -> 620
- R15: value 1k -> 2.2k
- R18: value 100 -> 270
- R19, R2, R20, R21, R22, R23, R3, R31, R4, R5, R6: value 100 -> 4700
- R28: value 100 -> 30
- moved QuadEncode4 123.5 mm to (170.6, 108.0)
- moved H4 121.0 mm to (139.9, 116.8), turned to 0 degrees
- moved Conn5 116.3 mm to (162.0, 99.5), turned to 0 degrees
- moved Conn3 115.2 mm to (162.0, 84.5)
- moved Conn6 111.9 mm to (162.0, 107.0), turned to 0 degrees
- moved Conn4 110.0 mm to (162.0, 92.0)
- moved Conn7 108.2 mm to (162.0, 114.5), turned to 0 degrees
- moved QuadEncode3 107.6 mm to (170.6, 100.2)
- moved SW10 103.0 mm to (171.5, 114.6), turned to 0 degrees
- moved SW4 100.1 mm to (153.7, 101.3)
- moved SW1 99.9 mm to (153.7, 83.1)
- moved D2 97.3 mm to (119.6, 109.1), turned to 0 degrees
- moved H3 91.9 mm to (139.9, 107.4), turned to 0 degrees
- moved QuadEncode2 91.7 mm to (170.6, 92.5)
- moved R2 89.6 mm to (124.0, 96.4), turned to 0 degrees
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Connections:
- net Servo_SP renamed Servo_2
- Conn10 pad 1: +3V3 -> /M+
- Conn10 pad 2: MOCO2_FWD -> /M-
- Conn2 pad 1: +3V3 -> /M+
- Conn2 pad 2: MOCO_SP_FWD -> /M-
- Conn9 pad 1: +3V3 -> /M+
- Conn9 pad 2: MOCO1_FWD -> /M-
- D13 pad 2: +3V3 -> +12V
- D14 pad 1: GND -> Net-(D14-K)
- D14 pad 2: Net-(D14-A) -> +12V
- D15 pad 1: GND -> Net-(D15-K)
- D15 pad 2: Net-(D15-A) -> +12V
- D16 pad 1: GND -> Net-(D16-K)
- D16 pad 2: Net-(D16-A) -> +12V
- D2 pad 1: GND -> DIR_SW
- QuadEncode2 pad 2: Encoder_2a -> Encoder_1a
- QuadEncode2 pad 3: Encoder_2b -> Encoder_1b
- QuadEncode3 pad 2: Encoder_3a -> Encoder_1a
- QuadEncode3 pad 3: Encoder_3b -> Encoder_1b
- QuadEncode4 pad 2: Encoder_4a -> Encoder_1a
- QuadEncode4 pad 3: Encoder_4b -> Encoder_1b
- R19 pad 2: Net-(D14-A) -> GND
- R2 pad 1: Net-(D2-A) -> GND
- R20 pad 2: Net-(D15-A) -> GND
- R21 pad 2: Net-(D16-A) -> GND
- R22 pad 2: Net-(D17-A) -> GND
- R23 pad 2: Net-(D18-A) -> GND
- R24 pad 1: SW6 -> Net-(U11-HO)
- R25 pad 1: SW7 -> Net-(U11-LO)
- R28 pad 1: Net-(D13-K) -> +3V3
- R28 pad 2: DIR_SW -> Net-(D2-A)
- R29 pad 2: Encoder_1a -> Net-(Q15-G)
- R3 pad 1: Net-(D3-A) -> GND
- R30 pad 1: Encoder_1b -> Net-(U14-LO)
- R31 pad 1: Net-(D25-A) -> SW6
- R31 pad 2: Encoder_2a -> GND
- R4 pad 1: Net-(D4-A) -> GND
- R5 pad 1: Net-(D5-A) -> GND
- R6 pad 1: Net-(D6-A) -> GND
- U1 pad 15: h -> unconnected-(U1-A1-Pad15)
- U1 pad 16: a -> unconnected-(U1-A2-Pad16)
- U1 pad 17: a -> unconnected-(U1-A3-Pad17)
- U1 pad 18: a -> unconnected-(U1-A4-Pad18)
- U1 pad 22: LimitSwitch1 -> unconnected-(U1-A8-Pad22)
- U1 pad 30: SW7 -> unconnected-(U1-CRX3-Pad30)
- U1 pad 7: MOCO_SP_RVS -> unconnected-(U1-RX2-Pad7)
- U1 pad 8: MOCO_SP_FWD -> unconnected-(U1-TX2-Pad8)
Routing:
- net +3V3: track 279.3 -> 0.00 mm, vias 2 -> 0
- net +5V: track 216.8 -> 0.00 mm
- net Encoder_4a: track 103.9 -> 0.00 mm
- net Encoder_4b: track 98.4 -> 0.00 mm
- net Encoder_1a: track 91.3 -> 0.00 mm
- net Encoder_1b: track 86.2 -> 0.00 mm
- net Encoder_2b: track 83.6 -> 0.00 mm
- net Encoder_2a: track 83.2 -> 0.00 mm
- net Encoder_3a: track 82.5 -> 0.00 mm
- net Encoder_3b: track 79.6 -> 0.00 mm
- net LimitSwitch1: track 71.3 -> 0.00 mm, vias 1 -> 0
- net LimitSwitch2: track 60.1 -> 0.00 mm, vias 1 -> 0
- net LED: track 58.2 -> 0.00 mm
- net T-: track 52.2 -> 0.00 mm
- net T+: track 52.2 -> 0.00 mm
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
Commit message: Cleaned Schematic, Restarted PCB, Grouped components for each section
Parts:
- moved D1 393.0 mm to (483.5, -42.1)
- moved D7 393.0 mm to (483.5, -36.9)
- moved Q1 393.0 mm to (485.5, -110.4)
- moved Q2 393.0 mm to (485.5, -103.9)
- moved Q3 393.0 mm to (485.5, -97.5)
- moved Q4 393.0 mm to (485.5, -91.0)
- moved C10 393.0 mm to (483.4, -57.2)
- moved C12 393.0 mm to (483.4, -52.1)
- moved C8 393.0 mm to (483.4, -59.7)
- moved R1 393.0 mm to (487.8, -54.6)
- moved R7 393.0 mm to (492.1, -64.7)
- moved R8 393.0 mm to (492.1, -62.2)
- moved R9 393.0 mm to (492.1, -59.7)
- moved U4 393.0 mm to (502.4, -97.5)
- moved U5 393.0 mm to (502.4, -91.0)
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Routing:
- net GND: track 0.00 -> 12.0 mm
- net Net-(D9-A): track 0.00 -> 4.08 mm
- net Net-(D12-A): track 0.00 -> 4.08 mm
- net Net-(D8-A): track 0.00 -> 3.97 mm
Other:
- board text added: "12V"
- board text added: "3V3"
- board text added: "5V"
- board text added: "Buck Converter"
- board text added: "Buttons"
- board text added: "Dir. Switch"
- board text added: "LEDs"
- board text added: "Limit Switch Connectors"
- board text added: "MOCOs"
- board text added: "Power"
- board text added: "Quadrature Encoder"
- board text added: "RJ45 Ethernet"
- board text added: "Servos"
- board text added: "Teensy"

Commit message: Reposition all components
Parts:
- moved U4 373.4 mm to (182.8, 95.6), turned to 90 degrees
- moved U3 369.0 mm to (187.9, 85.5), turned to 90 degrees
- moved U5 363.1 mm to (190.9, 95.6), turned to 90 degrees
- moved Q1 349.8 mm to (183.0, 65.4), turned to 90 degrees
- moved Q3 347.9 mm to (183.0, 74.6), turned to 90 degrees
- moved R7 346.2 mm to (182.0, 89.3)
- moved Q2 339.4 mm to (191.4, 65.7), turned to 90 degrees
- moved Q4 337.6 mm to (191.4, 74.8), turned to 90 degrees
- moved R1 337.2 mm to (182.0, 87.5)
- moved R8 335.2 mm to (192.2, 87.5)
- moved R9 334.9 mm to (192.2, 89.3)
- moved C8 332.5 mm to (182.0, 80.6)
- moved C10 332.1 mm to (182.0, 82.4)
- moved C12 324.5 mm to (187.9, 81.9)
- moved D1 316.1 mm to (192.2, 80.6)
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Routing:
- net /M-: track 0.00 -> 8.05 mm
- net /M+: track 0.00 -> 7.58 mm
- net GND: track 12.0 -> 17.1 mm
- net Net-(U13-LO): track 0.00 -> 0.97 mm
