File: Hardware/Science Actuation/Science_Actuation.kicad_sch (KiCad schematic)
At the start: 108 parts, among them J2 RJ45_LED_Shielded, Q1 BSS138, Q10 AO3401A, Q9 BSS138, SW1 SW_Push, SW10 SW_SPDT, SW2 SW_Push, SW3 SW_Push, SW4 SW_Push, SW5 SW_Push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

Commit message: Updated Science Actuation schematic (removed some unnecessary components)
Parts:
- removed Conn14, Conn15, Conn16, Conn18: Molex_SL_03, MRDT_Connectors:MOLEX_SL_03_Vertical, symbol MRDT_Connectors:Molex_SL_03
- removed Conn2, Conn6 (x2), Conn8: Molex_SL_02, MRDT_Connectors:MOLEX_SL_02_Vertical, symbol MRDT_Connectors:Molex_SL_02
- removed D1, D16 (x2): Orange, LED_SMD:LED_0603_1608Metric_Pad1.05x0.95mm_HandSolder, symbol Device:LED
- removed D21: Blue, LED_SMD:LED_0603_1608Metric_Pad1.05x0.95mm_HandSolder, symbol Device:LED
- removed D7: YELLOW, LED_SMD:LED_0603_1608Metric_Pad1.05x0.95mm_HandSolder, symbol Device:LED
- removed Q1, Q9 (x2): BSS138, Package_TO_SOT_SMD:SOT-23, symbol Transistor_FET:BSS138
- removed Q10 (x2): AO3401A, Package_TO_SOT_SMD:SOT-23, symbol Transistor_FET:AO3401A
- removed R1: 300, Resistor_SMD:R_0603_1608Metric_Pad0.98x0.95mm_HandSolder, symbol Device:R
- removed R26, R7: 100, Resistor_SMD:R_0603_1608Metric_Pad0.98x0.95mm_HandSolder, symbol Device:R
- removed R36 (x2): 4.7k, Resistor_SMD:R_0603_1608Metric_Pad0.98x0.95mm_HandSolder, symbol Device:R
- removed R37 (x2), R38 (x2): 10k, Resistor_SMD:R_0603_1608Metric_Pad0.98x0.95mm_HandSolder, symbol Device:R
- removed R39 (x2): 1k, Resistor_SMD:R_0603_1608Metric_Pad0.98x0.95mm_HandSolder, symbol Device:R
- removed SW8: SW_Push, Button_Switch_SMD:SW_SPST_TL3305A, symbol Switch:SW_Push
- added Conn2: Molex_SL_03, MRDT_Connectors:MOLEX_SL_03_Vertical, symbol MRDT_Connectors:Molex_SL_03
Connections:
- net +3V3: now also Conn2.1
- net Heater_On: no longer names the net of U2.20 (A6)
- net Heater_On2: no longer names the net of U2.9 (OUT1C)
- net Heater_On3 renamed MOCO_SP_RVS
- net MOCO_SP_RVS: now also Conn2.3
- net Heater_On4: no longer names the net of U2.28 (RX7)
- net Heater_Temp: no longer names the net of U2.19 (A5)
- net Heater_Temp2: no longer names the net of U2.10 (CS1)
- net Heater_Temp3 renamed MOCO_SP_FWD
- net MOCO_SP_FWD: now also Conn2.2
- net Heater_Temp4: no longer names the net of U2.33 (MCLK2)
- net LAS: no longer names the net of U2.31 (CTX3)
- net LimitSwitch6: no longer names the net of U2.30 (CRX3)
- net Pump1: no longer names the net of U2.27 (A13)
- net Pump2: no longer names the net of U2.26 (A12)
- net SW8: no longer names the net of U2.34 (RX8)
- net Servo_2 renamed Servo_SP
Other:
- note added: "DIR. SWITCH"
- note removed: "Heater"
- note removed: "LASER"
- note removed: "Pumps"
- moved on the sheet: C3, C4, Conn10, Conn11, Conn17, Conn9, D12, D13, D14, D15, D16, D17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

Commit message: Updated Science Actuation again (definitely not finished)
Parts:
- added D30, D31: YELLOW, LED_SMD:LED_0603_1608Metric_Pad1.05x0.95mm_HandSolder, symbol Device:LED
- added QuadEncode4: Molex_SL_04, MRDT_Connectors:MOLEX_SL_04_Vertical, symbol MRDT_Connectors:Molex_SL_04
- added R40, R41: 100, Resistor_SMD:R_0603_1608Metric_Pad0.98x0.95mm_HandSolder, symbol Device:R
Connections:
- net +5V: now also QuadEncode4.1
- net DIR_SW: now also U2.31 (CTX3)
- net GND: now also D30.1 (K), D31.1 (K), QuadEncode4.4
- net LimitSwitch5: no longer U2.24 (A10)
- net MOCO1_FWD: now also U2.9 (OUT1C); no longer U2.5 (IN2)
- net MOCO1_RVS: now also U2.10 (CS1); no longer U2.6 (OUT1D)
- net MOCO2_FWD: now also U2.11 (MOSI)
- net MOCO2_RVS: now also U2.12 (MISO)
- net MOCO4_FWD: now also U2.5 (IN2); no longer U2.7 (RX2)
- net MOCO4_RVS: now also U2.6 (OUT1D); no longer U2.8 (TX2)
- net MOCO_SP_FWD: now also U2.8 (TX2); no longer U2.12 (MISO)
- net MOCO_SP_RVS: now also U2.7 (RX2); no longer U2.11 (MOSI)
- net SW1: now also U2.26 (A12); no longer U2.41 (A17)
- net SW2: now also U2.25 (A11); no longer U2.40 (A16)
- net SW3: now also U2.24 (A10); no longer U2.39 (A15)
- net SW4: now also U2.27 (A13), U2.36 (CS2); no longer U2.38 (A14)
- net SW5: now also U2.28 (RX7)
- net SW6: now also U2.29 (TX7); no longer U2.36 (CS2)
- net SW7: now also U2.30 (CRX3)
- net Servo_1: no longer U2.25 (A11)
- net Servo_SP: no longer U2.29 (TX7)
- new net: D30.2 (A), R40.1
- new net: D31.2 (A), R41.2
- new net Encoder_4a: QuadEncode4.2, R40.2
- new net Encoder_4b: QuadEncode4.3, R41.1
- new net a: U2.38 (A14), U2.40 (A16)
- new net q: U2.41 (A17)
- new net s: U2.39 (A15)
- no-connect marks 10 -> 14
Other:
- moved on the sheet: Conn10, Conn11, Conn17, Conn2, Conn3, Conn4, Conn5, Conn6, Conn7, Conn9, D2, D3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
